File: zasilanie/projekt/rov4/Rov4PS_HP.sch (KiCad schematic (older format))
At the start: 67 parts, among them IC2 UWE-12_10-Q12PB-C, J22 Manip_Silnik_1, J23 Manip_Silnik_2, J25 Extra, J26 Extra, J28 ESC2, J29 ESC3, J30 Torpedy_serwo_7v, J31 ESC4, J32 ESC5, J33 Extra, J34 ESC6, J35 Extra, J36 ESC7, J37 ESC8, J38 Manip_sil_12v, J39 Torp_EleMagnes, J40 Manip_serwo, J41 Extra, J42 Extra, J43 Extra, J44 Extra, J46 RC_HP_12V, J47 ESC1, Q6 Q, Q7 Q, U3 Transoptor, U4 XL4015, U7 XL4015, U8 XL4015, U9 Transoptor

Commit message: Modyfikacje schematu i PCB
Parts:
- removed C18: 33uF, Capacitor_SMD:C_2816_7142Metric_Pad3.20x4.45mm_HandSolder, symbol Device:C_Small
- removed C19: 1uF, Capacitor_SMD:C_0805_2012Metric_Pad1.15x1.40mm_HandSolder, symbol Device:C_Small
- removed C20: 10uF, Capacitor_SMD:C_0805_2012Metric_Pad1.15x1.40mm_HandSolder, symbol Device:C_Small
- removed C21: 5000uF, Capacitor_SMD:C_Elec_8x10.2, symbol Device:C_Small
- removed D16, D18, D20: LED_B, LED_SMD:LED_0805_2012Metric_Pad1.15x1.40mm_HandSolder, symbol Device:LED_Small
- removed F4: 20A_fast, symbol Device:Fuse
- removed R11: 2k2, Resistor_SMD:R_0805_2012Metric_Pad1.15x1.40mm_HandSolder, symbol Device:R_Small
- removed R12: 800, Resistor_SMD:R_0805_2012Metric_Pad1.15x1.40mm_HandSolder, symbol Device:R_Small
- removed R14: 400, Resistor_SMD:R_0805_2012Metric_Pad1.15x1.40mm_HandSolder, symbol Device:R_Small
- removed U7: XL4015, XL4015:xl4015, symbol XL4015:XL4015
- added C18: 33uF, Capacitor_SMD:CP_Elec_6.3x5.4, symbol Device:CP_Small
- added C24, C25, C26, C27: 100nF, Capacitor_SMD:C_0805_2012Metric, symbol Device:C_Small
- added C28: 10uF, Capacitor_SMD:C_0805_2012Metric, symbol Device:C_Small
- added C29: 200uF, Capacitor_SMD:CP_Elec_8x10, symbol Device:CP_Small
- added J18: HP_Enable, Connector_PinHeader_2.54mm:PinHeader_1x02_P2.54mm_Vertical, symbol Connector_Generic:Conn_01x02
- added TP6: HP_14V, Connector_PinHeader_2.54mm:PinHeader_1x01_P2.54mm_Vertical, symbol Connector:TestPoint
- added TP7: HP_7V, Connector_PinHeader_2.54mm:PinHeader_1x01_P2.54mm_Vertical, symbol Connector:TestPoint
- added TP8: HP_12V, Connector_PinHeader_2.54mm:PinHeader_1x01_P2.54mm_Vertical, symbol Connector:TestPoint
- added TP9: HP_5V, Connector_PinHeader_2.54mm:PinHeader_1x01_P2.54mm_Vertical, symbol Connector:TestPoint
- added U5: XL4015, XL4015:xl4015, symbol XL4015:XL4015
- D12, D14, D19: footprint LED_SMD:LED_0805_2012Metric_Pad1.15x1.40mm_HandSolder -> LED_SMD:LED_0805_2012Metric
- D13, D15, D17: footprint Diode_SMD:D_MiniMELF_Handsoldering -> Diode_SMD:D_MiniMELF
- J46: footprint Connector_PinHeader_2.54mm:PinHeader_1x01_P2.54mm_Vertical -> Connector_PinHeader_2.54mm:PinHeader_1x02_P2.54mm_Vertical
- Q6, Q7: footprint (none) -> Package_TO_SOT_THT:TO-220-3_Vertical
- R10, R13, R9: footprint Resistor_SMD:R_0805_2012Metric_Pad1.15x1.40mm_HandSolder -> Resistor_SMD:R_0805_2012Metric
Connections:
- net +BattPow: now also IC2.1 (+VIN), C18.1, U5.1 (Vin)
- net GND: now also C18.2, C24.2, C25.2, C26.2, C27.2, C28.2, C29.2, U5.2 (GND), U5.4 (GND)
- net at IC2.7 (+SENSE), IC2.8 (+VOUT), J38.1 (Pin_1)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: now also C26.1, C28.1, C29.1, TP8.1
- net at J30.1 (Pin_1), J33.1 (Pin_1), J35.1 (Pin_1): now also C25.1, TP7.1, U5.3 (Vout)
- net at J40.1 (Pin_1), J43.1 (Pin_1), J44.1 (Pin_1)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: now also C27.1, TP9.1
- net at J22.1 (Pin_1), J23.1 (Pin_1), J25.1 (Pin_1)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: now also C24.1, TP6.1
- net GNDD: no longer names the net of U3.2
- net GNDD: now also J18.1 (Pin_1)
- net PowerEnable: no longer names the net of U3.1
- net PowerEnable: now also J18.2 (Pin_2)
Other:
- note added: "Da sie\n"
- note removed: "CHYBA SIE TAK NIE DA"

Commit message: Update
Parts:
- removed D12: LED_R, LED_SMD:LED_0805_2012Metric, symbol Device:LED
- removed D13, D15: BAT48, Diode_SMD:D_MiniMELF, symbol Device:D_Schottky_Small
- removed D14: LED_G, LED_SMD:LED_0805_2012Metric, symbol Device:LED
- removed Q6, Q7: Q, Package_TO_SOT_THT:TO-220-3_Vertical, symbol Device:Q_NMOS_GDS
- removed U5, U8: XL4015, XL4015:xl4015, symbol XL4015:XL4015
- added D10: LED_G, LED_SMD:LED_0805_2012Metric, symbol Device:LED
- added D11: LED_R, LED_SMD:LED_0805_2012Metric, symbol Device:LED
- added D12, D13: BAT48, Diode_SMD:D_MiniMELF, symbol Device:D_Schottky
- added Q6, Q7, Q8, Q9: IPT004N03L, Package_TO_SOT_SMD:Infineon_PG-HSOF-8-1, symbol Device:Q_NMOS_GSD
- added R8: 3k, Resistor_SMD:R_0805_2012Metric, symbol Device:R
- added U4, U5: lm2596, lm2596:lm2596-44_8mm_x_23mm, symbol lm2596:lm2596
- C22: renamed from C10; footprint (none) -> Capacitor_THT:C_Radial_D12.5mm_H25.0mm_P5.00mm
- C23: renamed from C11; footprint (none) -> Capacitor_THT:C_Radial_D12.5mm_H25.0mm_P5.00mm
- C24: renamed from C12; footprint (none) -> Capacitor_THT:C_Radial_D12.5mm_H25.0mm_P5.00mm
- C25: renamed from C13; footprint (none) -> Capacitor_THT:C_Radial_D12.5mm_H25.0mm_P5.00mm
- C26: renamed from C14; footprint (none) -> Capacitor_THT:C_Radial_D12.5mm_H25.0mm_P5.00mm
- C27: renamed from C15; footprint (none) -> Capacitor_THT:C_Radial_D12.5mm_H25.0mm_P5.00mm
- C28: renamed from C16; footprint (none) -> Capacitor_THT:C_Radial_D12.5mm_H25.0mm_P5.00mm
- C29: renamed from C17; footprint (none) -> Capacitor_THT:C_Radial_D12.5mm_H20.0mm_P5.00mm
- J39: renamed from J47; footprint (none) -> rozlaczna_gniazdo_5_08:2_pin_5_08mm
- J40: renamed from J28; footprint (none) -> rozlaczna_gniazdo_5_08:2_pin_5_08mm
- J41: renamed from J29; footprint (none) -> rozlaczna_gniazdo_5_08:2_pin_5_08mm
- J42: renamed from J31; footprint (none) -> rozlaczna_gniazdo_5_08:2_pin_5_08mm
- J43: renamed from J32; footprint (none) -> rozlaczna_gniazdo_5_08:2_pin_5_08mm
- J44: renamed from J34; footprint (none) -> rozlaczna_gniazdo_5_08:2_pin_5_08mm
- J45: renamed from J36; footprint (none) -> rozlaczna_gniazdo_5_08:2_pin_5_08mm
- J46: renamed from J37; footprint (none) -> rozlaczna_gniazdo_5_08:2_pin_5_08mm
- L1, L2, L3, L4, L5, L6, L7, L8: footprint (none) -> 74435571100:74435571100
- R10: value 3k -> 10k
- R9: value 10k -> 100
- renumbered C18 to C15, C26 to C16, C28 to C17, C29 to C18, C25 to C19, C27 to C20, C24 to C21, D19 to D14, D17 to D9, J18 to J23, J38 to J24, J39 to J25, J42 to J26, J46 to J27, J41 to J28, J30 to J29, J33 to J30, J35 to J31, J40 to J32, J43 to J33, J44 to J34, J22 to J35, J23 to J36, J25 to J37, J26 to J38, R13 to R11, TP8 to TP6, TP9 to TP8, TP6 to TP9, U3 to U2, U9 to U3, U4 to U6
Connections:
- net +BattPow: now also Q7.1 (G), Q9.1 (G), R8.1, U4.1 (Vin), U5.1 (Vin); no longer R10.1
- net -BattPower: now also R10.2, D12.1 (K), D13.2 (A), Q6.2 (S), Q8.2 (S); no longer R9.1
- net GND: now also Q7.2 (S), Q9.2 (S), U4.2 (GND), U4.4 (GND), U5.2 (GND), U5.4 (GND)
- net at C19.1, J29.1 (Pin_1), J30.1 (Pin_1)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: now also U4.3 (Vout)
- net at C20.1, J32.1 (Pin_1), J33.1 (Pin_1)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: now also U5.3 (Vout)
- net at D9.2 (A), U2.3: now also R9.1; no longer R9.2
- new net: Q6.3 (D), Q7.3 (D), Q8.3 (D), Q9.3 (D)
- new net: Q6.1 (G), Q8.1 (G), R10.1, R9.2
- new net: D10.2 (A), D11.1 (K), R8.2
- new net: D10.1 (K), D12.2 (A)
- new net: D11.2 (A), D13.1 (K)
Other:
- moved on the sheet: C21, D9, J23, J35, J36, J37, J38, TP9, U2, U6

Commit message: sync
Parts:
- removed J37: Extra, Connector_PinHeader_2.54mm:PinHeader_1x02_P2.54mm_Vertical, symbol Connector_Generic:Conn_01x02
- added C30: 100nF, Capacitor_SMD:C_0805_2012Metric, symbol Device:C_Small
- added J51, J52: Extra, Connector_PinHeader_2.54mm:PinHeader_1x02_P2.54mm_Vertical, symbol Connector_Generic:Conn_01x02
- added TP10: EXTRA, Connector_PinHeader_2.54mm:PinHeader_1x01_P2.54mm_Vertical, symbol Connector:TestPoint
- added U7: lm2596, lm2596:lm2596-44_8mm_x_23mm, symbol lm2596:lm2596
Connections:
- net labels added: +BattDigit, -BattDigit
- wire segments 241 -> 271
Other:
- moved on the sheet: J35, J36
Changed lines of the file:
@@
 L Connector_Generic:Conn_01x02 J?
 U 1 1 5C9B947B
-P 2850 4700
+P 9300 3050
 AR Path="/5C9B947B" Ref="J?"  Part="1"
 AR Path="/5C93D53B/5C9B947B" Ref="J35"  Part="1"
-F 0 "J35" H 3050 4600 50  0000 R CNN
-F 1 "Manip_Silnik_1" H 3050 4500 39  0000 R CNN
-F 2 "Connector_PinHeader_2.54mm:PinHeader_1x02_P2.54mm_Vertical" H 2850 4700 50  0001 C CNN
-F 3 "~" H 2850 4700 50  0001 C CNN
-	1    2850 4700
+F 0 "J35" H 9500 2950 50  0000 R CNN
+F 1 "Manip_Silnik_1" H 9500 2850 39  0000 R CNN
+F 2 "Connector_PinHeader_2.54mm:PinHeader_1x02_P2.54mm_Vertical" H 9300 3050 50  0001 C CNN
+F 3 "~" H 9300 3050 50  0001 C CNN
+	1    9300 3050
 	0    -1   1    0
 $EndComp
@@
 L Connector_Generic:Conn_01x02 J?
 U 1 1 5C9C12E4
-P 3350 4700
+P 9800 3050
 AR Path="/5C9C12E4" Ref="J?"  Part="1"
 AR Path="/5C93D53B/5C9C12E4" Ref="J36"  Part="1"
-F 0 "J36" H 3550 4600 50  0000 R CNN
-F 1 "Manip_Silnik_2" H 3550 4500 39  0000 R CNN
-F 2 "Connector_PinHeader_2.54mm:PinHeader_1x02_P2.54mm_Vertical" H 3350 4700 50  0001 C CNN
-F 3 "~" H 3350 4700 50  0001 C CNN
-	1    3350 4700
+F 0 "J36" H 10000 2950 50  0000 R CNN
+F 1 "Manip_Silnik_2" H 10000 2850 39  0000 R CNN
+F 2 "Connector_PinHeader_2.54mm:PinHeader_1x02_P2.54mm_Vertical" H 9800 3050 50  0001 C CNN
+F 3 "~" H 9800 3050 50  0001 C CNN
+	1    9800 3050
 	0    -1   1    0
 $EndComp
@@
 	1    10500 2850
 	1    0    0    -1
-$EndComp
-$Comp
-L Connector_Generic:Conn_01x02 J?
-U 1 1 5CAF206E
-P 4150 4700
-AR Path="/5CAF206E" Ref="J?"  Part="1"
-AR Path="/5C93D53B/5CAF206E" Ref="J38"  Part="1"
-F 0 "J38" V 4050 4550 50  0000 R CNN
-F 1 "Extra" V 4250 4750 50  0000 R CNN
-F 2 "Connector_PinHeader_2.54mm:PinHeader_1x02_P2.54mm_Vertical" H 4150 4700 50  0001 C CNN
-F 3 "~" H 4150 4700 50  0001 C CNN
-	1    4150 4700
-	0    -1   1    0
-$EndComp
-$Comp
-L Connector_Generic:Conn_01x02 J?
-U 1 1 5CAF2075
-P 3750 4700
-AR Path="/5CAF2075" Ref="J?"  Part="1"
-AR Path="/5C93D53B/5CAF2075" Ref="J37"  Part="1"
-F 0 "J37" V 3650 4550 50  0000 R CNN
-F 1 "Extra" V 3850 4750 50  0000 R CNN
-F 2 "Connector_PinHeader_2.54mm:PinHeader_1x02_P2.54mm_Vertical" H 3750 4700 50  0001 C CNN
-F 3 "~" H 3750 4700 50  0001 C CNN
-	1    3750 4700
-	0    -1   1    0
 $EndComp
 $Comp
@@
 Connection ~ 10150 2550
 Wire Wire Line
-	10150 2550 10150 2850
+	10150 2550 10150 2750
 Wire Wire Line
 	10300 2850 10150 2850
@@
 	10300 2950 10250 2950
 Wire Wire Line
-	10250 2950 10250 2650
+	10250 2950 10250 2800
 Connection ~ 10250 2250
 Connection ~ 10250 2650
@@
 	9200 3900 9250 3900
 Connection ~ 9250 3900
+$Comp
+L Connector_Generic:Conn_01x02 J52
+U 1 1 5CC73B50
+P 3150 6200
+F 0 "J52" V 3050 6050 50  0000 R CNN
+F 1 "Extra" V 3250 6250 50  0000 R CNN
+F 2 "Connector_PinHeader_2.54mm:PinHeader_1x02_P2.54mm_Vertical" H 3150 6200 50  0001 C CNN
+F 3 "~" H 3150 6200 50  0001 C CNN
+	1    3150 6200
+	0    -1   1    0
+$EndComp
+$Comp
+L Connector_Generic:Conn_01x02 J51
+U 1 1 5CC73B57
+P 2750 6200
+F 0 "J51" V 2650 6050 50  0000 R CNN
+F 1 "Extra" V 2850 6250 50  0000 R CNN
+F 2 "Connector_PinHeader_2.54mm:PinHeader_1x02_P2.54mm_Vertical" H 2750 6200 50  0001 C CNN
+F 3 "~" H 2750 6200 50  0001 C CNN
+	1    2750 6200
+	0    -1   1    0
+$EndComp
+$Comp
+L Connector_Generic:Conn_01x02 J38
+U 1 1 5CC73B5E
+P 2350 6200
+F 0 "J38" V 2250 6050 50  0000 R CNN
+F 1 "Extra" V 2450 6250 50  0000 R CNN
+F 2 "Connector_PinHeader_2.54mm:PinHeader_1x02_P2.54mm_Vertical" H 2350 6200 50  0001 C CNN
+F 3 "~" H 2350 6200 50  0001 C CNN
+	1    2350 6200
+	0    -1   1    0
+$EndComp
+Wire Wire Line
+	2350 5400 2350 6000
+Wire Wire Line
+	2450 5900 2850 5900
+Wire Wire Line
+	3250 6000 3250 5900
+Wire Wire Line
+	2850 6000 2850 5900
+Connection ~ 2850 5900
+Wire Wire Line
+	2850 5900 3250 5900
+Wire Wire Line
+	2750 6000 2750 5400
+Connection ~ 2750 5400
+Wire Wire Line
+	2750 5400 2350 5400
+Wire Wire Line
+	3150 6000 3150 5400
+Wire Wire Line
+	2750 5400 3150 5400
+Connection ~ 2450 5900
+Wire Wire Line
+	2450 5900 2450 6000
+Connection ~ 2350 5400
+Text GLabel 1150 5400 0    50   Input ~ 0
++BattDigit
+$Comp
+L Connector:TestPoint TP10
+U 1 1 5CC73B74
+P 2350 5350
+F 0 "TP10" H 2409 5471 50  0000 L CNN
+F 1 "EXTRA" H 2409 5378 50  0000 L CNN
+F 2 "Connector_PinHeader_2.54mm:PinHeader_1x01_P2.54mm_Vertical" H 2550 5350 50  0001 C CNN
+F 3 "~" H 2550 5350 50  0001 C CNN
+	1    2350 5350
+	1    0    0    -1
+$EndComp
+Wire Wire Line
+	2350 5400 2350 5350
+$Comp
+L Device:C_Small C?
+U 1 1 5CC73B7C
+P 2050 5600
+AR Path="/5CC73B7C" Ref="C?"  Part="1"
+AR Path="/5C93D53B/5CC73B7C" Ref="C30"  Part="1"
+F 0 "C30" H 2075 5675 50  0000 L CNN
+F 1 "100nF" H 2075 5525 50  0000 L CNN
+F 2 "Capacitor_SMD:C_0805_2012Metric" H 2050 5600 50  0001 C CNN
+F 3 "~" H 2050 5600 50  0001 C CNN
+	1    2050 5600
+	1    0    0    -1
+$EndComp
+Wire Wire Line
+	2050 5500 2050 5400
+Wire Wire Line
+	2050 5700 2050 5900
+Connection ~ 2050 5900
+Wire Wire Line
+	2050 5900 2450 5900
+Wire Wire Line
+	2000 5400 2050 5400
+Wire Wire Line
+	2350 5400 2050 5400
+Connection ~ 2050 5400
+Text GLabel 1150 5900 0    50   Input ~ 0
+-BattDigit
+$Comp
+L lm2596:lm2596 U7
+U 1 1 5CC73B8B
+P 1600 5400
+F 0 "U7" H 1600 5719 50  0000 C CNN
+F 1 "lm2596" H 1600 5626 50  0000 C CNN
+F 2 "lm2596:lm2596-44_8mm_x_23mm" H 1600 5300 50  0001 C CNN
+F 3 "" H 1600 5300 50  0001 C CNN
+	1    1600 5400
+	1    0    0    -1
+$EndComp
+Wire Wire Line
+	1600 5650 1600 5900
+Wire Wire Line
+	1600 5900 2050 5900
+Connection ~ 1600 5900
+Wire Wire Line
+	1200 5400 1150 5400
+Wire Wire Line
+	1150 5900 1600 5900
+Wire Wire Line
+	9300 2850 9300 2750
+Wire Wire Line
+	9300 2750 9800 2750
+Connection ~ 10150 2750
+Wire Wire Line
+	10150 2750 10150 2850
+Wire Wire Line
+	9800 2850 9800 2750
+Connection ~ 9800 2750
+Wire Wire Line
+	9800 2750 10150 2750
+Wire Wire Line
+	9400 2850 9400 2800
+Wire Wire Line
+	9400 2800 9900 2800
+Wire Wire Line
+	9900 2800 9900 2850
+Wire Wire Line
+	9900 2800 10250 2800
+Connection ~ 9900 2800
+Connection ~ 10250 2800
+Wire Wire Line
+	10250 2800 10250 2650
 $EndSCHEMATC

Commit message: test2
Parts:
- removed C21: 100nF, Capacitor_SMD:C_0805_2012Metric, symbol Device:C_Small
- removed TP9: HP_14V, Connector_PinHeader_2.54mm:PinHeader_1x01_P2.54mm_Vertical, symbol Connector:TestPoint
- removed U6: XL4015, XL4015:xl4015, symbol XL4015:XL4015
Connections:
- net labels removed: +BattDigit, -BattDigit
- wire segments 271 -> 247
Other:
- note added: "Osobne pcb"
- note removed: "14v"
- note removed: "Da sie\n"
- moved on the sheet: C19, C20, C22, C23, C24, C25, C26, C27, C28, C29, C30, J29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
