File: zasilanie/projekt/rov4/rov4.kicad_pcb (KiCad board)
At the start: 2 copper layers, 105 parts, among them IC1 UWE-12_10-Q12PB-C, IC2 UWE-12_10-Q12PB-C, J1 Battery digital, J10 Switch, J11 Kamera 1, J12 Extra, J13 Kamera 2, J14 Extra, J15 Extra, J16 Extra, J17 BatteryPower, J18 RPi_PowerEnable, J2 Reed switch, J20 Manip_SterSil1, J21 Manip_SterSil2, J22 Manip_Silnik_1, J23 Manip_Silnik_2, J24 RC_D_15V, J25 Extra, J26 Extra, J27 RC_D_5V, J3 Extra, J30 Torpedy_serwo_7v, J33 Extra, J35 Extra, J38 Manip_sil_12v, J39 Torp_EleMagnes, J4 Extra, J40 Manip_serwo, J41 Extra, J42 Extra, J43 Extra, J44 Extra, J45 RC_D_12V, J46 RC_HP_12V, J5 Extra, J6 RPi, J7 Router, J8 Xavier, J9 Hydrofony, Q1 IRFZ44N, Q2 Q_NPN_BCE, Q3 Q_NPN_BCE, Q4 Q_NPN_BCE, U1 HFV7A_012ZST, U2 XL4015, U3 Transoptor, U4 XL4015, U7 XL4015, U8 XL4015, U9 Transoptor

Commit message: Modyfikacje schematu i PCB
Parts:
- removed D16, D18, D20, D3: LED_B, LED_SMD:LED_0805_2012Metric_Pad1.15x1.40mm_HandSolder
- removed R11: 2k2, Resistor_SMD:R_0805_2012Metric_Pad1.15x1.40mm_HandSolder
- removed R12: 800, Resistor_SMD:R_0805_2012Metric_Pad1.15x1.40mm_HandSolder
- removed R14: 400, Resistor_SMD:R_0805_2012Metric_Pad1.15x1.40mm_HandSolder
- removed R3: 3k, Resistor_SMD:R_0805_2012Metric_Pad1.15x1.40mm_HandSolder
- removed U7: XL4015, XL4015:xl4015
- added C22: 200uF, Capacitor_SMD:CP_Elec_8x10, B.Cu at (223.5, 62.2)
- added C23: 100nF, Capacitor_SMD:C_0805_2012Metric, B.Cu at (232.4, 146.1)
- added C24: 100nF, Capacitor_SMD:C_0805_2012Metric, B.Cu at (69.8, 76.2)
- added C25: 100nF, Capacitor_SMD:C_0805_2012Metric, B.Cu at (69.8, 141.0)
- added C26: 100nF, Capacitor_SMD:C_0805_2012Metric, B.Cu at (95.2, 180.3)
- added C27: 100nF, Capacitor_SMD:C_0805_2012Metric, B.Cu at (69.8, 106.7)
- added C28: 10uF, Capacitor_SMD:C_0805_2012Metric, B.Cu at (87.6, 180.3)
- added C29: 200uF, Capacitor_SMD:CP_Elec_8x10, B.Cu at (80.0, 180.3)
- added Q6: Q, Package_TO_SOT_THT:TO-220-3_Vertical, F.Cu at (59.7, 35.6)
- added Q7: Q, Package_TO_SOT_THT:TO-220-3_Vertical, F.Cu at (53.3, 40.6)
- added TP6: HP_14V, Connector_PinHeader_2.54mm:PinHeader_1x01_P2.54mm_Vertical, F.Cu at (77.5, 67.3)
- added TP7: HP_7V, Connector_PinHeader_2.54mm:PinHeader_1x01_P2.54mm_Vertical, F.Cu at (77.5, 132.1)
- added TP8: HP_12V, Connector_PinHeader_2.54mm:PinHeader_1x01_P2.54mm_Vertical, F.Cu at (100.3, 172.7)
- added TP9: HP_5V, Connector_PinHeader_2.54mm:PinHeader_1x01_P2.54mm_Vertical, F.Cu at (76.2, 97.8)
- added U5: XL4015, XL4015:xl4015, F.Cu at (44.5, 141.0)
- C1, C18, C2, C3: footprint Capacitor_SMD:C_2816_7142Metric_Pad3.20x4.45mm_HandSolder -> Capacitor_SMD:CP_Elec_6.3x5.4; moved to B.Cu
- C19, C4, C6: value 1uF -> 100nF; footprint Capacitor_SMD:C_0805_2012Metric_Pad1.15x1.40mm_HandSolder -> Capacitor_SMD:C_0805_2012Metric; moved to B.Cu
- C20: value 10uF -> 200uF; footprint Capacitor_SMD:C_0805_2012Metric_Pad1.15x1.40mm_HandSolder -> Capacitor_SMD:CP_Elec_8x10; moved to B.Cu
- C21: value 5000uF -> 10uF; footprint Capacitor_SMD:C_Elec_8x10.2 -> Capacitor_SMD:C_0805_2012Metric; moved to B.Cu
- C5: footprint Capacitor_SMD:C_0805_2012Metric_Pad1.15x1.40mm_HandSolder -> Capacitor_SMD:C_0805_2012Metric; moved to B.Cu
- C7: value 5000uF -> 100nF; footprint Capacitor_SMD:C_Elec_8x10.2 -> Capacitor_SMD:C_0805_2012Metric; moved to B.Cu
- C8: value 10uF -> 100uF; footprint Capacitor_SMD:C_0805_2012Metric_Pad1.15x1.40mm_HandSolder -> Capacitor_SMD:CP_Elec_6.3x7.7; moved to B.Cu
- C9: value 5000uF -> 100uF; footprint Capacitor_SMD:C_Elec_8x10.2 -> Capacitor_SMD:CP_Elec_6.3x7.7; moved to B.Cu
- D1, D2: footprint Diode_SMD:D_SMA_Handsoldering -> Diode_SMD:D_SMA; moved to B.Cu
- D10, D12, D14, D19, D4, D5, D6, D7, D8: footprint LED_SMD:LED_0805_2012Metric_Pad1.15x1.40mm_HandSolder -> LED_SMD:LED_0805_2012Metric
- D11, D13, D15, D17, D9: footprint Diode_SMD:D_MiniMELF_Handsoldering -> Diode_SMD:D_MiniMELF
- J18: value RPi_PowerEnable -> HP_Enable; footprint Connector_PinHeader_2.54mm:PinHeader_1x01_P2.54mm_Vertical -> Connector_PinHeader_2.54mm:PinHeader_1x02_P2.54mm_Vertical
- J46: footprint Connector_PinHeader_2.54mm:PinHeader_1x01_P2.54mm_Vertical -> Connector_PinHeader_2.54mm:PinHeader_1x02_P2.54mm_Vertical
- J9: footprint Connector_PinHeader_2.54mm:PinHeader_1x02_P2.54mm_Vertical -> Connector_PinHeader_2.54mm:PinHeader_1x03_P2.54mm_Vertical
- Q1: footprint Package_TO_SOT_SMD:SOT-23_Handsoldering -> Package_TO_SOT_SMD:SOT-23; moved to B.Cu
- Q2, Q3, Q4: value Q_NPN_BCE -> BC847A; footprint Package_TO_SOT_SMD:SOT-23_Handsoldering -> Package_TO_SOT_SMD:SOT-23; moved to B.Cu
- R1, R2: footprint Resistor_SMD:R_0805_2012Metric_Pad1.15x1.40mm_HandSolder -> Resistor_SMD:R_0805_2012Metric; moved to B.Cu
- R10, R13, R4, R5, R6, R7, R8, R9: footprint Resistor_SMD:R_0805_2012Metric_Pad1.15x1.40mm_HandSolder -> Resistor_SMD:R_0805_2012Metric
- TP1, TP3: value TestPoint -> D_5V
- TP2: value TestPoint -> D_-5V
- TP4: value TestPoint -> D_12V
- TP5: value TestPoint -> EXTRA
- moved C21 369.2 mm to (236.2, 62.2), turned to 270 degrees
- moved C19 317.7 mm to (238.8, 62.2), turned to 270 degrees
- moved C20 306.7 mm to (222.2, 38.1), turned to 90 degrees
- moved J39 227.5 mm to (105.4, 179.1)
- moved J40 219.1 mm to (86.4, 105.4)
- moved J38 218.8 mm to (100.3, 179.1)
- moved J41 199.4 mm to (110.5, 179.1)
- moved D17 194.4 mm to (40.6, 38.1), turned to 270 degrees
- moved J26 185.2 mm to (87.6, 74.9)
- moved D19 184.8 mm to (111.1, 172.7), turned to 180 degrees
- moved U8 184.4 mm to (44.5, 106.7)
- moved J23 177.3 mm to (82.5, 74.9)
- moved R13 175.4 mm to (105.7, 172.7)
- moved J33 174.5 mm to (83.0, 139.6)
- moved J35 173.5 mm to (77.5, 139.7)
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Connections:
- C1 pad 1: Net-(C1-Pad1) -> +BattDigit
- C18 pad 1: Net-(C18-Pad1) -> +BattPow
- C2 pad 1: Net-(C2-Pad1) -> +BattDigit
- C20 pad 1: Net-(C19-Pad1) -> Net-(C20-Pad1)
- C3 pad 1: Net-(C3-Pad1) -> +BattDigit
- C4 pad 1: Net-(C4-Pad1) -> Net-(C20-Pad1)
- C5 pad 1: Net-(C4-Pad1) -> Net-(C20-Pad1)
- C7 pad 1: Net-(C4-Pad1) -> GND
- C7 pad 2: GND -> Net-(C7-Pad2)
- C9 pad 1: Net-(C6-Pad1) -> GND
- C9 pad 2: GND -> Net-(C7-Pad2)
- IC1 pad 1: Net-(C3-Pad1) -> +BattDigit
- IC1 pad 6: Net-(IC1-Pad6) -> (no net)
- IC1 pad 7: Net-(C6-Pad1) -> Net-(C19-Pad1)
- IC1 pad 8: Net-(C6-Pad1) -> Net-(C19-Pad1)
- IC2 pad 1: Net-(C18-Pad1) -> +BattPow
- IC2 pad 6: Net-(IC2-Pad6) -> (no net)
- IC2 pad 7: Net-(C19-Pad1) -> Net-(C26-Pad1)
- IC2 pad 8: Net-(C19-Pad1) -> Net-(C26-Pad1)
- J10 pad 1: Net-(C4-Pad1) -> Net-(C20-Pad1)
- J11 pad 1: Net-(C6-Pad1) -> Net-(C19-Pad1)
- J12 pad 1: Net-(C4-Pad1) -> Net-(C20-Pad1)
- J13 pad 1: Net-(C6-Pad1) -> Net-(C19-Pad1)
- J14 pad 1: Net-(C4-Pad1) -> Net-(C20-Pad1)
- J15 pad 1: Net-(C6-Pad1) -> Net-(C19-Pad1)
- J16 pad 1: Net-(C6-Pad1) -> Net-(C19-Pad1)
- J18 pad 1: /Rov4PS_HP/PowerEnable -> Net-(J18-Pad1)
- J20 pad 1: Net-(C4-Pad1) -> Net-(C20-Pad1)
- J21 pad 1: Net-(C4-Pad1) -> Net-(C20-Pad1)
- J38 pad 1: Net-(C19-Pad1) -> Net-(C26-Pad1)
- J39 pad 1: Net-(C19-Pad1) -> Net-(C26-Pad1)
- J41 pad 1: Net-(C19-Pad1) -> Net-(C26-Pad1)
- J42 pad 1: Net-(C19-Pad1) -> Net-(C26-Pad1)
- J6 pad 1: Net-(C4-Pad1) -> Net-(C20-Pad1)
- J7 pad 1: Net-(C4-Pad1) -> Net-(C20-Pad1)
- J8 pad 1: Net-(C6-Pad1) -> Net-(C19-Pad1)
- J9 pad 1: Net-(J9-Pad1) -> Net-(C6-Pad1)
- PS1 pad 1: Net-(C2-Pad1) -> +BattDigit
- PS1 pad 4: Net-(PS1-Pad4) -> (no net)
- PS1 pad 6: Net-(C4-Pad1) -> Net-(C20-Pad1)
- PS2 pad 11: Net-(J9-Pad3) -> Net-(C7-Pad2)
- PS2 pad 14: Net-(J9-Pad1) -> Net-(C6-Pad1)
- PS2 pad 22: Net-(C1-Pad1) -> +BattDigit
- PS2 pad 23: Net-(C1-Pad1) -> +BattDigit
- Q2 pad 2: Net-(PS2-Pad1) -> GND
- Q2 pad 3: GND -> Net-(PS2-Pad1)
- Q3 pad 1: Net-(J27-Pad1) -> Net-(J45-Pad1)
- Q3 pad 2: Net-(PS1-Pad3) -> GND
- Q3 pad 3: GND -> Net-(IC1-Pad2)
- Q4 pad 1: Net-(J45-Pad1) -> Net-(J27-Pad1)
- Q4 pad 2: Net-(IC1-Pad2) -> GND
- Q4 pad 3: GND -> Net-(PS1-Pad3)
- R13 pad 1: Net-(C19-Pad1) -> Net-(C26-Pad1)
- R4 pad 2: Net-(J9-Pad1) -> Net-(C6-Pad1)
- R5 pad 1: Net-(J9-Pad3) -> Net-(C7-Pad2)
- R6 pad 2: Net-(C4-Pad1) -> Net-(C20-Pad1)
- R7 pad 2: Net-(C6-Pad1) -> Net-(C19-Pad1)
- TP1 pad 1: Net-(J9-Pad1) -> Net-(C6-Pad1)
- TP2 pad 1: Net-(J9-Pad3) -> Net-(C7-Pad2)
- TP3 pad 1: Net-(C4-Pad1) -> Net-(C20-Pad1)
- TP4 pad 1: Net-(C6-Pad1) -> Net-(C19-Pad1)
- U1 pad 87a: Net-(U1-Pad87a) -> (no net)
- U3 pad 1: /Rov4PS_HP/PowerEnable -> Net-(J18-Pad2)
- U3 pad 2: GND -> Net-(J18-Pad1)

Commit message: Update
Parts:
- removed D15, D17: BAT48, Diode_SMD:D_MiniMELF
- removed D19: LED_B, LED_SMD:LED_0805_2012Metric
- removed R13: 1k8, Resistor_SMD:R_0805_2012Metric
- removed U8: XL4015, XL4015:xl4015
- removed U9: Transoptor, Package_DIP:DIP-4_W7.62mm
- added C10: 100nF, Capacitor_SMD:C_0805_2012Metric, B.Cu at (199.7, 165.1)
- added C11: 100uF, Capacitor_SMD:CP_Elec_6.3x7.7, B.Cu at (201.9, 151.8)
- added C12: 33uF, Capacitor_SMD:CP_Elec_6.3x5.4, B.Cu at (196.8, 142.2)
- added C13: 100nF, Capacitor_SMD:C_0805_2012Metric, B.Cu at (194.0, 165.1)
- added C14: 100uF, Capacitor_SMD:CP_Elec_6.3x7.7, B.Cu at (191.8, 151.8)
- added C15: 33uF, Capacitor_SMD:CP_Elec_6.3x5.4, B.Cu at (132.1, 134.6)
- added C16: 100nF, Capacitor_SMD:C_0805_2012Metric, B.Cu at (132.1, 181.6)
- added C17: 10uF, Capacitor_SMD:C_0805_2012Metric, B.Cu at (132.1, 185.4)
- added D3: BAT48, Diode_SMD:D_MiniMELF, F.Cu at (226.7, 20.3)
- added J19: Extra, Connector_PinHeader_2.54mm:PinHeader_1x02_P2.54mm_Vertical, F.Cu at (289.6, 148.0)
- added J28: Extra, Connector_PinHeader_2.54mm:PinHeader_1x02_P2.54mm_Vertical, F.Cu at (129.5, 190.5)
- added J29: Torpedy_serwo_7v, Connector_PinHeader_2.54mm:PinHeader_1x02_P2.54mm_Vertical, F.Cu at (91.4, 180.3)
- added J31: Extra, Connector_PinHeader_2.54mm:PinHeader_1x02_P2.54mm_Vertical, F.Cu at (99.1, 188.0)
- added J32: Manip_serwo, Connector_PinHeader_2.54mm:PinHeader_1x02_P2.54mm_Vertical, F.Cu at (63.5, 180.3)
- added J34: Extra, Connector_PinHeader_2.54mm:PinHeader_1x02_P2.54mm_Vertical, F.Cu at (71.1, 188.0)
- added J36: Manip_Silnik_2, Connector_PinHeader_2.54mm:PinHeader_1x02_P2.54mm_Vertical, F.Cu at (27.9, 188.0)
- added J37: Extra, Connector_PinHeader_2.54mm:PinHeader_1x02_P2.54mm_Vertical, F.Cu at (35.6, 188.0)
- added L1: L, 74435571100:74435571100, F.Cu at (104.1, 36.8)
- added L2: L, 74435571100:74435571100, F.Cu at (81.3, 36.8)
- added L3: L, 74435571100:74435571100, F.Cu at (58.4, 36.8)
- added L4: L, 74435571100:74435571100, F.Cu at (35.6, 36.8)
- added L5: L, 74435571100:74435571100, F.Cu at (35.6, 66.0)
- added L6: L, 74435571100:74435571100, F.Cu at (61.0, 66.0)
- added L7: L, 74435571100:74435571100, F.Cu at (86.4, 66.0)
- added L8: L, 74435571100:74435571100, F.Cu at (111.8, 66.0)
- added Q5: BC847A, Package_TO_SOT_SMD:SOT-23, B.Cu at (194.3, 134.6)
- added Q8: IPT004N03L, Package_TO_SOT_SMD:Infineon_PG-HSOF-8-1, F.Cu at (144.8, 41.7)
- added Q9: IPT004N03L, Package_TO_SOT_SMD:Infineon_PG-HSOF-8-1, F.Cu at (144.8, 24.5)
- added R11: 1k8, Resistor_SMD:R_0805_2012Metric, F.Cu at (138.4, 184.5)
- added R3: 10k, Resistor_SMD:R_0805_2012Metric, F.Cu at (233.0, 22.9)
- added U6: XL4015, XL4015:xl4015, F.Cu at (35.6, 147.3)
- C18: value 33uF -> 200uF; footprint Capacitor_SMD:CP_Elec_6.3x5.4 -> Capacitor_SMD:CP_Elec_8x10
- C2: value 33uF -> 100nF; footprint Capacitor_SMD:CP_Elec_6.3x5.4 -> Capacitor_SMD:C_0805_2012Metric
- C20: value 200uF -> 100nF; footprint Capacitor_SMD:CP_Elec_8x10 -> Capacitor_SMD:C_0805_2012Metric
- C21: value 10uF -> 100nF
- C22: value 200uF -> C; footprint Capacitor_SMD:CP_Elec_8x10 -> Capacitor_THT:C_Radial_D12.5mm_H25.0mm_P5.00mm; moved to F.Cu
- C23, C24, C25, C26, C27: value 100nF -> C; footprint Capacitor_SMD:C_0805_2012Metric -> Capacitor_THT:C_Radial_D12.5mm_H25.0mm_P5.00mm; moved to F.Cu
- C28: value 10uF -> C; footprint Capacitor_SMD:C_0805_2012Metric -> Capacitor_THT:C_Radial_D12.5mm_H25.0mm_P5.00mm; moved to F.Cu
- C29: value 200uF -> C; footprint Capacitor_SMD:CP_Elec_8x10 -> Capacitor_THT:C_Radial_D12.5mm_H20.0mm_P5.00mm; moved to F.Cu
- C3: value 33uF -> 10uF; footprint Capacitor_SMD:CP_Elec_6.3x5.4 -> Capacitor_SMD:C_0805_2012Metric
- C4: value 100nF -> 200uF; footprint Capacitor_SMD:C_0805_2012Metric -> Capacitor_SMD:CP_Elec_8x10
- C5: value 10uF -> 33uF; footprint Capacitor_SMD:C_0805_2012Metric -> Capacitor_SMD:CP_Elec_6.3x5.4
- C7: value 100nF -> 10uF
- C8: value 100uF -> 200uF; footprint Capacitor_SMD:CP_Elec_6.3x7.7 -> Capacitor_SMD:CP_Elec_8x10
- C9: value 100uF -> 100nF; footprint Capacitor_SMD:CP_Elec_6.3x7.7 -> Capacitor_SMD:C_0805_2012Metric
- D1: value SS34 -> LED_G; footprint Diode_SMD:D_SMA -> LED_SMD:LED_0805_2012Metric; moved to F.Cu
- D10: value LED_B -> LED_G
- D11: value BAT48 -> LED_R; footprint Diode_SMD:D_MiniMELF -> LED_SMD:LED_0805_2012Metric
- D12: value LED_R -> BAT48; footprint LED_SMD:LED_0805_2012Metric -> Diode_SMD:D_MiniMELF
- D14: value LED_G -> LED_B
- D2: value SS34 -> LED_R; footprint Diode_SMD:D_SMA -> LED_SMD:LED_0805_2012Metric; moved to F.Cu
- D4: value LED_B -> BAT48; footprint LED_SMD:LED_0805_2012Metric -> Diode_SMD:D_MiniMELF
- J1: value Battery digital -> Reed switch
- J11: value Kamera 1 -> BatteryPower
- J12: value Extra -> RC_D_12V; footprint Connector_PinHeader_2.54mm:PinHeader_1x02_P2.54mm_Vertical -> Connector_PinHeader_2.54mm:PinHeader_1x01_P2.54mm_Vertical
- J13: value Kamera 2 -> Xavier
- J14: value Extra -> Kamera 1
- J15: value Extra -> Kamera 2
- J17: value BatteryPower -> Extra
- J18: value HP_Enable -> Hydrofony; footprint Connector_PinHeader_2.54mm:PinHeader_1x02_P2.54mm_Vertical -> Connector_PinHeader_2.54mm:PinHeader_1x03_P2.54mm_Vertical
- J2: value Reed switch -> Battery digital; footprint Connector_PinHeader_2.54mm:PinHeader_1x02_P2.54mm_Vertical -> Connector_PinSocket_2.54mm:PinSocket_2x01_P2.54mm_Vertical
- J20: value Manip_SterSil1 -> Extra
- J21: value Manip_SterSil2 -> Extra
- J22: value Manip_Silnik_1 -> RC_D_15V; footprint Connector_PinHeader_2.54mm:PinHeader_1x02_P2.54mm_Vertical -> Connector_PinHeader_2.54mm:PinHeader_1x01_P2.54mm_Vertical
- J23: value Manip_Silnik_2 -> HP_Enable
- J24: value RC_D_15V -> Manip_sil_12v; footprint Connector_PinHeader_2.54mm:PinHeader_1x01_P2.54mm_Vertical -> Connector_PinHeader_2.54mm:PinHeader_1x02_P2.54mm_Vertical
- J25: value Extra -> Torp_EleMagnes
- J27: value RC_D_5V -> RC_HP_12V; footprint Connector_PinHeader_2.54mm:PinHeader_1x01_P2.54mm_Vertical -> Connector_PinHeader_2.54mm:PinHeader_1x02_P2.54mm_Vertical
- J3: value Extra -> Manip_SterSil2
- J30: value Torpedy_serwo_7v -> Extra
- J35: value Extra -> Manip_Silnik_1
- J38: value Manip_sil_12v -> Extra
- J39: value Torp_EleMagnes -> ESC1; footprint Connector_PinHeader_2.54mm:PinHeader_1x02_P2.54mm_Vertical -> rozlaczna_gniazdo_5_08:2_pin_5_08mm
- J4: value Extra -> Manip_SterSil1
- J40: value Manip_serwo -> ESC2; footprint Connector_PinHeader_2.54mm:PinHeader_1x02_P2.54mm_Vertical -> rozlaczna_gniazdo_5_08:2_pin_5_08mm
- J41: value Extra -> ESC3; footprint Connector_PinHeader_2.54mm:PinHeader_1x02_P2.54mm_Vertical -> rozlaczna_gniazdo_5_08:2_pin_5_08mm
- J42: value Extra -> ESC4; footprint Connector_PinHeader_2.54mm:PinHeader_1x02_P2.54mm_Vertical -> rozlaczna_gniazdo_5_08:2_pin_5_08mm
- J43: value Extra -> ESC5; footprint Connector_PinHeader_2.54mm:PinHeader_1x02_P2.54mm_Vertical -> rozlaczna_gniazdo_5_08:2_pin_5_08mm
- J44: value Extra -> ESC6; footprint Connector_PinHeader_2.54mm:PinHeader_1x02_P2.54mm_Vertical -> rozlaczna_gniazdo_5_08:2_pin_5_08mm
- J45: value RC_D_12V -> ESC7; footprint Connector_PinHeader_2.54mm:PinHeader_1x01_P2.54mm_Vertical -> rozlaczna_gniazdo_5_08:2_pin_5_08mm
- J46: value RC_HP_12V -> ESC8; footprint Connector_PinHeader_2.54mm:PinHeader_1x02_P2.54mm_Vertical -> rozlaczna_gniazdo_5_08:2_pin_5_08mm
- J6: value RPi -> Extra
- J7: value Router -> RC_D_5V; footprint Connector_PinHeader_2.54mm:PinHeader_1x02_P2.54mm_Vertical -> Connector_PinHeader_2.54mm:PinHeader_1x01_P2.54mm_Vertical
- J8: value Xavier -> RPi
- J9: value Hydrofony -> Router; footprint Connector_PinHeader_2.54mm:PinHeader_1x03_P2.54mm_Vertical -> Connector_PinHeader_2.54mm:PinHeader_1x02_P2.54mm_Vertical
- Q1: value IRFZ44N -> IPT004N03L; footprint Package_TO_SOT_SMD:SOT-23 -> Package_TO_SOT_SMD:Infineon_PG-HSOF-8-1; moved to F.Cu
- Q2: value BC847A -> IPT004N03L; footprint Package_TO_SOT_SMD:SOT-23 -> Package_TO_SOT_SMD:Infineon_PG-HSOF-8-1; moved to F.Cu
- Q6, Q7: value Q -> IPT004N03L; footprint Package_TO_SOT_THT:TO-220-3_Vertical -> Package_TO_SOT_SMD:Infineon_PG-HSOF-8-1
- R1: value 1k -> 3k; moved to F.Cu
- R10: value 3k -> 10k
- R2: value 100k -> 100; moved to F.Cu
- R4: value 2k4 -> 400
- R5: value 2k4 -> 1k8
- R6: value 400 -> 2k4
- R7: value 1k8 -> 2k4
- R9: value 10k -> 100
- TP2: value D_-5V -> D_12V
- TP3: value D_5V -> EXTRA
- TP4: value D_12V -> D_5V
- TP5: value EXTRA -> D_-5V
- TP6: value HP_14V -> HP_12V
- TP8: value HP_12V -> HP_5V
- TP9: value HP_5V -> HP_14V
- U1: value HFV7A_012ZST -> lm2596; footprint Custom Relay:HFV7A_012ZST -> lm2596:lm2596-44_8mm_x_23mm
- U2: value XL4015 -> Transoptor; footprint XL4015:xl4015 -> Package_DIP:DIP-4_W7.62mm
- U4, U5: value XL4015 -> lm2596; footprint XL4015:xl4015 -> lm2596:lm2596-44_8mm_x_23mm
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Connections:
- C1 pad 2: GND -> -BattDigit
- C18 pad 1: +BattPow -> Net-(C16-Pad1)
- C18 pad 2: GND -> -BattPow
- C19 pad 2: GND -> -BattPow
- C2 pad 1: +BattDigit -> Net-(C2-Pad1)
- C2 pad 2: GND -> -BattDigit
- C20 pad 2: GND -> -BattPow
- C21 pad 1: Net-(C19-Pad1) -> Net-(C21-Pad1)
- C21 pad 2: GND -> -BattPow
- C22 pad 1: Net-(C19-Pad1) -> Net-(C22-Pad1)
- C22 pad 2: GND -> -BattPow
- C23 pad 2: GND -> -BattPow
- C24 pad 2: GND -> -BattPow
- C25 pad 2: GND -> -BattPow
- C26 pad 2: GND -> -BattPow
- C27 pad 2: GND -> -BattPow
- C28 pad 1: Net-(C26-Pad1) -> Net-(C28-Pad1)
- C28 pad 2: GND -> -BattPow
- C29 pad 1: Net-(C26-Pad1) -> Net-(C29-Pad1)
- C29 pad 2: GND -> -BattPow
- C3 pad 1: +BattDigit -> Net-(C2-Pad1)
- C3 pad 2: GND -> -BattDigit
- C4 pad 1: Net-(C20-Pad1) -> Net-(C2-Pad1)
- C4 pad 2: GND -> -BattDigit
- C5 pad 1: Net-(C20-Pad1) -> +BattDigit
- C5 pad 2: GND -> -BattDigit
- C6 pad 2: GND -> -BattDigit
- C7 pad 1: GND -> Net-(C6-Pad1)
- C7 pad 2: Net-(C7-Pad2) -> -BattDigit
- C8 pad 2: GND -> -BattDigit
- C9 pad 1: GND -> Net-(C9-Pad1)
- C9 pad 2: Net-(C7-Pad2) -> -BattDigit
- D1 pad 1: /+Batt -> Net-(D1-Pad1)
- D11 pad 1: GND -> Net-(D10-Pad2)
- D11 pad 2: Net-(D10-Pad1) -> Net-(D11-Pad2)
- D12 pad 1: Net-(D12-Pad1) -> /Rov4PS_HP/-BattPower
- D12 pad 2: Net-(D12-Pad2) -> Net-(D10-Pad1)
- D13 pad 1: Net-(D12-Pad2) -> Net-(D11-Pad2)
- D14 pad 1: Net-(D14-Pad1) -> -BattPow
- D14 pad 2: Net-(D12-Pad1) -> Net-(D14-Pad2)
- D2 pad 1: Net-(D2-Pad1) -> Net-(D1-Pad2)
- D2 pad 2: Net-(D1-Pad2) -> Net-(D2-Pad2)
- D4 pad 1: GND -> Net-(D2-Pad2)
- D4 pad 2: Net-(D4-Pad2) -> /-Batt
- D5 pad 1: Net-(D5-Pad1) -> -BattDigit
- D5 pad 2: GND -> Net-(D5-Pad2)
- D6 pad 1: GND -> -BattDigit
- D7 pad 1: GND -> -BattDigit
- D8 pad 1: Net-(D10-Pad2) -> Net-(D8-Pad1)
- D8 pad 2: Net-(D8-Pad2) -> -BattDigit
- D9 pad 1: Net-(D8-Pad2) -> +BattPow
- D9 pad 2: GND -> Net-(D9-Pad2)
- IC1 pad 3: GND -> -BattDigit
- IC1 pad 4: GND -> -BattDigit
- IC1 pad 5: GND -> -BattDigit
- IC1 pad 7: Net-(C19-Pad1) -> Net-(C6-Pad1)
- IC1 pad 8: Net-(C19-Pad1) -> Net-(C6-Pad1)
- IC2 pad 3: GND -> -BattPow
- IC2 pad 4: GND -> -BattPow
- IC2 pad 5: GND -> -BattPow
- IC2 pad 7: Net-(C26-Pad1) -> Net-(C16-Pad1)
- IC2 pad 8: Net-(C26-Pad1) -> Net-(C16-Pad1)
- J1 pad 1: /+Batt -> Net-(J1-Pad1)
- J1 pad 2: GND -> +BattDigit
- J10 pad 1: Net-(C20-Pad1) -> Net-(C2-Pad1)
- J10 pad 2: GND -> -BattDigit
- J11 pad 1: Net-(C19-Pad1) -> +BattPow
- J11 pad 2: GND -> /Rov4PS_HP/-BattPower
- J12 pad 1: Net-(C20-Pad1) -> Net-(J12-Pad1)
- J13 pad 1: Net-(C19-Pad1) -> Net-(C6-Pad1)
- J13 pad 2: GND -> -BattDigit
- J14 pad 1: Net-(C20-Pad1) -> Net-(C6-Pad1)
- J14 pad 2: GND -> -BattDigit
- J15 pad 1: Net-(C19-Pad1) -> Net-(C6-Pad1)
- J15 pad 2: GND -> -BattDigit
- J16 pad 1: Net-(C19-Pad1) -> Net-(C6-Pad1)
- J16 pad 2: GND -> -BattDigit
- J17 pad 1: +BattPow -> Net-(C6-Pad1)
- J17 pad 2: /Rov4PS_HP/-BattPower -> -BattDigit
- J18 pad 1: Net-(J18-Pad1) -> Net-(C10-Pad1)
- J18 pad 2: Net-(J18-Pad2) -> -BattDigit
- J2 pad 1: /+Batt -> +BattDigit
- J2 pad 2: Net-(J2-Pad2) -> /-Batt
- J20 pad 1: Net-(C20-Pad1) -> Net-(C9-Pad1)
- J20 pad 2: Net-(J20-Pad2) -> -BattDigit
- J21 pad 1: Net-(C20-Pad1) -> Net-(C9-Pad1)
- J21 pad 2: GND -> -BattDigit
- J22 pad 1: Net-(C24-Pad1) -> Net-(J22-Pad1)
- J23 pad 1: Net-(C24-Pad1) -> Net-(J23-Pad1)
- J23 pad 2: GND -> Net-(J23-Pad2)
- J24 pad 1: Net-(J24-Pad1) -> Net-(C16-Pad1)
- J25 pad 1: Net-(C24-Pad1) -> Net-(C16-Pad1)
- J25 pad 2: GND -> -BattPow
- J26 pad 1: Net-(C24-Pad1) -> Net-(C16-Pad1)
- J26 pad 2: GND -> -BattPow
- J3 pad 1: Net-(C23-Pad1) -> Net-(C2-Pad1)
- J3 pad 2: GND -> -BattDigit
- J30 pad 1: Net-(C25-Pad1) -> Net-(C19-Pad1)
- J30 pad 2: GND -> -BattPow
- J33 pad 1: Net-(C25-Pad1) -> Net-(C20-Pad1)
- J33 pad 2: GND -> -BattPow
- J35 pad 1: Net-(C25-Pad1) -> Net-(C21-Pad1)
- J35 pad 2: GND -> -BattPow
- J38 pad 1: Net-(C26-Pad1) -> Net-(C21-Pad1)
- J38 pad 2: GND -> -BattPow
- J39 pad 1: Net-(C26-Pad1) -> Net-(C22-Pad1)
- J39 pad 2: GND -> -BattPow
- J4 pad 1: Net-(C23-Pad1) -> Net-(C2-Pad1)
- J4 pad 2: GND -> Net-(J4-Pad2)
- J40 pad 1: Net-(C27-Pad1) -> Net-(C23-Pad1)
- J40 pad 2: GND -> -BattPow
- J41 pad 1: Net-(C26-Pad1) -> Net-(C24-Pad1)
- J41 pad 2: GND -> -BattPow
- J42 pad 1: Net-(C26-Pad1) -> Net-(C25-Pad1)
- J42 pad 2: GND -> -BattPow
- J43 pad 1: Net-(C27-Pad1) -> Net-(C26-Pad1)
- J43 pad 2: GND -> -BattPow
- J44 pad 2: GND -> -BattPow
- J45 pad 1: Net-(J45-Pad1) -> Net-(C28-Pad1)
- J46 pad 1: Net-(J46-Pad1) -> Net-(C29-Pad1)
- J46 pad 2: Net-(J46-Pad2) -> -BattPow
- J5 pad 1: Net-(C23-Pad1) -> Net-(C2-Pad1)
- J5 pad 2: GND -> -BattDigit
- J6 pad 1: Net-(C20-Pad1) -> Net-(C2-Pad1)
- J6 pad 2: GND -> -BattDigit
- J7 pad 1: Net-(C20-Pad1) -> Net-(J7-Pad1)
- J8 pad 1: Net-(C19-Pad1) -> Net-(C2-Pad1)
- J8 pad 2: GND -> -BattDigit
- J9 pad 1: Net-(C6-Pad1) -> Net-(C2-Pad1)
- J9 pad 2: GND -> Net-(J4-Pad2)
- PS1 pad 2: GND -> -BattDigit
- PS1 pad 5: GND -> -BattDigit
- PS1 pad 6: Net-(C20-Pad1) -> Net-(C2-Pad1)
- PS2 pad 11: Net-(C7-Pad2) -> Net-(C13-Pad2)
- PS2 pad 14: Net-(C6-Pad1) -> Net-(C10-Pad1)
- PS2 pad 16: GND -> -BattDigit
- PS2 pad 2: GND -> -BattDigit
- PS2 pad 3: GND -> -BattDigit
- PS2 pad 9: GND -> -BattDigit
- Q1 pad 2: Net-(D2-Pad1) -> /-Batt
- Q1 pad 3: GND -> Net-(Q1-Pad3)
- Q2 pad 1: Net-(J24-Pad1) -> +BattDigit
- Q2 pad 2: GND -> -BattDigit
- Q2 pad 3: Net-(PS2-Pad1) -> Net-(Q1-Pad3)
- Q3 pad 1: Net-(J45-Pad1) -> Net-(J7-Pad1)
- Q3 pad 2: GND -> -BattDigit
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Routing:
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
Commit message: idea slotow
Parts:
- Q7, Q9: moved to B.Cu
- moved J46 230.3 mm to (-113.0, 30.5), turned to 180 degrees
- moved C29 222.7 mm to (-101.6, 27.9), turned to 0 degrees
- moved L8 218.0 mm to (-105.4, 47.0), turned to 180 degrees
- moved J45 171.4 mm to (-64.8, 7.62), turned to 180 degrees
- moved C28 166.3 mm to (-67.3, 25.4), turned to 180 degrees
- moved L7 151.2 mm to (-63.5, 45.7), turned to 180 degrees
- moved J44 134.2 mm to (-44.5, 7.62), turned to 180 degrees
- moved C27 124.4 mm to (-47.0, 25.4), turned to 180 degrees
- moved L6 106.1 mm to (-43.2, 45.7), turned to 180 degrees
- moved J43 100.0 mm to (-24.1, 7.62), turned to 180 degrees
- moved C26 80.8 mm to (-26.7, 25.4), turned to 180 degrees
- moved D10 79.7 mm to (195.3, 23.5)
- moved D11 79.7 mm to (195.3, 26.0)
- moved D12 79.7 mm to (197.0, 21.0)
- moved D13 79.7 mm to (197.0, 28.6)
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Routing:
- net -BattPow: track 0.00 -> 322.6 mm
- net Net-(C28-Pad1): track 0.00 -> 30.9 mm

Commit message: test
Parts:
- Q7, Q9: moved to F.Cu
- moved Q9 101.4 mm to (168.2, 55.9)
- moved Q7 76.8 mm to (154.8, 55.9)
- moved Q8 1.98 mm to (168.2, 72.2)

Commit message: footprint list
Parts:
- added J47: Extra, Connector_Molex:Molex_Mini-Fit_Jr_5566-02A_2x01_P4.20mm_Vertical, F.Cu at (394.4, -4.84)
- added J48: Extra, Connector_Molex:Molex_Mini-Fit_Jr_5566-02A_2x01_P4.20mm_Vertical, F.Cu at (400.8, -4.84)
- added J49: Extra, Connector_Molex:Molex_Mini-Fit_Jr_5566-02A_2x01_P4.20mm_Vertical, F.Cu at (369.0, -4.84)
- added J50: Extra, Connector_Molex:Molex_Mini-Fit_Jr_5566-02A_2x01_P4.20mm_Vertical, F.Cu at (375.4, -4.84)
- added J51: Extra, Connector_Molex:Molex_Mini-Fit_Jr_5566-02A_2x01_P4.20mm_Vertical, F.Cu at (381.9, -4.84)
- added J52: HP_OUT, Connector_Molex:Molex_Mini-Fit_Jr_5566-04A_2x02_P4.20mm_Vertical, F.Cu at (302.9, -46.5)
- added J53: HP_IN, Connector_Molex:Molex_Mini-Fit_Jr_5566-04A_2x02_P4.20mm_Vertical, F.Cu at (328.1, -46.5)
- added J54: HP_IN, Connector_Molex:Molex_Mini-Fit_Jr_5566-04A_2x02_P4.20mm_Vertical, F.Cu at (353.2, -62.0)
- added J55: LP_OUT, Connector_Molex:Molex_Mini-Fit_Jr_5566-04A_2x02_P4.20mm_Vertical, F.Cu at (302.9, -62.0)
- added J56: LP_IN, Connector_Molex:Molex_Mini-Fit_Jr_5566-04A_2x02_P4.20mm_Vertical, F.Cu at (328.1, -62.0)
- C10, C13: value 100nF -> 100uF; footprint Capacitor_SMD:C_0805_2012Metric -> Capacitor_SMD:CP_Elec_6.3x7.7
- C11: value 100uF -> 33uF; footprint Capacitor_SMD:CP_Elec_6.3x7.7 -> Capacitor_SMD:CP_Elec_6.3x5.4
- C12: value 33uF -> 100nF; footprint Capacitor_SMD:CP_Elec_6.3x5.4 -> Capacitor_SMD:C_0805_2012Metric
- C14: value 100uF -> 100nF; footprint Capacitor_SMD:CP_Elec_6.3x7.7 -> Capacitor_SMD:C_0805_2012Metric
- C15: value 33uF -> C; footprint Capacitor_SMD:CP_Elec_6.3x5.4 -> Capacitor_THT:C_Radial_D10.0mm_H20.0mm_P5.00mm
- C16, C19, C20, C21: value 100nF -> C; footprint Capacitor_SMD:C_0805_2012Metric -> Capacitor_THT:C_Radial_D10.0mm_H20.0mm_P5.00mm
- C17: value 10uF -> C; footprint Capacitor_SMD:C_0805_2012Metric -> Capacitor_THT:C_Radial_D10.0mm_H20.0mm_P5.00mm
- C18: value 200uF -> C; footprint Capacitor_SMD:CP_Elec_8x10 -> Capacitor_THT:C_Radial_D10.0mm_H20.0mm_P5.00mm
- C22: footprint Capacitor_THT:C_Radial_D12.5mm_H25.0mm_P5.00mm -> Capacitor_THT:C_Radial_D12.5mm_H20.0mm_P5.00mm
- C23: value C -> 33uF; footprint Capacitor_THT:C_Radial_D12.5mm_H25.0mm_P5.00mm -> Capacitor_SMD:CP_Elec_6.3x5.4
- C24, C27, C28: value C -> 100nF; footprint Capacitor_THT:C_Radial_D12.5mm_H25.0mm_P5.00mm -> Capacitor_SMD:C_0805_2012Metric
- C25: value C -> 10uF; footprint Capacitor_THT:C_Radial_D12.5mm_H25.0mm_P5.00mm -> Capacitor_SMD:C_0805_2012Metric
- C26: value C -> 200uF; footprint Capacitor_THT:C_Radial_D12.5mm_H25.0mm_P5.00mm -> Capacitor_SMD:CP_Elec_8x10
- C29: value C -> 100nF; footprint Capacitor_THT:C_Radial_D12.5mm_H20.0mm_P5.00mm -> Capacitor_SMD:C_0805_2012Metric
- J1: value Reed switch -> Battery digital; footprint Connector_PinHeader_2.54mm:PinHeader_1x02_P2.54mm_Vertical -> power_connectors:XT60UPB-M
- J10: value Switch -> Router; footprint Connector_PinHeader_2.54mm:PinHeader_1x02_P2.54mm_Vertical -> Connector_Molex:Molex_Mini-Fit_Jr_5566-02A_2x01_P4.20mm_Vertical
- J11: value BatteryPower -> Switch; footprint Connector_PinHeader_2.54mm:PinHeader_1x02_P2.54mm_Vertical -> Connector_Molex:Molex_Mini-Fit_Jr_5566-02A_2x01_P4.20mm_Vertical
- J12: value RC_D_12V -> Enko_inkrementalny; footprint Connector_PinHeader_2.54mm:PinHeader_1x01_P2.54mm_Vertical -> Connector_Molex:Molex_Mini-Fit_Jr_5566-02A_2x01_P4.20mm_Vertical
- J13: value Xavier -> Torpedy, hall, laser; footprint Connector_PinHeader_2.54mm:PinHeader_1x02_P2.54mm_Vertical -> Connector_Molex:Molex_Mini-Fit_Jr_5566-02A_2x01_P4.20mm_Vertical
- J14: value Kamera 1 -> Enko_absolutny_1; footprint Connector_PinHeader_2.54mm:PinHeader_1x02_P2.54mm_Vertical -> Connector_Molex:Molex_Mini-Fit_Jr_5566-02A_2x01_P4.20mm_Vertical
- J15: value Kamera 2 -> Enko_absolutny_2; footprint Connector_PinHeader_2.54mm:PinHeader_1x02_P2.54mm_Vertical -> Connector_Molex:Molex_Mini-Fit_Jr_5566-02A_2x01_P4.20mm_Vertical
- J16: value Extra -> RC_D_12V; footprint Connector_PinHeader_2.54mm:PinHeader_1x02_P2.54mm_Vertical -> Connector_PinHeader_2.54mm:PinHeader_1x01_P2.54mm_Vertical
- J17: value Extra -> Xavier; footprint Connector_PinHeader_2.54mm:PinHeader_1x02_P2.54mm_Vertical -> Connector_Molex:Molex_Mini-Fit_Jr_5566-02A_2x01_P4.20mm_Vertical
- J18: value Hydrofony -> Kamera 1; footprint Connector_PinHeader_2.54mm:PinHeader_1x03_P2.54mm_Vertical -> Connector_Molex:Molex_Mini-Fit_Jr_5566-02A_2x01_P4.20mm_Vertical
- J19: value Extra -> Kamera 2; footprint Connector_PinHeader_2.54mm:PinHeader_1x02_P2.54mm_Vertical -> Connector_Molex:Molex_Mini-Fit_Jr_5566-02A_2x01_P4.20mm_Vertical
- J2: value Battery digital -> Reed switch; footprint Connector_PinSocket_2.54mm:PinSocket_2x01_P2.54mm_Vertical -> Connector_Molex:Molex_SPOX_5267-02A_1x02_P2.50mm_Vertical
- J20, J21, J26, J38, J6: footprint Connector_PinHeader_2.54mm:PinHeader_1x02_P2.54mm_Vertical -> Connector_Molex:Molex_Mini-Fit_Jr_5566-02A_2x01_P4.20mm_Vertical
- J22: value RC_D_15V -> hydrofony; footprint Connector_PinHeader_2.54mm:PinHeader_1x01_P2.54mm_Vertical -> Connector_Molex:Molex_Mini-Fit_Jr_5566-04A_2x02_P4.20mm_Vertical
- J23: value HP_Enable -> RC_D_15V; footprint Connector_PinHeader_2.54mm:PinHeader_1x02_P2.54mm_Vertical -> Connector_PinHeader_2.54mm:PinHeader_1x01_P2.54mm_Vertical
- J24: value Manip_sil_12v -> Extra; footprint Connector_PinHeader_2.54mm:PinHeader_1x02_P2.54mm_Vertical -> Connector_Molex:Molex_Mini-Fit_Jr_5566-02A_2x01_P4.20mm_Vertical
- J25: value Torp_EleMagnes -> Extra; footprint Connector_PinHeader_2.54mm:PinHeader_1x02_P2.54mm_Vertical -> Connector_Molex:Molex_Mini-Fit_Jr_5566-02A_2x01_P4.20mm_Vertical
- J27: value RC_HP_12V -> HP_Enable; footprint Connector_PinHeader_2.54mm:PinHeader_1x02_P2.54mm_Vertical -> Connector_Molex:Molex_SPOX_5267-02A_1x02_P2.50mm_Vertical
- J28: value Extra -> ESC1; footprint Connector_PinHeader_2.54mm:PinHeader_1x02_P2.54mm_Vertical -> Connector_Molex:Molex_Mini-Fit_Jr_5566-04A_2x02_P4.20mm_Vertical
- J29: value Torpedy_serwo_7v -> ESC2; footprint Connector_PinHeader_2.54mm:PinHeader_1x02_P2.54mm_Vertical -> Connector_Molex:Molex_Mini-Fit_Jr_5566-04A_2x02_P4.20mm_Vertical
- J3: value Manip_SterSil2 -> RC_D_5V; footprint Connector_PinHeader_2.54mm:PinHeader_1x02_P2.54mm_Vertical -> Connector_PinHeader_2.54mm:PinHeader_1x01_P2.54mm_Vertical
- J30: value Extra -> ESC3; footprint Connector_PinHeader_2.54mm:PinHeader_1x02_P2.54mm_Vertical -> Connector_Molex:Molex_Mini-Fit_Jr_5566-04A_2x02_P4.20mm_Vertical
- J31: value Extra -> ESC4; footprint Connector_PinHeader_2.54mm:PinHeader_1x02_P2.54mm_Vertical -> Connector_Molex:Molex_Mini-Fit_Jr_5566-04A_2x02_P4.20mm_Vertical
- J32: value Manip_serwo -> ESC5; footprint Connector_PinHeader_2.54mm:PinHeader_1x02_P2.54mm_Vertical -> Connector_Molex:Molex_Mini-Fit_Jr_5566-04A_2x02_P4.20mm_Vertical
- J33: value Extra -> ESC6; footprint Connector_PinHeader_2.54mm:PinHeader_1x02_P2.54mm_Vertical -> Connector_Molex:Molex_Mini-Fit_Jr_5566-04A_2x02_P4.20mm_Vertical
- J34: value Extra -> ESC7; footprint Connector_PinHeader_2.54mm:PinHeader_1x02_P2.54mm_Vertical -> Connector_Molex:Molex_Mini-Fit_Jr_5566-04A_2x02_P4.20mm_Vertical
- J35: value Manip_Silnik_1 -> ESC8; footprint Connector_PinHeader_2.54mm:PinHeader_1x02_P2.54mm_Vertical -> Connector_Molex:Molex_Mini-Fit_Jr_5566-04A_2x02_P4.20mm_Vertical
- J36: value Manip_Silnik_2 -> Manip_sil_12v; footprint Connector_PinHeader_2.54mm:PinHeader_1x02_P2.54mm_Vertical -> Connector_Molex:Molex_Mini-Fit_Jr_5566-02A_2x01_P4.20mm_Vertical
- J37: value Extra -> Torp_EleMagnes; footprint Connector_PinHeader_2.54mm:PinHeader_1x02_P2.54mm_Vertical -> Connector_Molex:Molex_Mini-Fit_Jr_5566-02A_2x01_P4.20mm_Vertical
- J39: value ESC1 -> RC_HP_12V; footprint rozlaczna_gniazdo_5_08:2_pin_5_08mm -> Connector_Molex:Molex_SPOX_5267-02A_1x02_P2.50mm_Vertical
- J4: value Manip_SterSil1 -> Manip_SterSil2; footprint Connector_PinHeader_2.54mm:PinHeader_1x02_P2.54mm_Vertical -> Connector_Molex:Molex_Mini-Fit_Jr_5566-02A_2x01_P4.20mm_Vertical
- J40: value ESC2 -> Extra; footprint rozlaczna_gniazdo_5_08:2_pin_5_08mm -> Connector_Molex:Molex_Mini-Fit_Jr_5566-02A_2x01_P4.20mm_Vertical
- J41: value ESC3 -> Manip_Silnik_1; footprint rozlaczna_gniazdo_5_08:2_pin_5_08mm -> Connector_Molex:Molex_Mini-Fit_Jr_5566-02A_2x01_P4.20mm_Vertical
- J42: value ESC4 -> Manip_Silnik_2; footprint rozlaczna_gniazdo_5_08:2_pin_5_08mm -> Connector_Molex:Molex_Mini-Fit_Jr_5566-02A_2x01_P4.20mm_Vertical
- J43: value ESC5 -> Torpedy_serwo_7v; footprint rozlaczna_gniazdo_5_08:2_pin_5_08mm -> Connector_Molex:Molex_Mini-Fit_Jr_5566-02A_2x01_P4.20mm_Vertical
- J44: value ESC6 -> Extra; footprint rozlaczna_gniazdo_5_08:2_pin_5_08mm -> Connector_Molex:Molex_Mini-Fit_Jr_5566-02A_2x01_P4.20mm_Vertical
- J45: value ESC7 -> Extra; footprint rozlaczna_gniazdo_5_08:2_pin_5_08mm -> Connector_Molex:Molex_Mini-Fit_Jr_5566-02A_2x01_P4.20mm_Vertical
- J46: value ESC8 -> Manip_serwo; footprint rozlaczna_gniazdo_5_08:2_pin_5_08mm -> Connector_Molex:Molex_Mini-Fit_Jr_5566-02A_2x01_P4.20mm_Vertical
- J5: value Extra -> Manip_SterSil1; footprint Connector_PinHeader_2.54mm:PinHeader_1x02_P2.54mm_Vertical -> Connector_Molex:Molex_Mini-Fit_Jr_5566-02A_2x01_P4.20mm_Vertical
- J7: value RC_D_5V -> Extra; footprint Connector_PinHeader_2.54mm:PinHeader_1x01_P2.54mm_Vertical -> Connector_Molex:Molex_Mini-Fit_Jr_5566-02A_2x01_P4.20mm_Vertical
- J8: value RPi -> STM32; footprint Connector_PinHeader_2.54mm:PinHeader_1x02_P2.54mm_Vertical -> Connector_Molex:Molex_Mini-Fit_Jr_5566-02A_2x01_P4.20mm_Vertical
- J9: value Router -> RPi; footprint Connector_PinHeader_2.54mm:PinHeader_1x02_P2.54mm_Vertical -> Connector_Molex:Molex_Mini-Fit_Jr_5566-02A_2x01_P4.20mm_Vertical
- TP3: value EXTRA -> D_5V
- TP4: value D_5V -> D_-5V
- TP5: value D_-5V -> EXTRA
- TP9: value HP_14V -> EXTRA
- U6: value XL4015 -> lm2596; footprint XL4015:xl4015 -> lm2596:lm2596-44_8mm_x_23mm
Connections:
- C11 pad 1: Net-(C10-Pad1) -> +BattDigit
- C12 pad 1: +BattDigit -> -BattDigit
- C12 pad 2: -BattDigit -> Net-(C12-Pad2)
- C13 pad 2: Net-(C13-Pad2) -> Net-(C12-Pad2)
- C14 pad 1: -BattDigit -> Net-(C14-Pad1)
- C14 pad 2: Net-(C13-Pad2) -> Net-(C14-Pad2)
- C15 pad 1: +BattPow -> Net-(C15-Pad1)
- C17 pad 1: Net-(C16-Pad1) -> Net-(C17-Pad1)
- C18 pad 1: Net-(C16-Pad1) -> Net-(C18-Pad1)
- C23 pad 1: Net-(C23-Pad1) -> +BattPow
- C25 pad 1: Net-(C25-Pad1) -> Net-(C24-Pad1)
- C26 pad 1: Net-(C26-Pad1) -> Net-(C24-Pad1)
- C27 pad 2: -BattPow -> Net-(C27-Pad2)
- C28 pad 2: -BattPow -> Net-(C27-Pad2)
- C29 pad 2: -BattPow -> Net-(C29-Pad2)
- C9 pad 1: Net-(C9-Pad1) -> Net-(C10-Pad1)
- D12 pad 1: /Rov4PS_HP/-BattPower -> /moc_main/-BattPower
- D13 pad 2: /Rov4PS_HP/-BattPower -> /moc_main/-BattPower
- D3 pad 1: /-Batt -> /logika_main/-Batt
- D4 pad 2: /-Batt -> /logika_main/-Batt
- D5 pad 1: -BattDigit -> Net-(D5-Pad1)
- D5 pad 2: Net-(D5-Pad2) -> Net-(C2-Pad1)
- IC2 pad 7: Net-(C16-Pad1) -> Net-(C24-Pad1)
- IC2 pad 8: Net-(C16-Pad1) -> Net-(C24-Pad1)
- J1 pad 1: Net-(J1-Pad1) -> +BattDigit
- J1 pad 2: +BattDigit -> /logika_main/-Batt
- J10 pad 2: -BattDigit -> Net-(J10-Pad2)
- J11 pad 1: +BattPow -> Net-(C2-Pad1)
- J11 pad 2: /Rov4PS_HP/-BattPower -> -BattDigit
- J12 pad 1: Net-(J12-Pad1) -> Net-(C2-Pad1)
- J13 pad 1: Net-(C6-Pad1) -> -BattDigit
- J13 pad 2: -BattDigit -> Net-(C2-Pad1)
- J16 pad 1: Net-(C6-Pad1) -> Net-(J16-Pad1)
- J18 pad 1: Net-(C10-Pad1) -> Net-(C6-Pad1)
- J19 pad 1: Net-(C9-Pad1) -> Net-(C6-Pad1)
- J2 pad 1: +BattDigit -> Net-(J2-Pad1)
- J2 pad 2: /-Batt -> +BattDigit
- J20 pad 1: Net-(C9-Pad1) -> Net-(C6-Pad1)
- J21 pad 1: Net-(C9-Pad1) -> Net-(C6-Pad1)
- J22 pad 1: Net-(J22-Pad1) -> Net-(C10-Pad1)
- J24 pad 1: Net-(C16-Pad1) -> Net-(C14-Pad1)
- J24 pad 2: -BattPow -> Net-(C14-Pad2)
- J25 pad 1: Net-(C16-Pad1) -> Net-(C14-Pad1)
- J25 pad 2: -BattPow -> Net-(C14-Pad2)
- J26 pad 1: Net-(C16-Pad1) -> Net-(C14-Pad1)
- J26 pad 2: -BattPow -> Net-(C14-Pad2)
- J28 pad 1: Net-(C16-Pad1) -> Net-(C15-Pad1)
- J28 pad 2: -BattPow -> Net-(C15-Pad1)
- J29 pad 1: Net-(C19-Pad1) -> Net-(C16-Pad1)
- J29 pad 2: -BattPow -> Net-(C16-Pad1)
- J3 pad 1: Net-(C2-Pad1) -> Net-(J3-Pad1)
- J30 pad 1: Net-(C19-Pad1) -> Net-(C17-Pad1)
- J30 pad 2: -BattPow -> Net-(C17-Pad1)
- J31 pad 1: Net-(C19-Pad1) -> Net-(C18-Pad1)
- J31 pad 2: -BattPow -> Net-(C18-Pad1)
- J32 pad 1: Net-(C20-Pad1) -> Net-(C19-Pad1)
- J32 pad 2: -BattPow -> Net-(C19-Pad1)
- J33 pad 2: -BattPow -> Net-(C20-Pad1)
- J34 pad 1: Net-(C20-Pad1) -> Net-(C21-Pad1)
- J34 pad 2: -BattPow -> Net-(C21-Pad1)
- J35 pad 1: Net-(C21-Pad1) -> Net-(C22-Pad1)
- J35 pad 2: -BattPow -> Net-(C22-Pad1)
- J36 pad 1: Net-(C21-Pad1) -> Net-(C24-Pad1)
- J37 pad 1: Net-(C21-Pad1) -> Net-(C24-Pad1)
- J38 pad 1: Net-(C21-Pad1) -> Net-(C24-Pad1)
- J39 pad 1: Net-(C22-Pad1) -> Net-(J39-Pad1)
- J39 pad 2: -BattPow -> Net-(J39-Pad2)
- J4 pad 2: Net-(J4-Pad2) -> -BattDigit
- J40 pad 1: Net-(C23-Pad1) -> Net-(C24-Pad1)
- J42 pad 1: Net-(C25-Pad1) -> Net-(C24-Pad1)
- J43 pad 1: Net-(C26-Pad1) -> Net-(C27-Pad1)
- J43 pad 2: -BattPow -> Net-(C27-Pad2)
- J44 pad 2: -BattPow -> Net-(C27-Pad2)
- J45 pad 1: Net-(C28-Pad1) -> Net-(C27-Pad1)
- J45 pad 2: -BattPow -> Net-(C27-Pad2)
- J46 pad 1: Net-(C29-Pad1) -> Net-(C28-Pad1)
- J46 pad 2: -BattPow -> Net-(C27-Pad2)
- J5 pad 2: -BattDigit -> Net-(J10-Pad2)
- J7 pad 1: Net-(J7-Pad1) -> Net-(C2-Pad1)
- J9 pad 2: Net-(J4-Pad2) -> -BattDigit
- L1 pad 2: Net-(C22-Pad1) -> Net-(C15-Pad1)
- L2 pad 2: Net-(C23-Pad1) -> Net-(C16-Pad1)
- L3 pad 2: Net-(C24-Pad1) -> Net-(C17-Pad1)
- L4 pad 2: Net-(C25-Pad1) -> Net-(C18-Pad1)
- L5 pad 2: Net-(C26-Pad1) -> Net-(C19-Pad1)
- L6 pad 2: Net-(C27-Pad1) -> Net-(C20-Pad1)
- L7 pad 2: Net-(C28-Pad1) -> Net-(C21-Pad1)
- L8 pad 2: Net-(C29-Pad1) -> Net-(C22-Pad1)
- PS2 pad 11: Net-(C13-Pad2) -> Net-(C12-Pad2)
- Q1 pad 2: /-Batt -> /logika_main/-Batt
- Q3 pad 1: Net-(J7-Pad1) -> Net-(J3-Pad1)
- Q4 pad 1: Net-(J12-Pad1) -> Net-(J16-Pad1)
- Q5 pad 1: Net-(J22-Pad1) -> Net-(J23-Pad1)
- Q6 pad 2: /Rov4PS_HP/-BattPower -> /moc_main/-BattPower
- Q8 pad 2: /Rov4PS_HP/-BattPower -> /moc_main/-BattPower
- R10 pad 2: /Rov4PS_HP/-BattPower -> /moc_main/-BattPower
- R11 pad 1: Net-(C16-Pad1) -> Net-(C24-Pad1)
- R2 pad 1: Net-(J1-Pad1) -> Net-(J2-Pad1)
- R3 pad 2: /-Batt -> /logika_main/-Batt
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Routing:
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
Commit message: pcb_logiczna rozstawienie footprintow
Parts:
- added R12: 3k3, Resistor_SMD:R_0805_2012Metric, F.Cu at (38.1, 151.1)
- added R13: 3k3, Resistor_SMD:R_0805_2012Metric, F.Cu at (33.0, 110.5)
- added R14: 3k3, Resistor_SMD:R_0805_2012Metric, F.Cu at (38.1, 196.8)
- C14, C15, C16, C17, C18, C19, C20, C21, Q3, Q4, Q5: moved to F.Cu
- J16, J23, J3: footprint Connector_PinHeader_2.54mm:PinHeader_1x01_P2.54mm_Vertical -> Connector_Molex:Molex_SPOX_5267-02A_1x02_P2.50mm_Vertical
- Q1, Q2, R2, R3: moved to B.Cu
- moved TP8 537.8 mm to (285.6, -258.5), turned to 0 degrees
- moved TP7 484.1 mm to (259.8, -222.4), turned to 0 degrees
- moved J46 482.6 mm to (274.1, -257.6), turned to 0 degrees
- moved U4 471.0 mm to (233.7, -248.8), turned to 0 degrees
- moved U5 459.7 mm to (233.7, -225.6), turned to 0 degrees
- moved C29 443.9 mm to (318.8, -114.6)
- moved TP9 443.4 mm to (315.2, -113.8), turned to 0 degrees
- moved U6 438.5 mm to (320.6, -127.2), turned to 0 degrees
- moved J45 421.2 mm to (271.9, -245.5), turned to 0 degrees
- moved J44 419.5 mm to (280.6, -257.6), turned to 0 degrees
- moved J38 412.0 mm to (150.3, -161.1), turned to 0 degrees
- moved J35 399.8 mm to (140.0, -149.0), turned to 0 degrees
- moved J31 391.7 mm to (129.4, -149.8), turned to 0 degrees
- moved J37 390.1 mm to (125.4, -137.8), turned to 0 degrees
- moved J43 389.6 mm to (261.2, -257.6), turned to 0 degrees
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Connections:
- D1 pad 1: Net-(D1-Pad1) -> /logika_main/-Batt
- D2 pad 1: Net-(D1-Pad2) -> Net-(D2-Pad1)
- D2 pad 2: Net-(D2-Pad2) -> /logika_main/-Batt
- D3 pad 1: /logika_main/-Batt -> Net-(D1-Pad2)
- D3 pad 2: Net-(D1-Pad1) -> Net-(D3-Pad2)
- D4 pad 1: Net-(D2-Pad2) -> Net-(D3-Pad2)
- D4 pad 2: /logika_main/-Batt -> Net-(D2-Pad1)
- J13 pad 1: -BattDigit -> Net-(C2-Pad1)
- J13 pad 2: Net-(C2-Pad1) -> -BattDigit
- Q3 pad 1: Net-(J3-Pad1) -> Net-(Q3-Pad1)
- Q4 pad 1: Net-(J16-Pad1) -> Net-(Q4-Pad1)
- Q5 pad 1: Net-(J23-Pad1) -> Net-(Q5-Pad1)
- R1 pad 2: Net-(D1-Pad2) -> Net-(D3-Pad2)
Routing:
- net -BattPow: track 322.6 -> 0.00 mm
- net Net-(C28-Pad1): track 12.5 -> 0.00 mm
- net Net-(D2-Pad2): track 2.73 -> 0.00 mm
Other:
- rule pad_to_mask_clearance: 0.051 -> 0

Commit message: poprawki do extra_pcb od logiki
Parts:
- added J57: LP_OUT, Connector_Molex:Molex_Mini-Fit_Jr_5566-04A_2x02_P4.20mm_Vertical, F.Cu at (256.5, 113.0)
- Q1, Q2, R2, R3: moved to F.Cu
- moved J55 217.4 mm to (63.5, 194.3)
- moved J26 181.9 mm to (226.1, 149.9)
- moved J56 162.4 mm to (231.1, 113.0), turned to 180 degrees
- moved U1 141.2 mm to (241.3, 132.1)
- moved J24 133.9 mm to (236.2, 149.9)
- moved J25 131.8 mm to (246.4, 149.9)
- moved TP5 129.8 mm to (256.5, 149.9)
- moved C14 113.3 mm to (263.5, 131.4), turned to 270 degrees
- moved J13 94.0 mm to (106.7, 147.3), turned to 0 degrees
- moved J12 74.0 mm to (116.8, 147.3), turned to 0 degrees
- moved D3 72.8 mm to (97.8, 83.8)
- moved D1 72.8 mm to (97.2, 78.7)
- moved D2 72.8 mm to (93.3, 78.7)
- moved R1 72.8 mm to (95.2, 85.7)
- moved D4 72.8 mm to (92.7, 83.8)
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