File: zasilanie/projekt/rov4/rov4.kicad_pcb (KiCad board)
At the start: 2 copper layers, 120 x 188 mm, 150 parts, among them IC1 UWE-12_10-Q12PB-C, IC2 UWE-12_10-Q12PB-C, J1 Battery digital, J10 Router, J11 Switch, J12 Enko_inkrementalny, J13 Torpedy, hall, laser, J14 Enko_absolutny_1, J15 Enko_absolutny_2, J16 RC_D_12V, J17 Xavier, J18 Kamera 1, J19 Kamera 2, J2 Reed switch, J20 Extra, J21 Extra, J22 hydrofony, J23 RC_D_15V, J24 Extra, J25 Extra, J26 Extra, J27 HP_Enable, J28 ESC1, J29 ESC2, J3 RC_D_5V, J30 ESC3, J31 ESC4, J32 ESC5, J33 ESC6, J34 ESC7, J35 ESC8, J36 Manip_sil_12v, J37 Torp_EleMagnes, J38 Extra, J39 RC_HP_12V, J4 Manip_SterSil2, J40 Extra, J41 Manip_Silnik_1, J42 Manip_Silnik_2, J43 Torpedy_serwo_7v, J44 Extra, J45 Extra, J46 Manip_serwo, J47 Extra, J48 Extra, J49 Extra, J5 Manip_SterSil1, J50 Extra, J51 Extra, J52 HP_OUT, J53 HP_IN, J54 HP_IN, J55 LP_OUT, J56 LP_IN, J57 LP_OUT, J6 Extra, J7 Extra, J8 STM32, J9 RPi, Q1 IPT004N03L, Q2 IPT004N03L, Q3 BC847A, Q4 BC847A, Q5 BC847A, Q6 IPT004N03L, Q7 IPT004N03L, Q8 IPT004N03L, Q9 IPT004N03L, U1 lm2596, U2 Transoptor, U3 Transoptor, U4 lm2596, U5 lm2596, U6 lm2596

Commit message: Moc - filtry - pcb
Parts:
- added J58: +BattPower, MountingHole:MountingHole_5.5mm_Pad, F.Cu at (-15.0, -210.0)
- added J59: -BattPower, MountingHole:MountingHole_5.5mm_Pad, F.Cu at (7.00, -210.0)
- C22: footprint Capacitor_THT:C_Radial_D12.5mm_H20.0mm_P5.00mm -> Capacitor_THT:C_Radial_D10.0mm_H20.0mm_P5.00mm
- D12, D13, D9, Q6, Q7, Q8, Q9, R10, R8, R9: moved to B.Cu
- J10, J11, J12, J13, J14, J15, J17, J18, J19, J20, J21, J24, J25, J26, J36, J37, J38, J4, J40, J41, J42, J43, J44, J45, J46, J47, J48, J49, J5, J50, J51, J6, J7, J8, J9: footprint Connector_Molex:Molex_Mini-Fit_Jr_5566-02A_2x01_P4.20mm_Vertical -> molex_3d_2pin:Molex_Mini-Fit_Jr_5566-02A_2x01_P4.20mm_Vertical
- moved C15 322.6 mm to (-170.0, -140.0), turned to 180 degrees
- moved J35 307.7 mm to (-160.0, -217.5), turned to 90 degrees
- moved C21 289.8 mm to (-137.5, -217.5), turned to 90 degrees
- moved L1 282.0 mm to (-165.0, -160.0)
- moved J29 275.9 mm to (-125.0, -137.5), turned to 90 degrees
- moved C1 271.8 mm to (76.2, 118.1)
- moved C2 271.8 mm to (76.2, 158.8)
- moved C3 271.8 mm to (76.2, 162.6)
- moved C4 271.8 mm to (76.2, 147.3)
- moved D4 271.8 mm to (50.0, 39.4)
- moved J23 271.8 mm to (58.4, 181.6)
- moved PS2 271.8 mm to (80.0, 189.2)
- moved Q5 271.8 mm to (59.4, 195.6)
- moved R14 271.8 mm to (58.4, 190.5)
- moved R2 271.8 mm to (47.3, 52.1)
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Connections:
- D11 pad 1: Net-(D10-Pad2) -> Net-(D11-Pad1)
- D11 pad 2: Net-(D11-Pad2) -> Net-(D10-Pad1)
- D12 pad 1: /moc_main/-BattPower -> Net-(D10-Pad2)
- D12 pad 2: Net-(D10-Pad1) -> Net-(D12-Pad2)
- D13 pad 1: Net-(D11-Pad2) -> Net-(D12-Pad2)
- D13 pad 2: /moc_main/-BattPower -> Net-(D11-Pad1)
- Q6 pad 2: /moc_main/-BattPower -> Net-(D10-Pad1)
- Q8 pad 2: /moc_main/-BattPower -> Net-(D10-Pad1)
- R10 pad 2: /moc_main/-BattPower -> Net-(D10-Pad1)
- R8 pad 2: Net-(D10-Pad2) -> Net-(D12-Pad2)
Routing:
- net +BattPow: track 0.00 -> 497.1 mm
- net (no net): track 0.00 -> 275.0 mm
- net -BattPow: track 0.00 -> 145.0 mm
Other:
- board size 120 x 188 mm -> 344.8 x 463.4 mm
- board text added: "logika main pcb"

Commit message: Jakieś zmainy wszystkiego
Parts:
- added J60: HP_OUT, Connector_Molex:Molex_Mini-Fit_Jr_5566-04A_2x02_P4.20mm_Vertical, F.Cu at (189.3, 185.6)
- added J61: HP_OUT, Connector_Molex:Molex_Mini-Fit_Jr_5566-04A_2x02_P4.20mm_Vertical, F.Cu at (66.9, 384.4)
- added R15: 680, Resistor_SMD:R_0805_2012Metric, B.Cu at (309.9, 57.1)
- added R16: 680, Resistor_SMD:R_0805_2012Metric, B.Cu at (322.6, 57.1)
- added REF**: MountingHole_3.2mm_M3_Pad_Via, MountingHole:MountingHole_3.2mm_M3_Pad_Via, F.Cu at (89.4, 150.2)
- added REF**: MountingHole_3.2mm_M3_Pad_Via, MountingHole:MountingHole_3.2mm_M3_Pad_Via, F.Cu at (460.0, 100.0)
- added REF**: MountingHole_3.2mm_M3_Pad_Via, MountingHole:MountingHole_3.2mm_M3_Pad_Via, F.Cu at (565.0, 100.0)
- added REF**: MountingHole_3.2mm_M3_Pad_Via, MountingHole:MountingHole_3.2mm_M3_Pad_Via, F.Cu at (565.0, 27.5)
- added REF**: MountingHole_3.2mm_M3_Pad_Via, MountingHole:MountingHole_3.2mm_M3_Pad_Via, F.Cu at (460.0, 27.5)
- added REF**: MountingHole_3.2mm_M3_Pad_Via, MountingHole:MountingHole_3.2mm_M3_Pad_Via, F.Cu at (460.0, 202.5)
- added REF**: MountingHole_3.2mm_M3_Pad_Via, MountingHole:MountingHole_3.2mm_M3_Pad_Via, F.Cu at (565.0, 202.5)
- added REF**: MountingHole_3.2mm_M3_Pad_Via, MountingHole:MountingHole_3.2mm_M3_Pad_Via, F.Cu at (198.6, 203.4)
- added REF**: MountingHole_3.2mm_M3_Pad_Via, MountingHole:MountingHole_3.2mm_M3_Pad_Via, F.Cu at (89.4, 203.4)
- added REF**: MountingHole_3.2mm_M3_Pad_Via, MountingHole:MountingHole_3.2mm_M3_Pad_Via, F.Cu at (198.6, 150.1)
- added REF**: MountingHole_3.2mm_M3_Pad, MountingHole:MountingHole_3.2mm_M3_Pad, F.Cu at (246.4, 33.0)
- added REF**: MountingHole_3.2mm_M3_Pad, MountingHole:MountingHole_3.2mm_M3_Pad, F.Cu at (246.4, 127.0)
- added REF**: MountingHole_3.2mm_M3_Pad, MountingHole:MountingHole_3.2mm_M3_Pad, F.Cu at (398.8, 127.0)
- added REF**: MountingHole_3.2mm_M3_Pad, MountingHole:MountingHole_3.2mm_M3_Pad, F.Cu at (398.8, 33.0)
- added REF**: MountingHole_3.2mm_M3_Pad, MountingHole:MountingHole_3.2mm_M3_Pad, F.Cu at (86.4, 33.0)
- added REF**: MountingHole_3.2mm_M3_Pad, MountingHole:MountingHole_3.2mm_M3_Pad, F.Cu at (86.4, 127.0)
- C23, C24, C25, C26, C27, C28, R11: moved to B.Cu
- moved J44 562.0 mm to (94.5, 193.2), turned to 180 degrees
- moved J43 543.7 mm to (119.9, 193.2), turned to 180 degrees
- moved J45 541.9 mm to (107.2, 193.2), turned to 180 degrees
- moved C29 530.6 mm to (124.1, 379.0)
- moved J49 530.6 mm to (153.5, 369.7)
- moved J50 530.6 mm to (115.5, 380.8)
- moved J51 530.6 mm to (153.5, 357.6)
- moved J54 530.6 mm to (104.9, 380.8)
- moved TP9 530.6 mm to (120.6, 379.8)
- moved U6 530.6 mm to (126.0, 366.4)
- moved J48 526.7 mm to (94.5, 160.2)
- moved J46 523.9 mm to (107.2, 160.2)
- moved TP7 517.7 mm to (119.9, 200.8), turned to 180 degrees
- moved TP8 517.4 mm to (119.9, 152.6), turned to 180 degrees
- moved U4 512.8 mm to (154.2, 190.7), turned to 180 degrees
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Connections:
- U2 pad 1: Net-(J27-Pad1) -> Net-(R15-Pad1)
- U3 pad 1: Net-(J39-Pad1) -> Net-(R16-Pad1)
Routing:
- net +BattPow: track 497.1 -> 807.1 mm
- net (no net): track 275.0 -> 0.00 mm
- net -BattPow: track 145.0 -> 0.00 mm
Other:
- board size 344.8 x 463.4 mm -> 493.8 x 191 mm

Commit message: prawie  gotowe xdd
Parts:
- removed C14, C29: 100nF, Capacitor_SMD:C_0805_2012Metric
- removed J24, J25, J26, J49, J50, J51: Extra, molex_3d_2pin:Molex_Mini-Fit_Jr_5566-02A_2x01_P4.20mm_Vertical
- removed J54: HP_IN, Connector_Molex:Molex_Mini-Fit_Jr_5566-04A_2x02_P4.20mm_Vertical
- removed J56: LP_IN, Connector_Molex:Molex_Mini-Fit_Jr_5566-04A_2x02_P4.20mm_Vertical
- removed J57: LP_OUT, Connector_Molex:Molex_Mini-Fit_Jr_5566-04A_2x02_P4.20mm_Vertical
- removed J61: HP_OUT, Connector_Molex:Molex_Mini-Fit_Jr_5566-04A_2x02_P4.20mm_Vertical
- removed the REF** at (89.4, 150.2)
- removed the REF** at (460.0, 100.0)
- removed the REF** at (565.0, 100.0)
- removed the REF** at (565.0, 27.5)
- removed the REF** at (460.0, 27.5)
- removed the REF** at (460.0, 202.5)
- removed the REF** at (565.0, 202.5)
- removed the REF** at (198.6, 203.4)
- removed the REF** at (89.4, 203.4)
- removed the REF** at (198.6, 150.1)
- removed the REF** at (246.4, 33.0)
- removed the REF** at (246.4, 127.0)
- removed the REF** at (398.8, 127.0)
- removed the REF** at (398.8, 33.0)
- removed the REF** at (86.4, 33.0)
- removed the REF** at (86.4, 127.0)
- removed TP5, TP9: EXTRA, Connector_PinHeader_2.54mm:PinHeader_1x01_P2.54mm_Vertical
- removed U1, U6: lm2596, lm2596:lm2596-44_8mm_x_23mm
- added D15: D_TVS, Diode_SMD:D_SMB, B.Cu at (442.9, 44.9)
- added D16: D_TVS, Diode_SMD:D_SMB, B.Cu at (483.4, 32.0)
- added D17: D_TVS, Diode_SMD:D_SMB, B.Cu at (233.5, 50.2)
- added D18: D_TVS, Diode_SMD:D_SMB, B.Cu at (234.5, 77.3)
- added J62: bus_bar, MountingHole:MountingHole_3.2mm_M3_Pad, F.Cu at (30.0, 68.1)
- added J63: bus_bar, MountingHole:MountingHole_3.2mm_M3_Pad, F.Cu at (136.7, 68.1)
- added J64: bus_bar, MountingHole:MountingHole_3.2mm_M3_Pad, F.Cu at (65.5, 68.1)
- added J65: bus_bar, MountingHole:MountingHole_3.2mm_M3_Pad, F.Cu at (101.1, 68.1)
- added J66: bus_bar, MountingHole:MountingHole_3.2mm_M3_Pad, F.Cu at (197.6, 54.1)
- added J67: bus_bar, MountingHole:MountingHole_3.2mm_M3_Pad, F.Cu at (197.6, 68.1)
- added J68: bus_bar_bott, MountingHole:MountingHole_3.2mm_M3_Pad, F.Cu at (136.7, 47.8)
- added J69: bus_bar_bott, MountingHole:MountingHole_3.2mm_M3_Pad, F.Cu at (172.2, 88.4)
- added J70: bus_bar_bott, MountingHole:MountingHole_3.2mm_M3_Pad, F.Cu at (101.1, 88.4)
- added J71: bus_bar_bott, MountingHole:MountingHole_3.2mm_M3_Pad, F.Cu at (224.3, 88.4)
- added J72: bus_bar_bott, MountingHole:MountingHole_3.2mm_M3_Pad, F.Cu at (137.9, 88.4)
- added J73: bus_bar_bott, MountingHole:MountingHole_3.2mm_M3_Pad, F.Cu at (65.5, 47.8)
- added J74: bus_bar_bott, MountingHole:MountingHole_3.2mm_M3_Pad, F.Cu at (172.2, 47.8)
- added J75: bus_bar_bott, MountingHole:MountingHole_3.2mm_M3_Pad, F.Cu at (65.5, 88.4)
- added J76: bus_bar_bott, MountingHole:MountingHole_3.2mm_M3_Pad, F.Cu at (30.0, 47.8)
- added J77: bus_bar_bott, MountingHole:MountingHole_3.2mm_M3_Pad, F.Cu at (101.1, 47.8)
- added J78: bus_bar_bott, MountingHole:MountingHole_3.2mm_M3_Pad, F.Cu at (30.0, 88.4)
- added R17: 100, Resistor_SMD:R_0805_2012Metric, B.Cu at (468.5, 29.5)
- added R18: 100, Resistor_SMD:R_0805_2012Metric, B.Cu at (202.7, 75.7)
- added REF**: MountingHole_3.2mm_M3_Pad, MountingHole:MountingHole_3.2mm_M3_Pad, F.Cu at (125.8, 255.7)
- added REF**: MountingHole_3.2mm_M3_Pad, MountingHole:MountingHole_3.2mm_M3_Pad, F.Cu at (187.5, 20.4)
- added REF**: MountingHole_3.2mm_M3_Pad, MountingHole:MountingHole_3.2mm_M3_Pad, F.Cu at (187.5, 118.2)
- added REF**: MountingHole_3.2mm_M3_Pad, MountingHole:MountingHole_3.2mm_M3_Pad, F.Cu at (399.9, 21.4)
- added REF**: MountingHole_3.2mm_M3_Pad, MountingHole:MountingHole_3.2mm_M3_Pad, F.Cu at (514.9, 21.4)
- added REF**: MountingHole_3.2mm_M3_Pad, MountingHole:MountingHole_3.2mm_M3_Pad, F.Cu at (399.9, 122.9)
- added REF**: MountingHole_3.2mm_M3_Pad, MountingHole:MountingHole_3.2mm_M3_Pad, F.Cu at (514.9, 83.9)
- added REF**: MountingHole_3.2mm_M3_Pad, MountingHole:MountingHole_3.2mm_M3_Pad, F.Cu at (514.9, 194.9)
- added REF**: MountingHole_3.2mm_M3_Pad, MountingHole:MountingHole_3.2mm_M3_Pad, F.Cu at (399.9, 194.9)
- added REF**: MountingHole_3.2mm_M3_Pad, MountingHole:MountingHole_3.2mm_M3_Pad, F.Cu at (125.8, 314.1)
- added REF**: MountingHole_3.2mm_M3_Pad, MountingHole:MountingHole_3.2mm_M3_Pad, F.Cu at (11.5, 314.1)
- added REF**: MountingHole_3.2mm_M3_Pad, MountingHole:MountingHole_3.2mm_M3_Pad, F.Cu at (11.5, 255.7)
- added REF**: MountingHole_3.2mm_M3_Pad, MountingHole:MountingHole_3.2mm_M3_Pad, F.Cu at (514.9, 158.9)
- added REF**: MountingHole_3.2mm_M3_Pad, MountingHole:MountingHole_3.2mm_M3_Pad, F.Cu at (305.6, 118.2)
- added REF**: MountingHole_3.2mm_M3_Pad, MountingHole:MountingHole_3.2mm_M3_Pad, F.Cu at (305.6, 20.4)
- added REF**: MountingHole_3.2mm_M3_Pad, MountingHole:MountingHole_3.2mm_M3_Pad, F.Cu at (20.4, 20.4)
- added REF**: MountingHole_3.2mm_M3_Pad, MountingHole:MountingHole_3.2mm_M3_Pad, F.Cu at (20.4, 118.2)
- J2: value Reed switch -> Digital power: ON-OFF
- J27: value HP_Enable -> High power: ON-OFF
- J36: value Manip_sil_12v -> Extra
- J40: value Extra -> Manip_Silnik_3
- Q3, R12, R4: moved to B.Cu
- R11: moved to F.Cu
- moved J3 146.5 mm to (400.4, 105.4), turned to 270 degrees
- moved C28 136.0 mm to (62.3, 277.6)
- moved C27 135.7 mm to (62.3, 305.2)
- moved J53 134.9 mm to (115.3, 277.6), turned to 90 degrees
- moved J16 133.7 mm to (400.4, 71.9), turned to 270 degrees
- moved J60 133.2 mm to (115.3, 296.3), turned to 90 degrees
- moved U5 131.9 mm to (79.4, 270.9)
- moved J43 131.7 mm to (45.1, 301.6)
- moved J44 131.7 mm to (19.7, 301.6)
- moved J45 131.7 mm to (32.4, 301.6)
- moved J46 131.7 mm to (32.4, 268.6)
- moved J47 131.7 mm to (45.1, 268.6)
- moved J48 131.7 mm to (19.7, 268.6)
- moved TP7 131.7 mm to (45.1, 309.2)
- moved TP8 131.7 mm to (45.1, 260.9)
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Connections:
- J10 pad 2: Net-(J10-Pad2) -> -BattDigit
- J22 pad 1: Net-(C10-Pad1) -> Net-(C12-Pad2)
- J22 pad 2: Net-(C12-Pad2) -> Net-(C10-Pad1)
- J5 pad 2: Net-(J10-Pad2) -> -BattDigit
- Q2 pad 1: +BattDigit -> Net-(D16-Pad1)
- Q7 pad 1: +BattPow -> Net-(D18-Pad1)
- Q9 pad 1: +BattPow -> Net-(D18-Pad1)
Routing:
- net +BattPow: track 807.1 -> 34.4 mm, vias 0 -> 1
- net -BattPow: track 0.00 -> 391.4 mm, vias 0 -> 1
- net Net-(IC2-Pad2): track 0.00 -> 81.3 mm
- net Net-(D10-Pad1): track 0.00 -> 69.1 mm
- net +BattDigit: track 0.00 -> 44.3 mm, vias 0 -> 1
- net Net-(Q6-Pad3): track 0.00 -> 43.2 mm
- net Net-(D17-Pad1): track 0.00 -> 39.5 mm
- net Net-(D18-Pad1): track 0.00 -> 38.6 mm
- net /logika_main/-Batt: track 0.00 -> 31.6 mm
- net Net-(C24-Pad1): track 0.00 -> 30.0 mm
- net Net-(C6-Pad1): track 0.00 -> 24.5 mm
- net Net-(C2-Pad1): track 0.00 -> 24.3 mm
- net Net-(D15-Pad1): track 0.00 -> 23.3 mm
- net Net-(J23-Pad1): track 0.00 -> 21.9 mm
- net Net-(D16-Pad1): track 0.00 -> 15.8 mm
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- added copper zone on F.Cu, net +BattDigit
- added copper zone on F.Cu, net +BattPow
- added copper zone on B.Cu, net -BattDigit
- added copper zone on B.Cu, net -BattPow
- added copper zone on B.Cu, net /logika_main/-Batt
- added copper zone on F.Cu, net Net-(C10-Pad1)
- added copper zone on F.Cu, net Net-(C12-Pad2)
- added copper zone on F.Cu, net Net-(C15-Pad1)
- added copper zone on F.Cu, net Net-(C16-Pad1)
- added copper zone on F.Cu, net Net-(C17-Pad1)
- added copper zone on F.Cu, net Net-(C18-Pad1)
- added copper zone on F.Cu, net Net-(C19-Pad1)
- added copper zone on F.Cu, net Net-(C2-Pad1)
- added copper zone on F.Cu, net Net-(C20-Pad1)
- added copper zone on F.Cu, net Net-(C21-Pad1)
- added copper zone on F.Cu, net Net-(C22-Pad1)
- added copper zone on F.Cu, net Net-(C24-Pad1)
- added copper zone on F.Cu, net Net-(C27-Pad1)
- added copper zone on B.Cu, net Net-(C27-Pad2)
- added copper zone on F.Cu, net Net-(C28-Pad1)
- added copper zone on F.Cu, net Net-(C6-Pad1)
- added copper zone on B.Cu, net Net-(D10-Pad1)
- added copper zone on F.Cu, net Net-(J53-Pad1)
- added copper zone on B.Cu, net Net-(Q6-Pad3)
Other:
- board size 493.8 x 191 mm -> 513.5 x 304.4 mm
- rule via_min_size: 0.4 -> 0.5
- board text added: "+15V"
- board text added: "+15V OK"
- board text added: "-15V"
- board text added: "-15V OK"
- board text added: "12V OK"
- board text added: "5V OK"
- board text added: "COM"
- board text added: "Digital power output"
- board text added: "HP +"
- board text added: "HP -"
- board text added: "High power output"
- board text added: "Polaryzacja: zielone - ok czerwone - odwrotnie"
- board text added: "RC: +/-15V"
- board text added: "RC: 12V"
- board text added: "RC: 5V"
- board text removed: "logika main pcb"

Commit message: Ostatnie poprawki xd
Parts:
- added D19: D_TVS, Diode_SMD:D_SMB, F.Cu at (457.6, 48.0)
- added D20: D_TVS, Diode_SMD:D_SMB, F.Cu at (468.5, 48.0)
- added D21: D_TVS, Diode_SMD:D_SMB, F.Cu at (234.5, 58.2)
- added D22: D_TVS, Diode_SMD:D_SMB, F.Cu at (234.5, 67.2)
- added J79: BatDig_Sens, Connector_Molex:Molex_SPOX_5267-02A_1x02_P2.50mm_Vertical, F.Cu at (421.9, 21.8)
- added J80: BatPow_Sens, Connector_Molex:Molex_SPOX_5267-02A_1x02_P2.50mm_Vertical, F.Cu at (224.3, 23.6)
- J39: value RC_HP_12V -> RC: 12V
- moved D10 15.2 mm to (199.2, 22.4)
- moved D11 15.2 mm to (206.2, 22.4)
- moved D12 15.2 mm to (197.6, 24.9)
- moved D13 15.2 mm to (207.8, 24.9)
- moved R8 15.2 mm to (197.6, 27.4)
Routing:
- net -BattPow: track 391.4 -> 14.2 mm, vias 1 -> 2
- net /logika_main/-Batt: track 31.6 -> 67.6 mm, vias 0 -> 2
- net Net-(D10-Pad1): track 69.1 -> 104.6 mm, vias 0 -> 2
- net Net-(D19-Pad1): track 8.91 -> 25.4 mm, vias 0 -> 1
- net Net-(D21-Pad1): track 43.2 -> 58.1 mm, vias 0 -> 1
- net +BattPow: track 34.4 -> 26.4 mm
- net -BattDigit: track 7.76 -> 10.6 mm, vias 4 -> 5

Commit message: Fix + bus bary projekt
Parts:
- D19, D20: moved to B.Cu
Routing:
- net -BattDigit: track 10.6 -> 0.00 mm, vias 5 -> 4
- net Net-(D10-Pad1): track 104.6 -> 94.6 mm
- net -BattPow: track 14.2 -> 10.1 mm
- net +BattPow: track 26.4 -> 23.5 mm
- net Net-(D2-Pad1): track 3.76 -> 1.80 mm
- net Net-(D1-Pad2): track 3.45 -> 1.80 mm
- net Net-(D11-Pad1): track 4.67 -> 3.54 mm
- net Net-(D10-Pad2): track 4.67 -> 3.54 mm
- net Net-(D6-Pad2): track 6.29 -> 5.38 mm
- net /logika_main/-Batt: track 67.6 -> 67.5 mm, vias 2 -> 3
- net Net-(D19-Pad1): vias 1 -> 0
