File: zasilanie/projekt/rov4/kopia_pcb2.kicad_pcb (KiCad board)
At the start: 2 copper layers, 493.8 x 190.8 mm, 180 parts, among them IC1 UWE-12_10-Q12PB-C, IC2 UWE-12_10-Q12PB-C, J1 Battery digital, J10 Router, J11 Switch, J12 Enko_inkrementalny, J13 Torpedy, hall, laser, J14 Enko_absolutny_1, J15 Enko_absolutny_2, J16 RC_D_12V, J17 Xavier, J18 Kamera 1, J19 Kamera 2, J2 Digital power: ON-OFF, J20 Extra, J21 Extra, J22 hydrofony, J23 RC_D_15V, J27 High power: ON-OFF, J28 ESC1, J29 ESC2, J3 RC_D_5V, J30 ESC3, J31 ESC4, J32 ESC5, J33 ESC6, J34 ESC7, J35 ESC8, J36 Extra, J37 Torp_EleMagnes, J38 Extra, J39 RC_HP_12V, J4 Manip_SterSil2, J40 Manip_Silnik_3, J41 Manip_Silnik_1, J42 Manip_Silnik_2, J43 Torpedy_serwo_7v, J44 Extra, J45 Extra, J46 Manip_serwo, J47 Extra, J48 Extra, J5 Manip_SterSil1, J52 HP_OUT, J53 HP_IN, J55 LP_OUT, J58 +BattPower, J59 -BattPower, J6 Extra, J60 HP_OUT, J62 bus_bar, J63 bus_bar, J64 bus_bar, J65 bus_bar, J66 bus_bar, J67 bus_bar, J68 bus_bar_bott, J69 bus_bar_bott, J7 Extra, J70 bus_bar_bott, J71 bus_bar_bott, J72 bus_bar_bott, J73 bus_bar_bott, J74 bus_bar_bott, J75 bus_bar_bott, J76 bus_bar_bott, J77 bus_bar_bott, J78 bus_bar_bott, J8 STM32, J9 RPi, Q1 IPT004N03L, Q2 IPT004N03L, Q3 BC847A, Q4 BC847A, Q5 BC847A, Q6 IPT004N03L, Q7 IPT004N03L, Q8 IPT004N03L, Q9 IPT004N03L, U2 Transoptor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

Commit message: prawie  gotowe xdd
Changed lines of the file:
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@@
   (general
     (thickness 1.6)
-    (drawings 31)
+    (drawings 30)
     (tracks 215)
     (zones 0)
@@
   )
   (setup
-    (last_trace_width 0.25)
+    (last_trace_width 2)
     (user_trace_width 0.5)
     (user_trace_width 1)
@@
     )
   )
-  (gr_text "Polaryzacja: \nzielone - ok\nczerwone - odwrotnie" (at 490 27) (layer F.SilkS)
-    (effects (font (size 1 1) (thickness 0.2)))
-  )
   (gr_text "Polaryzacja: \nzielone - ok\nczerwone - odwrotnie" (at 282 29) (layer F.SilkS)
     (effects (font (size 1 1) (thickness 0.2)))
@@
   (segment (start 271.78 38.1) (end 261.62 48.26) (width 0.5) (layer B.Cu) (net 16))
   (segment (start 275.9225 38.1) (end 271.78 38.1) (width 0.5) (layer B.Cu) (net 16))
+  (segment (start 279.79 84.7) (end 279.79 86.53) (width 1) (layer B.Cu) (net 58))
+  (segment (start 280.67 83.82) (end 279.79 84.7) (width 1) (layer B.Cu) (net 58))
+  (segment (start 291.465 83.82) (end 280.67 83.82) (width 1) (layer B.Cu) (net 58))
+  (segment (start 292.49 86.53) (end 292.49 84.845) (width 1) (layer B.Cu) (net 58))
+  (segment (start 292.49 84.845) (end 291.465 83.82) (width 1) (layer B.Cu) (net 58))
   (segment (start 312.16 121.66) (end 312.42 121.92) (width 4) (layer B.Cu) (net 16))
   (segment (start 312.16 113.03) (end 312.16 121.66) (width 4) (layer B.Cu) (net 16))
@@
   (segment (start 479 188.95) (end 486.77 188.95) (width 1) (layer F.Cu) (net 43))
   (segment (start 520.13 41.639196) (end 511.22 41.639196) (width 10) (layer B.Cu) (net 44))
+  (segment (start 284.09 61.985) (end 284.09 60.3) (width 1) (layer B.Cu) (net 57))
+  (segment (start 283.21 62.865) (end 284.09 61.985) (width 1) (layer B.Cu) (net 57))
+  (segment (start 272.094998 62.865) (end 283.21 62.865) (width 1) (layer B.Cu) (net 57))
+  (segment (start 271.39 60.3) (end 271.39 62.160002) (width 1) (layer B.Cu) (net 57))
+  (segment (start 271.39 62.160002) (end 272.094998 62.865) (width 1) (layer B.Cu) (net 57))
   (segment (start 275.59 78.26) (end 275.59 69.35) (width 6) (layer B.Cu) (net 45))
   (segment (start 288.29 78.26) (end 288.29 69.35) (width 6) (layer B.Cu) (net 45))
@@
   (segment (start 528.18 37.439196) (end 527.570804 36.83) (width 1) (layer B.Cu) (net 56))
   (segment (start 527.570804 36.83) (end 523.760804 33.02) (width 1) (layer B.Cu) (net 56))
-  (segment (start 284.09 61.985) (end 284.09 60.3) (width 1) (layer B.Cu) (net 57))
-  (segment (start 283.21 62.865) (end 284.09 61.985) (width 1) (layer B.Cu) (net 57))
-  (segment (start 272.094998 62.865) (end 283.21 62.865) (width 1) (layer B.Cu) (net 57))
-  (segment (start 271.39 60.3) (end 271.39 62.160002) (width 1) (layer B.Cu) (net 57))
-  (segment (start 271.39 62.160002) (end 272.094998 62.865) (width 1) (layer B.Cu) (net 57))
   (segment (start 301.5 59.875) (end 304.9375 59.875) (width 1) (layer B.Cu) (net 57))
   (segment (start 284.09 61.985) (end 284.09 62.09) (width 1) (layer B.Cu) (net 57))
@@
   (segment (start 298.375 63) (end 301.5 59.875) (width 1) (layer B.Cu) (net 57))
   (segment (start 297.5 63) (end 298.375 63) (width 1) (layer B.Cu) (net 57))
-  (segment (start 279.79 84.7) (end 279.79 86.53) (width 1) (layer B.Cu) (net 58))
-  (segment (start 280.67 83.82) (end 279.79 84.7) (width 1) (layer B.Cu) (net 58))
-  (segment (start 291.465 83.82) (end 280.67 83.82) (width 1) (layer B.Cu) (net 58))
-  (segment (start 292.49 86.53) (end 292.49 84.845) (width 1) (layer B.Cu) (net 58))
-  (segment (start 292.49 84.845) (end 291.465 83.82) (width 1) (layer B.Cu) (net 58))
   (segment (start 267.6375 85.4225) (end 267.6375 86.36) (width 1) (layer B.Cu) (net 58))
   (segment (start 269.24 83.82) (end 267.6375 85.4225) (width 1) (layer B.Cu) (net 58))
