File: zasilanie/projekt/rov4/rov4.sch (KiCad schematic (older format))
At the start: 68 parts, among them IC1 UWE-12_10-Q12PB-C, J1 Battery digital, J10 Switch, J11 Kamera 1, J12 Extra, J13 Kamera 2, J14 Extra, J15 Extra, J16 Extra, J17 BatteryPower, J18 RPi_PowerEnable, J2 Reed switch, J20 Manip_SterSil1, J21 Manip_SterSil2, J24 RC_D_15V, J27 RC_D_5V, J3 Extra, J4 Extra, J45 RC_D_12V, J5 Extra, J6 RPi, J7 Router, J8 Xavier, J9 Hydrofony, Q1 IRFZ44N, Q2 Q_NPN_BCE, Q3 Q_NPN_BCE, Q4 Q_NPN_BCE, U1 HFV7A_012ZST, U2 XL4015

Commit message: Modyfikacje schematu i PCB
Parts:
- removed C1, C2, C3: 33uF, Capacitor_SMD:C_2816_7142Metric_Pad3.20x4.45mm_HandSolder, symbol Device:C_Small
- removed C6: 1uF, Capacitor_SMD:C_0805_2012Metric_Pad1.15x1.40mm_HandSolder, symbol Device:C
- removed C8: 10uF, Capacitor_SMD:C_0805_2012Metric_Pad1.15x1.40mm_HandSolder, symbol Device:C
- removed C9: 5000uF, Capacitor_SMD:C_Elec_8x10.2, symbol Device:C
- removed D3: LED_B, LED_SMD:LED_0805_2012Metric_Pad1.15x1.40mm_HandSolder, symbol Device:LED
- removed F1: 2-5A slow, symbol Device:Fuse
- removed F2: 20A_fast, symbol Device:Fuse
- removed F3: 10A_slow, symbol Device:Fuse
- removed J18: RPi_PowerEnable, Connector_PinHeader_2.54mm:PinHeader_1x01_P2.54mm_Vertical, symbol Connector_Generic:Conn_01x01
- removed Q2, Q3, Q4: Q_NPN_BCE, Package_TO_SOT_SMD:SOT-23_Handsoldering, symbol Device:Q_NPN_BCE
- removed R3: 3k, Resistor_SMD:R_0805_2012Metric_Pad1.15x1.40mm_HandSolder, symbol Device:R
- added C1, C2, C3: 33uF, Capacitor_SMD:CP_Elec_6.3x5.4, symbol Device:CP_Small
- added C19, C23, C6: 100nF, Capacitor_SMD:C_0805_2012Metric, symbol Device:C_Small
- added C20, C22: 200uF, Capacitor_SMD:CP_Elec_8x10, symbol Device:CP_Small
- added C21: 10uF, Capacitor_SMD:C_0805_2012Metric, symbol Device:C_Small
- added C8, C9: 100uF, Capacitor_SMD:CP_Elec_6.3x7.7, symbol Device:CP_Small
- added Q2, Q3, Q4: BC847A, Package_TO_SOT_SMD:SOT-23, symbol Device:Q_NPN_BEC
- C4: value 1uF -> 100nF; footprint Capacitor_SMD:C_0805_2012Metric_Pad1.15x1.40mm_HandSolder -> Capacitor_SMD:C_0805_2012Metric
- C5: footprint Capacitor_SMD:C_0805_2012Metric_Pad1.15x1.40mm_HandSolder -> Capacitor_SMD:C_0805_2012Metric
- C7: value 5000uF -> 100nF; footprint Capacitor_SMD:C_Elec_8x10.2 -> Capacitor_SMD:C_0805_2012Metric
- D1, D2: footprint Diode_SMD:D_SMA_Handsoldering -> Diode_SMD:D_SMA
- D10, D4, D5, D6, D7, D8: footprint LED_SMD:LED_0805_2012Metric_Pad1.15x1.40mm_HandSolder -> LED_SMD:LED_0805_2012Metric
- D11, D9: footprint Diode_SMD:D_MiniMELF_Handsoldering -> Diode_SMD:D_MiniMELF
- J9: footprint Connector_PinHeader_2.54mm:PinHeader_1x02_P2.54mm_Vertical -> Connector_PinHeader_2.54mm:PinHeader_1x03_P2.54mm_Vertical
- Q1: footprint Package_TO_SOT_SMD:SOT-23_Handsoldering -> Package_TO_SOT_SMD:SOT-23
- R1, R2, R4, R5, R6, R7, R8: footprint Resistor_SMD:R_0805_2012Metric_Pad1.15x1.40mm_HandSolder -> Resistor_SMD:R_0805_2012Metric
- TP1, TP3: value TestPoint -> D_5V
- TP2: value TestPoint -> D_-5V
- TP4: value TestPoint -> D_12V
- TP5: value TestPoint -> EXTRA
Connections:
- net +BattDigit: now also IC1.1 (+VIN), PS1.1 (+VIN), PS2.22 (+VIN_1), PS2.23 (+VIN_2), C1.1, C2.1, C3.1
- net GND: now also C7.1, C1.2, C19.2, C2.2, C20.2, C21.2, C22.2, C23.2, C3.2, C6.2, C8.2, C9.1, Q2.2 (E), Q3.2 (E), Q4.2 (E); no longer C7.2
- net at PS2.1 (R.C.): now also Q2.3 (C)
- net at J9.3 (Pin_3), PS2.11 (-VOUT), R5.1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: now also C7.2, C9.2
- net at J9.1 (Pin_1), PS2.14 (+VOUT), R4.2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: now also C6.1, C8.1
- net at IC1.2 (ON/OFF_CONTROL): now also Q3.3 (C)
- net at IC1.7 (+SENSE), IC1.8 (+VOUT), J11.1 (Pin_1)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: now also C19.1, C21.1, C22.1
- net at PS1.3 (CTRL): now also Q4.3 (C)
- net at C4.1, C5.1, J10.1 (Pin_1)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: now also C20.1; no longer C7.1
- net at J3.1 (Pin_1), J4.1 (Pin_1), J5.1 (Pin_1)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: now also C23.1
- net at J45.1 (Pin_1): now also Q3.1 (B)
- net at J27.1 (Pin_1): now also Q4.1 (B)
- net at J24.1 (Pin_1): now also Q2.1 (B)
Other:
- moved on the sheet: D4, D5, J24, J27, J45, J9, R4, R5, TP1, TP2

Commit message: Update
Parts:
- removed D1, D2: SS34, Diode_SMD:D_SMA, symbol Device:D_Schottky
- removed D10, D8: LED_B, LED_SMD:LED_0805_2012Metric, symbol Device:LED_Small
- removed D11, D9: BAT48, Diode_SMD:D_MiniMELF, symbol Device:D_Schottky_Small
- removed Q1: IRFZ44N, Package_TO_SOT_SMD:SOT-23, symbol Device:Q_NMOS_GDS
- removed R8: 3k, Resistor_SMD:R_0805_2012Metric, symbol Device:R_Small
- removed U1: HFV7A_012ZST, Custom Relay:HFV7A_012ZST, symbol hfv7a_012zst:HFV7A_012ZST
- removed U2: XL4015, XL4015:xl4015, symbol XL4015:XL4015
- added D1: LED_G, LED_SMD:LED_0805_2012Metric, symbol Device:LED
- added D2: LED_R, LED_SMD:LED_0805_2012Metric, symbol Device:LED
- added D3, D4: BAT48, Diode_SMD:D_MiniMELF, symbol Device:D_Schottky
- added J47: Enko_inkrementalny, Connector_PinHeader_2.54mm:PinHeader_1x02_P2.54mm_Vertical, symbol Connector_Generic:Conn_01x02
- added J48: Torpedy, hall, laser, Connector_PinHeader_2.54mm:PinHeader_1x02_P2.54mm_Vertical, symbol Connector_Generic:Conn_01x02
- added J49: Enko_absolutny_1, Connector_PinHeader_2.54mm:PinHeader_1x02_P2.54mm_Vertical, symbol Connector_Generic:Conn_01x02
- added J50: Enko_absolutny_2, Connector_PinHeader_2.54mm:PinHeader_1x02_P2.54mm_Vertical, symbol Connector_Generic:Conn_01x02
- added Q1, Q2: IPT004N03L, Package_TO_SOT_SMD:Infineon_PG-HSOF-8-1, symbol Device:Q_NMOS_GSD
- added R3: 10k, Resistor_SMD:R_0805_2012Metric, symbol Device:R
- added U1: lm2596, lm2596:lm2596-44_8mm_x_23mm, symbol lm2596:lm2596
- J1: value Battery digital -> Reed switch
- J2: value Reed switch -> Battery digital; footprint Connector_PinHeader_2.54mm:PinHeader_1x02_P2.54mm_Vertical -> Connector_PinSocket_2.54mm:PinSocket_2x01_P2.54mm_Vertical
- R1: value 1k -> 3k
- R2: value 100k -> 100
- renumbered C2 to C1, C6 to C10, C8 to C11, C1 to C12, C7 to C13, C9 to C14, C4 to C2, C5 to C3, C20 to C4, C3 to C5, C19 to C6, C21 to C7, C22 to C8, C23 to C9, D6 to D5, D7 to D6, D4 to D7, D5 to D8, J17 to J11, J45 to J12, J8 to J13, J11 to J14, J13 to J15, J15 to J16, J16 to J17, J9 to J18, J3 to J19, J4 to J20, J5 to J21, J24 to J22, J21 to J3, J20 to J4, J14 to J5, J12 to J6, J27 to J7, J6 to J8, J7 to J9, Q4 to Q3, Q3 to Q4, Q2 to Q5, R6 to R4, R7 to R5, R4 to R6, R5 to R7, TP3 to TP1, TP4 to TP2, TP5 to TP3, TP1 to TP4, TP2 to TP5
Connections:
- net +BattDigit: now also J1.2 (Pin_2), J2.1 (Pin_1), R1.1, Q2.1 (G), U1.1 (Vin)
- net at C6.1, C7.1, C8.1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: now also J49.1 (Pin_1), J50.1 (Pin_1)
- net at C2.1, C3.1, C4.1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: now also D5.2 (A), J47.1 (Pin_1), J48.2 (Pin_2); no longer R4.2
- net at R2.1: now also J1.1 (Pin_1); no longer R1.1
- net at R1.2: now also D1.2 (A), D2.1 (K); no longer J2.2 (Pin_2)
- net at C9.1, J19.1 (Pin_1), J20.1 (Pin_1)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: now also U1.3 (Vout)
- net at R4.1: now also D5.1 (K); no longer D5.2 (A)
- removed net +Batt: J1.1 (Pin_1), J2.1 (Pin_1)
- net GND renamed -BattDigit
- net -BattDigit: now also R4.2, J47.2 (Pin_2), J48.1 (Pin_1), J49.2 (Pin_2), J50.2 (Pin_2), Q2.2 (S), U1.2 (GND), U1.4 (GND); no longer D5.1 (K), J1.2 (Pin_2), R2.2
- new net: Q1.1 (G), R2.2, R3.1
- new net: Q1.3 (D), Q2.3 (D)
- new net: D1.1 (K), D3.2 (A)
- new net: D2.2 (A), D4.1 (K)
- new net -Batt: D3.1 (K), D4.2 (A), J2.2 (Pin_2), Q1.2 (S), R3.2
- no-connect marks 3 -> 2
Other:
- note added: "+/-15v:\n> in max 2 A,\n> fuse: 3-4-5A ?,\n> out min: +/- 0.04A\n> out max: +/- 0.8A\n\n-Hydrofony\n"
- note removed: "+/-15v:\n> in max 2 A,\n> fuse: 2A ?,\n> out min: +/- 0.04A\n> out max: +/- 0.8A\n\n-Hydrofony\n"
- moved on the sheet: C10, C11, C12, C13, C14, C9, D5, D7, D8, J11, J18, J19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

Commit message: sync
Parts:
- added J37: STM32, Connector_PinHeader_2.54mm:PinHeader_1x02_P2.54mm_Vertical, symbol Connector_Generic:Conn_01x02
- J19: footprint Connector_PinHeader_2.54mm:PinHeader_1x02_P2.54mm_Vertical -> Connector_Molex:Molex_SPOX_5267-02A_1x02_P2.50mm_Vertical
- J20: footprint Connector_PinHeader_2.54mm:PinHeader_1x02_P2.54mm_Vertical -> Connector_Molex:Molex_Mini-Fit_Jr_5566-02A_2x01_P4.20mm_Vertical
Connections:
- net -BattDigit: now also J37.2 (Pin_2)
- net at C2.1, C3.1, C4.1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: now also J37.1 (Pin_1)
Changed lines of the file:
@@
 F 0 "J20" V 9650 6300 50  0000 R CNN
 F 1 "Extra" V 9850 6500 50  0000 R CNN
-F 2 "Connector_PinHeader_2.54mm:PinHeader_1x02_P2.54mm_Vertical" H 9750 6450 50  0001 C CNN
+F 2 "Connector_Molex:Molex_Mini-Fit_Jr_5566-02A_2x01_P4.20mm_Vertical" H 9750 6450 50  0001 C CNN
 F 3 "~" H 9750 6450 50  0001 C CNN
 	1    9750 6450
@@
 F 0 "J19" V 9250 6300 50  0000 R CNN
 F 1 "Extra" V 9450 6500 50  0000 R CNN
-F 2 "Connector_PinHeader_2.54mm:PinHeader_1x02_P2.54mm_Vertical" H 9350 6450 50  0001 C CNN
+F 2 "Connector_Molex:Molex_SPOX_5267-02A_1x02_P2.50mm_Vertical" H 9350 6450 50  0001 C CNN
 F 3 "~" H 9350 6450 50  0001 C CNN
 	1    9350 6450
@@
 	10150 2600 10150 3000
 Wire Wire Line
-	9700 2600 10150 2600
+	9700 2600 10050 2600
 Wire Wire Line
 	10250 2900 10250 3000
@@
 Wire Wire Line
 	10650 2600 10600 2600
+$Comp
+L Connector_Generic:Conn_01x02 J37
+U 1 1 5CC327BE
+P 10050 2250
+F 0 "J37" V 9950 2100 50  0000 R CNN
+F 1 "STM32" V 10150 2300 50  0000 R CNN
+F 2 "Connector_PinHeader_2.54mm:PinHeader_1x02_P2.54mm_Vertical" H 10050 2250 50  0001 C CNN
+F 3 "~" H 10050 2250 50  0001 C CNN
+	1    10050 2250
+	0    -1   -1   0
+$EndComp
+Wire Wire Line
+	10050 2450 10050 2600
+Connection ~ 10050 2600
+Wire Wire Line
+	10050 2600 10150 2600
+Wire Wire Line
+	10150 2450 10150 2500
+Wire Wire Line
+	10150 2500 10250 2500
+Wire Wire Line
+	10250 2500 10250 2900
 $EndSCHEMATC

Commit message: test2
Other:
- note added: "TO na osobnym pcb"
- moved on the sheet: C10, C11, C12, C13, C14, C9, D7, D8, J11, J18, J19, J20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

Commit message: Reorganizacja struktury projektu
Parts:
- removed C1, C12, C5: 33uF, Capacitor_SMD:CP_Elec_6.3x5.4, symbol Device:CP_Small
- removed C10, C13, C2, C6, C9: 100nF, Capacitor_SMD:C_0805_2012Metric, symbol Device:C_Small
- removed C11, C14: 100uF, Capacitor_SMD:CP_Elec_6.3x7.7, symbol Device:CP_Small
- removed C3, C7: 10uF, Capacitor_SMD:C_0805_2012Metric, symbol Device:C_Small
- removed C4, C8: 200uF, Capacitor_SMD:CP_Elec_8x10, symbol Device:CP_Small
- removed D1: LED_G, LED_SMD:LED_0805_2012Metric, symbol Device:LED
- removed D2: LED_R, LED_SMD:LED_0805_2012Metric, symbol Device:LED
- removed D3, D4: BAT48, Diode_SMD:D_MiniMELF, symbol Device:D_Schottky
- removed D5, D6, D7, D8: LED_B, LED_SMD:LED_0805_2012Metric, symbol Device:LED
- removed IC1: UWE-12_10-Q12PB-C, UWE-12_10-Q12P-C:UWE-12_10-Q12P-C, symbol UWE-12_10-Q12P-C:UWE-12_10-Q12PB-C
- removed J1: Reed switch, Connector_PinHeader_2.54mm:PinHeader_1x02_P2.54mm_Vertical, symbol Connector_Generic:Conn_01x02
- removed J10: Switch, Connector_PinHeader_2.54mm:PinHeader_1x02_P2.54mm_Vertical, symbol Connector_Generic:Conn_01x02
- removed J11: BatteryPower, Connector_PinHeader_2.54mm:PinHeader_1x02_P2.54mm_Vertical, symbol Connector_Generic:Conn_01x02
- removed J12: RC_D_12V, Connector_PinHeader_2.54mm:PinHeader_1x01_P2.54mm_Vertical, symbol Connector_Generic:Conn_01x01
- removed J13: Xavier, Connector_PinHeader_2.54mm:PinHeader_1x02_P2.54mm_Vertical, symbol Connector_Generic:Conn_01x02
- removed J14: Kamera 1, Connector_PinHeader_2.54mm:PinHeader_1x02_P2.54mm_Vertical, symbol Connector_Generic:Conn_01x02
- removed J15: Kamera 2, Connector_PinHeader_2.54mm:PinHeader_1x02_P2.54mm_Vertical, symbol Connector_Generic:Conn_01x02
- removed J16, J17, J21, J5, J6: Extra, Connector_PinHeader_2.54mm:PinHeader_1x02_P2.54mm_Vertical, symbol Connector_Generic:Conn_01x02
- removed J18: Hydrofony, Connector_PinHeader_2.54mm:PinHeader_1x03_P2.54mm_Vertical, symbol Connector_Generic:Conn_01x03
- removed J19: Extra, Connector_Molex:Molex_SPOX_5267-02A_1x02_P2.50mm_Vertical, symbol Connector_Generic:Conn_01x02
- removed J2: Battery digital, Connector_PinSocket_2.54mm:PinSocket_2x01_P2.54mm_Vertical, symbol Connector_Generic:Conn_02x01
- removed J20: Extra, Connector_Molex:Molex_Mini-Fit_Jr_5566-02A_2x01_P4.20mm_Vertical, symbol Connector_Generic:Conn_01x02
- removed J22: RC_D_15V, Connector_PinHeader_2.54mm:PinHeader_1x01_P2.54mm_Vertical, symbol Connector_Generic:Conn_01x01
- removed J3: Manip_SterSil2, Connector_PinHeader_2.54mm:PinHeader_1x02_P2.54mm_Vertical, symbol Connector_Generic:Conn_01x02
- removed J37: STM32, Connector_PinHeader_2.54mm:PinHeader_1x02_P2.54mm_Vertical, symbol Connector_Generic:Conn_01x02
- removed J4: Manip_SterSil1, Connector_PinHeader_2.54mm:PinHeader_1x02_P2.54mm_Vertical, symbol Connector_Generic:Conn_01x02
- removed J47: Enko_inkrementalny, Connector_PinHeader_2.54mm:PinHeader_1x02_P2.54mm_Vertical, symbol Connector_Generic:Conn_01x02
- removed J48: Torpedy, hall, laser, Connector_PinHeader_2.54mm:PinHeader_1x02_P2.54mm_Vertical, symbol Connector_Generic:Conn_01x02
- removed J49: Enko_absolutny_1, Connector_PinHeader_2.54mm:PinHeader_1x02_P2.54mm_Vertical, symbol Connector_Generic:Conn_01x02
- removed J50: Enko_absolutny_2, Connector_PinHeader_2.54mm:PinHeader_1x02_P2.54mm_Vertical, symbol Connector_Generic:Conn_01x02
- removed J7: RC_D_5V, Connector_PinHeader_2.54mm:PinHeader_1x01_P2.54mm_Vertical, symbol Connector_Generic:Conn_01x01
- removed J8: RPi, Connector_PinHeader_2.54mm:PinHeader_1x02_P2.54mm_Vertical, symbol Connector_Generic:Conn_01x02
- removed J9: Router, Connector_PinHeader_2.54mm:PinHeader_1x02_P2.54mm_Vertical, symbol Connector_Generic:Conn_01x02
- removed PS1: RPA60-2405SFW_P, RPA60-2405SFW_P:RPA60-2405SFW_P, symbol RPA60-2405SFW_P:RPA60-2405SFW_P
- removed PS2: DCW12A-15, DCW12A-15:DCW12A-15, symbol DCW12A-15:DCW12A-15
- removed Q1, Q2: IPT004N03L, Package_TO_SOT_SMD:Infineon_PG-HSOF-8-1, symbol Device:Q_NMOS_GSD
- removed Q3, Q4, Q5: BC847A, Package_TO_SOT_SMD:SOT-23, symbol Device:Q_NPN_BEC
- removed R1: 3k, Resistor_SMD:R_0805_2012Metric, symbol Device:R
- removed R2: 100, Resistor_SMD:R_0805_2012Metric, symbol Device:R
- removed R3: 10k, Resistor_SMD:R_0805_2012Metric, symbol Device:R
- removed R4: 400, Resistor_SMD:R_0805_2012Metric, symbol Device:R
- removed R5: 1k8, Resistor_SMD:R_0805_2012Metric, symbol Device:R
- removed R6, R7: 2k4, Resistor_SMD:R_0805_2012Metric, symbol Device:R
- removed TP1, TP4: D_5V, Connector_PinHeader_2.54mm:PinHeader_1x01_P2.54mm_Vertical, symbol Connector:TestPoint
- removed TP2: D_12V, Connector_PinHeader_2.54mm:PinHeader_1x01_P2.54mm_Vertical, symbol Connector:TestPoint
- removed TP3: EXTRA, Connector_PinHeader_2.54mm:PinHeader_1x01_P2.54mm_Vertical, symbol Connector:TestPoint
- removed TP5: D_-5V, Connector_PinHeader_2.54mm:PinHeader_1x01_P2.54mm_Vertical, symbol Connector:TestPoint
- removed U1: lm2596, lm2596:lm2596-44_8mm_x_23mm, symbol lm2596:lm2596
Connections:
- no-connect marks 2 -> 0
Other:
- note removed: "+/-15v:\n> in max 2 A,\n> fuse: 3-4-5A ?,\n> out min: +/- 0.04A\n> out max: +/- 0.8A\n\n-Hydrofony\n"
- note removed: "+15V"
- note removed: "-15V"
- note removed: "12V"
- note removed: "12V:\n> in max 15 A,\n> fuse: 20A fast blown,\n> out max: 10A\n\n-Xavier: <4A\n-Kamera 1: <2A\n-Kamera 2: <2A\n\n-dodatkowe: <2A\n\n= 8A\n"
- note removed: "5V"
- note removed: "5V:\n> in max 8 A,\n> fuse: 10A slow blown,\n> out max: 12A\n\n-Router: 2A\n-Switch: 2A\n-RPi: 2A\n\n-AHRS, Bar02 (depth), distance?: <1A\n-Torpedy: hall, laser: <1A\n\n= 8A\n"
- note removed: "Dodatkow:\nxl4017 5A\n\n"
- note removed: "Przekaźnik do załączania zasilania zewnętrznym \nprzełącznikiem (kontaktronem) z zabezpieczeniem przed \nodwrotną polaryzacją"
- note removed: "RC:\nON 2.4-10 V | OPEN\nOFF 0-0.8V | GND"
- note removed: "RC:\nON 3.5-15 V | OPEN\nOFF 0-0.8V | GND"
- note removed: "RC:\nON >4 V | OPEN\nOFF <1V | GND"
- note removed: "TO na osobnym pcb"
