File: zasilanie/projekt/rov4/logika_main/rov4.kicad_pcb (KiCad board)
At the start: 2 copper layers, 146 parts, among them IC1 UWE-12_10-Q12PB-C, IC2 UWE-12_10-Q12PB-C, J1 Battery digital, J10 Router, J11 Switch, J12 Enko_inkrementalny, J13 Torpedy, hall, laser, J14 Enko_absolutny_1, J15 Enko_absolutny_2, J16 RC_D_12V, J17 Xavier, J18 Kamera 1, J19 Kamera 2, J2 Reed switch, J20 Extra, J21 Extra, J22 hydrofony, J23 RC_D_15V, J24 Extra, J25 Extra, J26 Extra, J27 HP_Enable, J28 ESC1, J29 ESC2, J3 RC_D_5V, J30 ESC3, J31 ESC4, J32 ESC5, J33 ESC6, J34 ESC7, J35 ESC8, J36 Manip_sil_12v, J37 Torp_EleMagnes, J38 Extra, J39 RC_HP_12V, J4 Manip_SterSil2, J40 Extra, J41 Manip_Silnik_1, J42 Manip_Silnik_2, J43 Torpedy_serwo_7v, J44 Extra, J45 Extra, J46 Manip_serwo, J47 Extra, J48 Extra, J49 Extra, J5 Manip_SterSil1, J50 Extra, J51 Extra, J52 HP_OUT, J53 HP_IN, J54 HP_IN, J55 LP_OUT, J56 LP_IN, J6 Extra, J7 Extra, J8 STM32, J9 RPi, Q1 IPT004N03L, Q2 IPT004N03L, Q3 BC847A, Q4 BC847A, Q5 BC847A, Q6 IPT004N03L, Q7 IPT004N03L, Q8 IPT004N03L, Q9 IPT004N03L, U1 lm2596, U2 Transoptor, U3 Transoptor, U4 lm2596, U5 lm2596, U6 lm2596

Commit message: PCB: logika_main
Parts:
- removed C14, C24, C27, C28, C29: 100nF, Capacitor_SMD:C_0805_2012Metric
- removed C15, C16, C17, C18, C19, C20, C21: C, Capacitor_THT:C_Radial_D10.0mm_H20.0mm_P5.00mm
- removed C22: C, Capacitor_THT:C_Radial_D12.5mm_H20.0mm_P5.00mm
- removed C23: 33uF, Capacitor_SMD:CP_Elec_6.3x5.4
- removed C25: 10uF, Capacitor_SMD:C_0805_2012Metric
- removed C26: 200uF, Capacitor_SMD:CP_Elec_8x10
- removed D10: LED_G, LED_SMD:LED_0805_2012Metric
- removed D11: LED_R, LED_SMD:LED_0805_2012Metric
- removed D12, D13, D9: BAT48, Diode_SMD:D_MiniMELF
- removed D14: LED_B, LED_SMD:LED_0805_2012Metric
- removed IC2: UWE-12_10-Q12PB-C, UWE-12_10-Q12P-C:UWE-12_10-Q12P-C
- removed J24, J25, J26, J38, J40, J44, J45, J47, J48, J49, J50, J51: Extra, Connector_Molex:Molex_Mini-Fit_Jr_5566-02A_2x01_P4.20mm_Vertical
- removed J27: HP_Enable, Connector_Molex:Molex_SPOX_5267-02A_1x02_P2.50mm_Vertical
- removed J28: ESC1, Connector_Molex:Molex_Mini-Fit_Jr_5566-04A_2x02_P4.20mm_Vertical
- removed J29: ESC2, Connector_Molex:Molex_Mini-Fit_Jr_5566-04A_2x02_P4.20mm_Vertical
- removed J30: ESC3, Connector_Molex:Molex_Mini-Fit_Jr_5566-04A_2x02_P4.20mm_Vertical
- removed J31: ESC4, Connector_Molex:Molex_Mini-Fit_Jr_5566-04A_2x02_P4.20mm_Vertical
- removed J32: ESC5, Connector_Molex:Molex_Mini-Fit_Jr_5566-04A_2x02_P4.20mm_Vertical
- removed J33: ESC6, Connector_Molex:Molex_Mini-Fit_Jr_5566-04A_2x02_P4.20mm_Vertical
- removed J34: ESC7, Connector_Molex:Molex_Mini-Fit_Jr_5566-04A_2x02_P4.20mm_Vertical
- removed J35: ESC8, Connector_Molex:Molex_Mini-Fit_Jr_5566-04A_2x02_P4.20mm_Vertical
- removed J36: Manip_sil_12v, Connector_Molex:Molex_Mini-Fit_Jr_5566-02A_2x01_P4.20mm_Vertical
- removed J37: Torp_EleMagnes, Connector_Molex:Molex_Mini-Fit_Jr_5566-02A_2x01_P4.20mm_Vertical
- removed J39: RC_HP_12V, Connector_Molex:Molex_SPOX_5267-02A_1x02_P2.50mm_Vertical
- removed J41: Manip_Silnik_1, Connector_Molex:Molex_Mini-Fit_Jr_5566-02A_2x01_P4.20mm_Vertical
- removed J42: Manip_Silnik_2, Connector_Molex:Molex_Mini-Fit_Jr_5566-02A_2x01_P4.20mm_Vertical
- removed J43: Torpedy_serwo_7v, Connector_Molex:Molex_Mini-Fit_Jr_5566-02A_2x01_P4.20mm_Vertical
- removed J46: Manip_serwo, Connector_Molex:Molex_Mini-Fit_Jr_5566-02A_2x01_P4.20mm_Vertical
- removed J52: HP_OUT, Connector_Molex:Molex_Mini-Fit_Jr_5566-04A_2x02_P4.20mm_Vertical
- removed J53, J54: HP_IN, Connector_Molex:Molex_Mini-Fit_Jr_5566-04A_2x02_P4.20mm_Vertical
- removed J56: LP_IN, Connector_Molex:Molex_Mini-Fit_Jr_5566-04A_2x02_P4.20mm_Vertical
- removed L1, L2, L3, L4, L5, L6, L7, L8: L, 74435571100:74435571100
- removed Q6, Q7, Q8, Q9: IPT004N03L, Package_TO_SOT_SMD:Infineon_PG-HSOF-8-1
- removed R10: 10k, Resistor_SMD:R_0805_2012Metric
- removed R11: 1k8, Resistor_SMD:R_0805_2012Metric
- removed R8: 3k, Resistor_SMD:R_0805_2012Metric
- removed R9: 100, Resistor_SMD:R_0805_2012Metric
- removed TP5, TP9: EXTRA, Connector_PinHeader_2.54mm:PinHeader_1x01_P2.54mm_Vertical
- removed TP6: HP_12V, Connector_PinHeader_2.54mm:PinHeader_1x01_P2.54mm_Vertical
- removed TP7: HP_7V, Connector_PinHeader_2.54mm:PinHeader_1x01_P2.54mm_Vertical
- removed TP8: HP_5V, Connector_PinHeader_2.54mm:PinHeader_1x01_P2.54mm_Vertical
- removed U1, U4, U5, U6: lm2596, lm2596:lm2596-44_8mm_x_23mm
- removed U2, U3: Transoptor, Package_DIP:DIP-4_W7.62mm
- added R12: 3k3, Resistor_SMD:R_0805_2012Metric, F.Cu at (125.7, 74.9)
- added R13: 3k3, Resistor_SMD:R_0805_2012Metric, B.Cu at (109.2, 82.5)
- added R14: 3k3, Resistor_SMD:R_0805_2012Metric, F.Cu at (205.7, 125.7)
- D3, D4, Q1, Q2, R1, R2, R3, R5: moved to B.Cu
- J16, J23, J3: footprint Connector_PinHeader_2.54mm:PinHeader_1x01_P2.54mm_Vertical -> Connector_Molex:Molex_SPOX_5267-02A_1x02_P2.50mm_Vertical
- Q3, Q5: moved to F.Cu
- moved J55 299.6 mm to (82.5, 141.0)
- moved J15 243.1 mm to (54.6, 55.9), turned to 180 degrees
- moved J21 238.5 mm to (55.9, 80.0)
- moved C7 230.5 mm to (50.2, 102.9), turned to 90 degrees
- moved J14 226.8 mm to (64.8, 55.9)
- moved J19 223.9 mm to (76.2, 80.0)
- moved J20 223.9 mm to (66.0, 80.0)
- moved C6 223.5 mm to (53.3, 102.9), turned to 90 degrees
- moved J17 217.2 mm to (76.2, 55.9), turned to 180 degrees
- moved R2 208.5 mm to (67.3, 136.8), turned to 90 degrees
- moved J1 205.6 mm to (61.0, 129.5), turned to 90 degrees
- moved D2 203.6 mm to (53.3, 133.7)
- moved D3 201.4 mm to (54.6, 124.9), turned to 270 degrees
- moved D1 201.2 mm to (53.3, 125.4), turned to 90 degrees
- moved D4 200.0 mm to (54.6, 134.1)
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Connections:
- D1 pad 1: Net-(D1-Pad1) -> /logika_main/-Batt
- D2 pad 1: Net-(D1-Pad2) -> Net-(D2-Pad1)
- D2 pad 2: Net-(D2-Pad2) -> /logika_main/-Batt
- D3 pad 1: /logika_main/-Batt -> Net-(D1-Pad2)
- D3 pad 2: Net-(D1-Pad1) -> Net-(D3-Pad2)
- D4 pad 1: Net-(D2-Pad2) -> Net-(D3-Pad2)
- D4 pad 2: /logika_main/-Batt -> Net-(D2-Pad1)
- J13 pad 1: -BattDigit -> Net-(C2-Pad1)
- J13 pad 2: Net-(C2-Pad1) -> -BattDigit
- Q3 pad 1: Net-(J3-Pad1) -> Net-(Q3-Pad1)
- Q4 pad 1: Net-(J16-Pad1) -> Net-(Q4-Pad1)
- Q5 pad 1: Net-(J23-Pad1) -> Net-(Q5-Pad1)
- R1 pad 2: Net-(D1-Pad2) -> Net-(D3-Pad2)
Routing:
- net -BattPow: track 322.6 -> 0.00 mm
- net Net-(C28-Pad1): track 12.5 -> 0.00 mm
- net Net-(D2-Pad2): track 2.73 -> 0.00 mm
Other:
- board outline added: 188 x 120 mm
- rule pad_to_mask_clearance: 0.051 -> 0

Commit message: Jakieś zmainy wszystkiego
Parts:
- added REF**: MountingHole_3.2mm_M3_Pad, MountingHole:MountingHole_3.2mm_M3_Pad, F.Cu at (135.0, 35.0)
- added REF**: MountingHole_3.2mm_M3_Pad, MountingHole:MountingHole_3.2mm_M3_Pad, F.Cu at (35.0, 35.0)
- added REF**: MountingHole_3.2mm_M3_Pad, MountingHole:MountingHole_3.2mm_M3_Pad, F.Cu at (35.0, 105.0)
- added REF**: MountingHole_3.2mm_M3_Pad, MountingHole:MountingHole_3.2mm_M3_Pad, F.Cu at (135.0, 105.0)
- added REF**: MountingHole_3.2mm_M3_Pad, MountingHole:MountingHole_3.2mm_M3_Pad, F.Cu at (135.0, 205.0)
- added REF**: MountingHole_3.2mm_M3_Pad, MountingHole:MountingHole_3.2mm_M3_Pad, F.Cu at (35.0, 205.0)
- J10, J11, J12, J13, J14, J15, J17, J18, J19, J20, J21, J4, J5, J6, J7, J8, J9: footprint Connector_Molex:Molex_Mini-Fit_Jr_5566-02A_2x01_P4.20mm_Vertical -> molex_3d_2pin:Molex_Mini-Fit_Jr_5566-02A_2x01_P4.20mm_Vertical
- moved Q5 167.2 mm to (59.4, 195.6), turned to 180 degrees
- moved R7 163.8 mm to (121.9, 198.1), turned to 180 degrees
- moved D8 162.6 mm to (117.2, 198.1), turned to 180 degrees
- moved R14 160.9 mm to (58.4, 190.5), turned to 90 degrees
- moved TP4 156.7 mm to (121.9, 193.0), turned to 0 degrees
- moved C11 156.2 mm to (64.8, 189.2), turned to 270 degrees
- moved C12 155.7 mm to (106.7, 194.3), turned to 270 degrees
- moved C13 155.4 mm to (100.3, 194.3), turned to 270 degrees
- moved PS2 150.8 mm to (80.0, 189.2), turned to 90 degrees
- moved J23 149.3 mm to (58.4, 181.6), turned to 270 degrees
- moved J22 146.9 mm to (115.6, 187.1), turned to 270 degrees
- moved TP3 146.2 mm to (121.9, 185.4), turned to 0 degrees
- moved C9 141.3 mm to (106.7, 184.2), turned to 270 degrees
- moved C10 141.0 mm to (100.3, 184.2), turned to 270 degrees
- moved R6 139.2 mm to (121.9, 180.3), turned to 0 degrees
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Other:
- board size 188 x 120 mm -> 120 x 190 mm
- board text added: "logika main pcb"
