File: zasilanie/projekt/rov4/logika_main/logika_pcb.kicad_pcb (KiCad board)
At the start: 2 copper layers, 125 x 183.5 mm, 80 parts, among them IC1 UWE-12_10-Q12PB-C, J1 Battery digital, J10 Router, J11 Switch, J12 Enko_inkrementalny, J13 Torpedy, hall, laser, J14 Enko_absolutny_1, J15 Enko_absolutny_2, J16 RC_D_12V, J17 Xavier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

Commit message: kosmetyka
Parts:
- D19, D20: moved to B.Cu
Routing:
- net -BattDigit: track 10.6 -> 7.76 mm, vias 5 -> 4
- net Net-(D19-Pad1): vias 1 -> 0
- net /logika_main/-Batt: vias 2 -> 3
