File: zasilanie/projekt/rov4/moc_main/rov4.kicad_pcb (KiCad board)
At the start: 2 copper layers, 121 parts, among them IC1 UWE-12_10-Q12PB-C, IC2 UWE-12_10-Q12PB-C, J1 Battery digital, J10 Router, J12 Enko_inkrementalny, J13 Torpedy, hall, laser, J14 Enko_absolutny_1, J15 Enko_absolutny_2, J16 RC_D_12V, J17 Xavier, J18 Kamera 1, J19 Kamera 2, J2 Reed switch, J20 Extra, J21 Extra, J22 hydrofony, J23 RC_D_15V, J24 Extra, J25 Extra, J26 Extra, J27 HP_Enable, J28 ESC1, J29 ESC2, J3 RC_D_5V, J30 ESC3, J31 ESC4, J32 ESC5, J33 ESC6, J34 ESC7, J35 ESC8, J36 Manip_sil_12v, J37 Torp_EleMagnes, J38 Extra, J4 Manip_SterSil2, J47 Extra, J48 Extra, J49 Extra, J5 Manip_SterSil1, J50 Extra, J51 Extra, J52 HP_OUT, J53 HP_IN, J54 HP_IN, J55 LP_OUT, J56 LP_IN, J6 Extra, J7 Extra, J8 STM32, J9 RPi, Q1 IPT004N03L, Q2 IPT004N03L, Q3 BC847A, Q4 BC847A, Q5 BC847A, Q6 IPT004N03L, Q7 IPT004N03L, Q8 IPT004N03L, Q9 IPT004N03L, U1 lm2596, U2 Transoptor, U3 Transoptor, U4 lm2596, U5 lm2596, U6 lm2596

Commit message: Jakieś zmainy wszystkiego
Parts:
- removed C1, C11, C5: 33uF, Capacitor_SMD:CP_Elec_6.3x5.4
- removed C10, C13: 100uF, Capacitor_SMD:CP_Elec_6.3x7.7
- removed C12, C14, C2, C6, C9: 100nF, Capacitor_SMD:C_0805_2012Metric
- removed C3, C7: 10uF, Capacitor_SMD:C_0805_2012Metric
- removed C4, C8: 200uF, Capacitor_SMD:CP_Elec_8x10
- removed D1: LED_G, LED_SMD:LED_0805_2012Metric
- removed D2: LED_R, LED_SMD:LED_0805_2012Metric
- removed D3, D4: BAT48, Diode_SMD:D_MiniMELF
- removed D5, D6, D7, D8: LED_B, LED_SMD:LED_0805_2012Metric
- removed IC1: UWE-12_10-Q12PB-C, UWE-12_10-Q12P-C:UWE-12_10-Q12P-C
- removed J1: Battery digital, power_connectors:XT60UPB-M
- removed J10: Router, Connector_Molex:Molex_Mini-Fit_Jr_5566-02A_2x01_P4.20mm_Vertical
- removed J12: Enko_inkrementalny, Connector_Molex:Molex_Mini-Fit_Jr_5566-02A_2x01_P4.20mm_Vertical
- removed J13: Torpedy, hall, laser, Connector_Molex:Molex_Mini-Fit_Jr_5566-02A_2x01_P4.20mm_Vertical
- removed J14: Enko_absolutny_1, Connector_Molex:Molex_Mini-Fit_Jr_5566-02A_2x01_P4.20mm_Vertical
- removed J15: Enko_absolutny_2, Connector_Molex:Molex_Mini-Fit_Jr_5566-02A_2x01_P4.20mm_Vertical
- removed J16: RC_D_12V, Connector_PinHeader_2.54mm:PinHeader_1x01_P2.54mm_Vertical
- removed J17: Xavier, Connector_Molex:Molex_Mini-Fit_Jr_5566-02A_2x01_P4.20mm_Vertical
- removed J18: Kamera 1, Connector_Molex:Molex_Mini-Fit_Jr_5566-02A_2x01_P4.20mm_Vertical
- removed J19: Kamera 2, Connector_Molex:Molex_Mini-Fit_Jr_5566-02A_2x01_P4.20mm_Vertical
- removed J2: Reed switch, Connector_Molex:Molex_SPOX_5267-02A_1x02_P2.50mm_Vertical
- removed J20, J21, J24, J25, J26, J47, J48, J49, J50, J51, J6, J7: Extra, Connector_Molex:Molex_Mini-Fit_Jr_5566-02A_2x01_P4.20mm_Vertical
- removed J22: hydrofony, Connector_Molex:Molex_Mini-Fit_Jr_5566-04A_2x02_P4.20mm_Vertical
- removed J23: RC_D_15V, Connector_PinHeader_2.54mm:PinHeader_1x01_P2.54mm_Vertical
- removed J3: RC_D_5V, Connector_PinHeader_2.54mm:PinHeader_1x01_P2.54mm_Vertical
- removed J4: Manip_SterSil2, Connector_Molex:Molex_Mini-Fit_Jr_5566-02A_2x01_P4.20mm_Vertical
- removed J5: Manip_SterSil1, Connector_Molex:Molex_Mini-Fit_Jr_5566-02A_2x01_P4.20mm_Vertical
- removed J53, J54: HP_IN, Connector_Molex:Molex_Mini-Fit_Jr_5566-04A_2x02_P4.20mm_Vertical
- removed J55: LP_OUT, Connector_Molex:Molex_Mini-Fit_Jr_5566-04A_2x02_P4.20mm_Vertical
- removed J56: LP_IN, Connector_Molex:Molex_Mini-Fit_Jr_5566-04A_2x02_P4.20mm_Vertical
- removed J8: STM32, Connector_Molex:Molex_Mini-Fit_Jr_5566-02A_2x01_P4.20mm_Vertical
- removed J9: RPi, Connector_Molex:Molex_Mini-Fit_Jr_5566-02A_2x01_P4.20mm_Vertical
- removed PS1: RPA60-2405SFW_P, RPA60-2405SFW_P:RPA60-2405SFW_P
- removed PS2: DCW12A-15, DCW12A-15:DCW12A-15
- removed Q1, Q2: IPT004N03L, Package_TO_SOT_SMD:Infineon_PG-HSOF-8-1
- removed Q3, Q4, Q5: BC847A, Package_TO_SOT_SMD:SOT-23
- removed R1: 3k, Resistor_SMD:R_0805_2012Metric
- removed R2: 100, Resistor_SMD:R_0805_2012Metric
- removed R3: 10k, Resistor_SMD:R_0805_2012Metric
- removed R4: 400, Resistor_SMD:R_0805_2012Metric
- removed R5: 1k8, Resistor_SMD:R_0805_2012Metric
- removed R6, R7: 2k4, Resistor_SMD:R_0805_2012Metric
- removed TP1, TP3: D_5V, Connector_PinHeader_2.54mm:PinHeader_1x01_P2.54mm_Vertical
- removed TP2: D_12V, Connector_PinHeader_2.54mm:PinHeader_1x01_P2.54mm_Vertical
- removed TP4: D_-5V, Connector_PinHeader_2.54mm:PinHeader_1x01_P2.54mm_Vertical
- removed TP5, TP9: EXTRA, Connector_PinHeader_2.54mm:PinHeader_1x01_P2.54mm_Vertical
- removed TP7: HP_7V, Connector_PinHeader_2.54mm:PinHeader_1x01_P2.54mm_Vertical
- removed TP8: HP_5V, Connector_PinHeader_2.54mm:PinHeader_1x01_P2.54mm_Vertical
- removed U1, U4, U5, U6: lm2596, lm2596:lm2596-44_8mm_x_23mm
- added C22: C, Capacitor_THT:C_Radial_D10.0mm_H20.0mm_P5.00mm, F.Cu at (59.9, 40.3)
- added C23: 33uF, Capacitor_SMD:CP_Elec_6.3x5.4, B.Cu at (295.9, 110.5)
- added C24: 100nF, Capacitor_SMD:C_0805_2012Metric, B.Cu at (295.9, 71.1)
- added C25: 10uF, Capacitor_SMD:C_0805_2012Metric, B.Cu at (295.9, 63.5)
- added C26: 200uF, Capacitor_SMD:CP_Elec_8x10, B.Cu at (295.9, 78.7)
- added J39: RC_HP_12V, Connector_Molex:Molex_SPOX_5267-02A_1x02_P2.50mm_Vertical, F.Cu at (278.1, 45.7)
- added J40: Extra, molex_3d_2pin:Molex_Mini-Fit_Jr_5566-02A_2x01_P4.20mm_Vertical, F.Cu at (341.6, 67.3)
- added J41: Manip_Silnik_1, molex_3d_2pin:Molex_Mini-Fit_Jr_5566-02A_2x01_P4.20mm_Vertical, F.Cu at (321.3, 77.5)
- added J42: Manip_Silnik_2, molex_3d_2pin:Molex_Mini-Fit_Jr_5566-02A_2x01_P4.20mm_Vertical, F.Cu at (321.3, 97.8)
- added J58: +BattPower, MountingHole:MountingHole_5.5mm_Pad, F.Cu at (217.4, 47.8)
- added J59: -BattPower, MountingHole:MountingHole_5.5mm_Pad, F.Cu at (239.4, 47.8)
- added L1: L, 74435571100:74435571100, F.Cu at (67.4, 97.8)
- added L2: L, 74435571100:74435571100, F.Cu at (102.4, 97.8)
- added L3: L, 74435571100:74435571100, F.Cu at (137.4, 97.8)
- added L4: L, 74435571100:74435571100, F.Cu at (172.4, 97.8)
- added L5: L, 74435571100:74435571100, F.Cu at (172.4, 57.8)
- added L6: L, 74435571100:74435571100, F.Cu at (137.4, 57.8)
- added L7: L, 74435571100:74435571100, F.Cu at (102.4, 57.8)
- added L8: L, 74435571100:74435571100, F.Cu at (67.4, 57.8)
- added R15: 680, Resistor_SMD:R_0805_2012Metric, B.Cu at (265.4, 55.9)
- added R16: 680, Resistor_SMD:R_0805_2012Metric, B.Cu at (278.1, 55.9)
- added REF**: MountingHole_3.2mm_M3_Pad, MountingHole:MountingHole_3.2mm_M3_Pad, F.Cu at (201.9, 31.8)
- added REF**: MountingHole_3.2mm_M3_Pad, MountingHole:MountingHole_3.2mm_M3_Pad, F.Cu at (201.9, 125.7)
- added REF**: MountingHole_3.2mm_M3_Pad, MountingHole:MountingHole_3.2mm_M3_Pad, F.Cu at (354.3, 125.7)
- added REF**: MountingHole_3.2mm_M3_Pad, MountingHole:MountingHole_3.2mm_M3_Pad, F.Cu at (354.3, 31.8)
- added REF**: MountingHole_3.2mm_M3_Pad, MountingHole:MountingHole_3.2mm_M3_Pad, F.Cu at (41.9, 31.8)
- added REF**: MountingHole_3.2mm_M3_Pad, MountingHole:MountingHole_3.2mm_M3_Pad, F.Cu at (41.9, 125.7)
- C15, C16, C17, C18, C19, C20, C21: moved to F.Cu
- D12, D13, D9, Q6, Q7, Q8, Q9, R10, R11, R8, R9: moved to B.Cu
- J36, J37, J38: footprint Connector_Molex:Molex_Mini-Fit_Jr_5566-02A_2x01_P4.20mm_Vertical -> molex_3d_2pin:Molex_Mini-Fit_Jr_5566-02A_2x01_P4.20mm_Vertical
- moved J36 360.1 mm to (341.6, 77.5), turned to 90 degrees
- moved J38 336.6 mm to (321.3, 67.3)
- moved J37 330.6 mm to (321.3, 87.6)
- moved D14 236.0 mm to (328.9, 113.0), turned to 0 degrees
- moved R11 231.1 mm to (327.7, 115.6), turned to 0 degrees
- moved J32 227.3 mm to (177.4, 40.3), turned to 90 degrees
- moved TP6 223.7 mm to (321.3, 113.0), turned to 0 degrees
- moved J33 217.7 mm to (142.4, 40.3), turned to 90 degrees
- moved J34 204.5 mm to (107.4, 40.3)
- moved IC2 203.8 mm to (295.9, 93.0), turned to 90 degrees
- moved C19 199.5 mm to (164.9, 40.3), turned to 90 degrees
- moved J35 199.0 mm to (72.4, 40.3), turned to 90 degrees
- moved C20 197.8 mm to (129.9, 40.3), turned to 90 degrees
- moved C21 196.3 mm to (94.9, 40.3), turned to 90 degrees
- moved U3 183.2 mm to (278.1, 52.1)
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Connections:
- D11 pad 1: Net-(D10-Pad2) -> Net-(D11-Pad1)
- D11 pad 2: Net-(D11-Pad2) -> Net-(D10-Pad1)
- D12 pad 1: /moc_main/-BattPower -> Net-(D10-Pad2)
- D12 pad 2: Net-(D10-Pad1) -> Net-(D12-Pad2)
- D13 pad 1: Net-(D11-Pad2) -> Net-(D12-Pad2)
- D13 pad 2: /moc_main/-BattPower -> Net-(D11-Pad1)
- Q6 pad 2: /moc_main/-BattPower -> Net-(D10-Pad1)
- Q8 pad 2: /moc_main/-BattPower -> Net-(D10-Pad1)
- R10 pad 2: /moc_main/-BattPower -> Net-(D10-Pad1)
- R8 pad 2: Net-(D10-Pad2) -> Net-(D12-Pad2)
- U2 pad 1: Net-(J27-Pad1) -> Net-(R15-Pad1)
Routing:
- net +BattPow: track 0.00 -> 807.1 mm
- net Net-(D2-Pad2): track 2.73 -> 0.00 mm
Other:
- board outline added: 327.7 x 109.2 mm
- rule pad_to_mask_clearance: 0.051 -> 0
- board text added: "logika main pcb"
