File: battery — kopia/_saved_battery.sch (KiCad schematic (older format))
At the start: 40 parts, among them J1 batt_1, J2 batt_2, J3 batt_3, J4 batt_4, J5 reed_switch, J6 toPcb+, J7 toPcb-, Q1 batt1_sw, Q2 batt2_sw, Q3 batt3_sw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

Commit message: robust version
Parts:
- removed Q?: Q_NPN_BCE, symbol Device:Q_NPN_BCE
- removed U?: LTV-817, Package_DIP:DIP-4_W7.62mm, symbol Isolator:LTV-817
- added Q5: Q_NPN_CBE, Package_TO_SOT_SMD:SOT-23, symbol Device:Q_NPN_CBE
- added U2: LTV-817S, Package_DIP:SMDIP-4_W9.53mm, symbol Isolator:LTV-817S
- D2, D3, D4, D5, D6, D7, D8, D9: footprint Diode_SMD:D_SMB_Handsoldering -> Diode_SMD:D_SMB
- J8: renamed from J?; footprint (none) -> Connector_Molex:Molex_SPOX_5267-02A_1x02_P2.50mm_Vertical
- R10: renamed from R?; footprint (none) -> Resistor_SMD:R_0805_2012Metric_Pad1.15x1.40mm_HandSolder
Changed lines of the file:
@@
 F 0 "D3" V 3503 3529 50  0000 L CNN
 F 1 "D_TVS" V 3596 3529 50  0000 L CNN
-F 2 "Diode_SMD:D_SMB_Handsoldering" H 3550 3450 50  0001 C CNN
+F 2 "Diode_SMD:D_SMB" H 3550 3450 50  0001 C CNN
 F 3 "~" H 3550 3450 50  0001 C CNN
 	1    3550 3450
@@
 F 0 "D2" V 2403 3529 50  0000 L CNN
 F 1 "D_TVS" V 2496 3529 50  0000 L CNN
-F 2 "Diode_SMD:D_SMB_Handsoldering" H 2450 3450 50  0001 C CNN
+F 2 "Diode_SMD:D_SMB" H 2450 3450 50  0001 C CNN
 F 3 "~" H 2450 3450 50  0001 C CNN
 	1    2450 3450
@@
 F 0 "D5" V 5103 3529 50  0000 L CNN
 F 1 "D_TVS" V 5196 3529 50  0000 L CNN
-F 2 "Diode_SMD:D_SMB_Handsoldering" H 5150 3450 50  0001 C CNN
+F 2 "Diode_SMD:D_SMB" H 5150 3450 50  0001 C CNN
 F 3 "~" H 5150 3450 50  0001 C CNN
 	1    5150 3450
@@
 F 0 "D4" V 4003 3529 50  0000 L CNN
 F 1 "D_TVS" V 4096 3529 50  0000 L CNN
-F 2 "Diode_SMD:D_SMB_Handsoldering" H 4050 3450 50  0001 C CNN
+F 2 "Diode_SMD:D_SMB" H 4050 3450 50  0001 C CNN
 F 3 "~" H 4050 3450 50  0001 C CNN
 	1    4050 3450
@@
 F 0 "D7" V 6703 3529 50  0000 L CNN
 F 1 "D_TVS" V 6796 3529 50  0000 L CNN
-F 2 "Diode_SMD:D_SMB_Handsoldering" H 6750 3450 50  0001 C CNN
+F 2 "Diode_SMD:D_SMB" H 6750 3450 50  0001 C CNN
 F 3 "~" H 6750 3450 50  0001 C CNN
 	1    6750 3450
@@
 F 0 "D6" V 5603 3529 50  0000 L CNN
 F 1 "D_TVS" V 5696 3529 50  0000 L CNN
-F 2 "Diode_SMD:D_SMB_Handsoldering" H 5650 3450 50  0001 C CNN
+F 2 "Diode_SMD:D_SMB" H 5650 3450 50  0001 C CNN
 F 3 "~" H 5650 3450 50  0001 C CNN
 	1    5650 3450
@@
 F 0 "D9" V 8303 3529 50  0000 L CNN
 F 1 "D_TVS" V 8396 3529 50  0000 L CNN
-F 2 "Diode_SMD:D_SMB_Handsoldering" H 8350 3450 50  0001 C CNN
+F 2 "Diode_SMD:D_SMB" H 8350 3450 50  0001 C CNN
 F 3 "~" H 8350 3450 50  0001 C CNN
 	1    8350 3450
@@
 F 0 "D8" V 7203 3529 50  0000 L CNN
 F 1 "D_TVS" V 7296 3529 50  0000 L CNN
-F 2 "Diode_SMD:D_SMB_Handsoldering" H 7250 3450 50  0001 C CNN
+F 2 "Diode_SMD:D_SMB" H 7250 3450 50  0001 C CNN
 F 3 "~" H 7250 3450 50  0001 C CNN
 	1    7250 3450
@@
 $EndComp
 $Comp
-L Isolator:LTV-817 U?
-U 1 1 5D439759
-P 7250 2050
-F 0 "U?" H 7250 2379 50  0000 C CNN
-F 1 "LTV-817" H 7250 2286 50  0000 C CNN
-F 2 "Package_DIP:DIP-4_W7.62mm" H 7050 1850 50  0001 L CIN
-F 3 "http://www.us.liteon.com/downloads/LTV-817-827-847.PDF" H 7250 1950 50  0001 L CNN
-	1    7250 2050
-	1    0    0    -1
-$EndComp
-$Comp
-L Connector_Generic:Conn_01x02 J?
+L Connector_Generic:Conn_01x02 J8
 U 1 1 5D4437CA
 P 6250 1950
-F 0 "J?" H 6250 2100 50  0000 C CNN
+F 0 "J8" H 6250 2100 50  0000 C CNN
 F 1 "on_signal" H 6250 1750 50  0000 C CNN
-F 2 "" H 6250 1950 50  0001 C CNN
+F 2 "Connector_Molex:Molex_SPOX_5267-02A_1x02_P2.50mm_Vertical" H 6250 1950 50  0001 C CNN
 F 3 "~" H 6250 1950 50  0001 C CNN
 	1    6250 1950
@@
 $EndComp
 $Comp
-L Device:R R?
+L Device:R R10
 U 1 1 5D44AE90
 P 6750 1950
-F 0 "R?" V 6540 1950 50  0000 C CNN
+F 0 "R10" V 6540 1950 50  0000 C CNN
 F 1 "R" V 6633 1950 50  0000 C CNN
-F 2 "" V 6680 1950 50  0001 C CNN
+F 2 "Resistor_SMD:R_0805_2012Metric_Pad1.15x1.40mm_HandSolder" V 6680 1950 50  0001 C CNN
 F 3 "~" H 6750 1950 50  0001 C CNN
 	1    6750 1950
@@
 Wire Wire Line
 	6900 2050 6450 2050
-$Comp
-L Device:Q_NPN_BCE Q?
-U 1 1 5D4542AE
-P 7950 2150
-F 0 "Q?" H 8141 2197 50  0000 L CNN
-F 1 "Q_NPN_BCE" H 8141 2104 50  0000 L CNN
-F 2 "" H 8150 2250 50  0001 C CNN
-F 3 "~" H 7950 2150 50  0001 C CNN
-	1    7950 2150
-	1    0    0    -1
-$EndComp
-Wire Wire Line
-	7550 1950 8050 1950
 Wire Wire Line
 	7750 2150 7550 2150
-Connection ~ 8050 1950
 Wire Wire Line
 	9350 1950 9350 2400
@@
 Connection ~ 8050 2400
 Wire Wire Line
+	8050 2400 8700 2400
+$Comp
+L Device:Q_NPN_CBE Q5
+U 1 1 5D48ACB7
+P 7950 2150
+F 0 "Q5" H 8141 2197 50  0000 L CNN
+F 1 "Q_NPN_CBE" H 8141 2104 50  0000 L CNN
+F 2 "Package_TO_SOT_SMD:SOT-23" H 8150 2250 50  0001 C CNN
+F 3 "~" H 7950 2150 50  0001 C CNN
+	1    7950 2150
+	1    0    0    -1
+$EndComp
+Wire Wire Line
+	7550 1950 8050 1950
+Connection ~ 8050 1950
+Wire Wire Line
 	8050 1950 9350 1950
-Wire Wire Line
-	8050 2400 8700 2400
+$Comp
+L Isolator:LTV-817S U2
+U 1 1 5D48BD4A
+P 7250 2050
+F 0 "U2" H 7250 2379 50  0000 C CNN
+F 1 "LTV-817S" H 7250 2286 50  0000 C CNN
+F 2 "Package_DIP:SMDIP-4_W9.53mm" H 7250 1750 50  0001 C CNN
+F 3 "http://www.us.liteon.com/downloads/LTV-817-827-847.PDF" H 6900 2350 50  0001 C CNN
+	1    7250 2050
+	1    0    0    -1
+$EndComp
 $EndSCHEMATC
