File: battery/battery.kicad_pcb (KiCad board)
At the start: 2 copper layers, 170.2 x 63.5 mm, 53 parts, among them J1 batt_1, J2 batt_2, J3 batt_3, J4 batt_4, J5 reed_switch, J6 toPcb+, J7 toPcb-, J8 on_signal, Q1 batt1_sw, Q2 batt2_sw, Q3 batt3_sw, Q4 batt4_sw, Q5 BC817-25, U1 LM1117-5.0, U2 LTV-817S

Commit message: drc fix
Parts:
- removed the C1 at (109.2, 71.4)
- removed the C10 at (164.8, 87.2)
- removed the C2 at (111.8, 71.4)
- removed the C3 at (121.0, 73.5)
- removed the C4 at (136.0, 73.5)
- removed the C5 at (151.3, 73.5)
- removed the C6 at (166.6, 73.5)
- removed the C7 at (119.1, 87.2)
- removed the C8 at (134.4, 87.2)
- removed the C9 at (149.6, 87.2)
- removed the D1 at (106.7, 79.4)
- removed the D10 at (113.0, 90.2)
- removed the D11 at (128.3, 90.2)
- removed the D12 at (143.5, 90.2)
- removed the D13 at (158.8, 90.2)
- removed the D2 at (120.8, 83.2)
- removed the D3 at (120.8, 77.5)
- removed the D4 at (136.1, 83.2)
- removed the D5 at (136.1, 77.5)
- removed the D6 at (151.3, 83.2)
- removed the D7 at (151.3, 77.5)
- removed the D8 at (166.5, 83.2)
- removed the D9 at (166.5, 77.5)
- removed the H1 at (102.9, 120.0)
- removed the H2 at (102.9, 64.1)
- removed the H3 at (184.2, 64.1)
- removed the H4 at (184.2, 120.0)
- removed the J1 at (121.9, 101.0)
- removed the J2 at (137.2, 101.0)
- removed the J3 at (152.4, 101.0)
- removed the J4 at (167.6, 101.0)
- removed the J5 at (104.1, 105.4)
- removed the J6 at (179.7, 108.0)
- removed the J7 at (179.7, 94.0)
- removed the J8 at (113.0, 105.4)
- removed the Q1 at (119.6, 80.0)
- removed the Q2 at (134.9, 80.3)
- removed the Q3 at (150.1, 80.3)
- removed the Q4 at (165.4, 80.3)
- removed the Q5 at (108.0, 95.9)
- removed the R1 at (105.4, 71.1)
- removed the R10 at (108.3, 112.4)
- removed the R11 at (113.6, 99.3)
- removed the R2 at (113.7, 95.6)
- removed the R3 at (128.9, 95.6)
- removed the R4 at (144.1, 95.6)
- removed the R5 at (159.4, 95.6)
- removed the R6 at (116.2, 97.5)
- removed the R7 at (131.4, 97.5)
- removed the R8 at (146.7, 97.5)
- removed the R9 at (161.9, 97.5)
- removed the U1 at (106.7, 78.1)
- removed the U2 at (108.6, 104.1)
- added C1: C_Small, Capacitor_SMD:C_0805_2012Metric_Pad1.15x1.40mm_HandSolder, B.Cu at (191.4, 68.6)
- added C1: C_Small, Capacitor_SMD:C_0805_2012Metric_Pad1.15x1.40mm_HandSolder, F.Cu at (103.3, 68.6)
- added C10: 100n, Capacitor_SMD:C_0805_2012Metric_Pad1.15x1.40mm_HandSolder, F.Cu at (207.3, 124.2)
- added C10: 100n, Capacitor_SMD:C_0805_2012Metric_Pad1.15x1.40mm_HandSolder, B.Cu at (87.4, 124.2)
- added C2: C_Small, Capacitor_SMD:C_0805_2012Metric_Pad1.15x1.40mm_HandSolder, B.Cu at (191.4, 71.1)
- added C2: C_Small, Capacitor_SMD:C_0805_2012Metric_Pad1.15x1.40mm_HandSolder, F.Cu at (103.3, 71.1)
- added C3: 10uF, Capacitor_SMD:C_1206_3216Metric_Pad1.42x1.75mm_HandSolder, F.Cu at (193.5, 80.4)
- added C3: 10uF, Capacitor_SMD:C_1206_3216Metric_Pad1.42x1.75mm_HandSolder, B.Cu at (101.1, 80.4)
- added C4: 10uF, Capacitor_SMD:C_1206_3216Metric_Pad1.42x1.75mm_HandSolder, F.Cu at (193.5, 95.4)
- added C4: 10uF, Capacitor_SMD:C_1206_3216Metric_Pad1.42x1.75mm_HandSolder, B.Cu at (101.1, 95.4)
- added C5: 10uF, Capacitor_SMD:C_1206_3216Metric_Pad1.42x1.75mm_HandSolder, F.Cu at (193.5, 110.6)
- added C5: 10uF, Capacitor_SMD:C_1206_3216Metric_Pad1.42x1.75mm_HandSolder, B.Cu at (101.1, 110.6)
- added C6: 10uF, Capacitor_SMD:C_1206_3216Metric_Pad1.42x1.75mm_HandSolder, F.Cu at (193.5, 126.0)
- added C6: 10uF, Capacitor_SMD:C_1206_3216Metric_Pad1.42x1.75mm_HandSolder, B.Cu at (101.1, 126.0)
- added C7: 100n, Capacitor_SMD:C_0805_2012Metric_Pad1.15x1.40mm_HandSolder, F.Cu at (207.3, 78.5)
- added C7: 100n, Capacitor_SMD:C_0805_2012Metric_Pad1.15x1.40mm_HandSolder, B.Cu at (87.4, 78.5)
- added C8: 100n, Capacitor_SMD:C_0805_2012Metric_Pad1.15x1.40mm_HandSolder, F.Cu at (207.3, 93.7)
- added C8: 100n, Capacitor_SMD:C_0805_2012Metric_Pad1.15x1.40mm_HandSolder, B.Cu at (87.4, 93.7)
- added C9: 100n, Capacitor_SMD:C_0805_2012Metric_Pad1.15x1.40mm_HandSolder, F.Cu at (207.3, 109.0)
- added C9: 100n, Capacitor_SMD:C_0805_2012Metric_Pad1.15x1.40mm_HandSolder, B.Cu at (87.4, 109.0)
- added D1: power_ok, LED_SMD:LED_0805_2012Metric, F.Cu at (199.4, 66.0)
- added D1: power_ok, LED_SMD:LED_0805_2012Metric, B.Cu at (95.2, 66.0)
- added D10: bat48, Diode_THT:D_DO-35_SOD27_P10.16mm_Horizontal, F.Cu at (210.2, 71.1)
- added D10: bat48, Diode_THT:D_DO-35_SOD27_P10.16mm_Horizontal, B.Cu at (84.5, 71.1)
- added D11: bat48, Diode_THT:D_DO-35_SOD27_P10.16mm_Horizontal, F.Cu at (210.2, 86.4)
- added D11: bat48, Diode_THT:D_DO-35_SOD27_P10.16mm_Horizontal, B.Cu at (84.5, 86.4)
- added D12: bat48, Diode_THT:D_DO-35_SOD27_P10.16mm_Horizontal, F.Cu at (210.2, 101.6)
- added D12: bat48, Diode_THT:D_DO-35_SOD27_P10.16mm_Horizontal, B.Cu at (84.5, 101.6)
- added D13: bat48, Diode_THT:D_DO-35_SOD27_P10.16mm_Horizontal, F.Cu at (210.2, 116.8)
- added D13: bat48, Diode_THT:D_DO-35_SOD27_P10.16mm_Horizontal, B.Cu at (84.5, 116.8)
- added D2: D_TVS, Diode_SMD:D_SMB, F.Cu at (203.2, 80.2)
- added D2: D_TVS, Diode_SMD:D_SMB, B.Cu at (91.4, 80.2)
- added D3: D_TVS, Diode_SMD:D_SMB, F.Cu at (197.5, 80.2)
- added D3: D_TVS, Diode_SMD:D_SMB, B.Cu at (97.2, 80.2)
- added D4: D_TVS, Diode_SMD:D_SMB, F.Cu at (203.2, 95.4)
- added D4: D_TVS, Diode_SMD:D_SMB, B.Cu at (91.4, 95.4)
- added D5: D_TVS, Diode_SMD:D_SMB, F.Cu at (197.5, 95.4)
- added D5: D_TVS, Diode_SMD:D_SMB, B.Cu at (97.2, 95.4)
- added D6: D_TVS, Diode_SMD:D_SMB, F.Cu at (203.2, 110.7)
- added D6: D_TVS, Diode_SMD:D_SMB, B.Cu at (91.4, 110.7)
- added D7: D_TVS, Diode_SMD:D_SMB, F.Cu at (197.5, 110.7)
- added D7: D_TVS, Diode_SMD:D_SMB, B.Cu at (97.2, 110.7)
- added D8: D_TVS, Diode_SMD:D_SMB, F.Cu at (203.2, 125.9)
- added D8: D_TVS, Diode_SMD:D_SMB, B.Cu at (91.4, 125.9)
- added D9: D_TVS, Diode_SMD:D_SMB, F.Cu at (197.5, 125.9)
- added D9: D_TVS, Diode_SMD:D_SMB, B.Cu at (97.2, 125.9)
- added H1: mnt, MountingHole:MountingHole_2.2mm_M2_DIN965_Pad, F.Cu at (240.0, 62.2)
- added H1: mnt, MountingHole:MountingHole_2.2mm_M2_DIN965_Pad, B.Cu at (54.6, 62.2)
- added H2: mnt, MountingHole:MountingHole_2.2mm_M2_DIN965_Pad, F.Cu at (184.2, 62.2)
- added H2: mnt, MountingHole:MountingHole_2.2mm_M2_DIN965_Pad, B.Cu at (110.5, 62.2)
- added H3: mnt, MountingHole:MountingHole_2.2mm_M2_DIN965_Pad, F.Cu at (184.2, 143.5)
- added H3: mnt, MountingHole:MountingHole_2.2mm_M2_DIN965_Pad, B.Cu at (110.5, 143.5)
- added H4: mnt, MountingHole:MountingHole_2.2mm_M2_DIN965_Pad, F.Cu at (240.0, 143.5)
- added H4: mnt, MountingHole:MountingHole_2.2mm_M2_DIN965_Pad, B.Cu at (54.6, 143.5)
- added J1: batt_1, power_connectors:XT60UPB-M, F.Cu at (221.0, 81.3)
- added J1: batt_1, power_connectors:XT60UPB-M, B.Cu at (73.7, 81.3)
- added J2: batt_2, power_connectors:XT60UPB-M, F.Cu at (221.0, 96.5)
- added J2: batt_2, power_connectors:XT60UPB-M, B.Cu at (73.7, 96.5)
- added J3: batt_3, power_connectors:XT60UPB-M, F.Cu at (221.0, 111.8)
- added J3: batt_3, power_connectors:XT60UPB-M, B.Cu at (73.7, 111.8)
- added J4: batt_4, power_connectors:XT60UPB-M, F.Cu at (221.0, 127.0)
- added J4: batt_4, power_connectors:XT60UPB-M, B.Cu at (73.7, 127.0)
- added J5: reed_switch, Connector_Molex:Molex_SPOX_5267-02A_1x02_P2.50mm_Vertical, F.Cu at (225.4, 63.5)
- added J5: reed_switch, Connector_Molex:Molex_SPOX_5267-02A_1x02_P2.50mm_Vertical, B.Cu at (69.2, 63.5)
- added J6: toPcb+, MountingHole:MountingHole_4.3mm_M4_DIN965_Pad, B.Cu at (228.0, 139.1)
- added J6: toPcb+, MountingHole:MountingHole_4.3mm_M4_DIN965_Pad, F.Cu at (66.7, 139.1)
- added J7: toPcb-, MountingHole:MountingHole_4.3mm_M4_DIN965_Pad, B.Cu at (214.0, 139.1)
- added J7: toPcb-, MountingHole:MountingHole_4.3mm_M4_DIN965_Pad, F.Cu at (80.6, 139.1)
- added J8: on_signal, Connector_Molex:Molex_SPOX_5267-02A_1x02_P2.50mm_Vertical, F.Cu at (225.4, 72.4)
- added J8: on_signal, Connector_Molex:Molex_SPOX_5267-02A_1x02_P2.50mm_Vertical, B.Cu at (69.2, 72.4)
- added Q1: batt1_sw, Package_TO_SOT_SMD:TO-263-2, B.Cu at (200.0, 79.0)
- added Q1: batt1_sw, Package_TO_SOT_SMD:TO-263-2, F.Cu at (94.6, 79.0)
- added Q2: batt2_sw, Package_TO_SOT_SMD:TO-263-2, B.Cu at (200.3, 94.2)
- added Q2: batt2_sw, Package_TO_SOT_SMD:TO-263-2, F.Cu at (94.4, 94.2)
- added Q3: batt3_sw, Package_TO_SOT_SMD:TO-263-2, B.Cu at (200.3, 109.5)
- added Q3: batt3_sw, Package_TO_SOT_SMD:TO-263-2, F.Cu at (94.4, 109.5)
- added Q4: batt4_sw, Package_TO_SOT_SMD:TO-263-2, B.Cu at (200.3, 124.7)
- added Q4: batt4_sw, Package_TO_SOT_SMD:TO-263-2, F.Cu at (94.4, 124.7)
- added Q5: BC817-25, Package_TO_SOT_SMD:SOT-23_Handsoldering, B.Cu at (215.9, 67.3)
- added Q5: BC817-25, Package_TO_SOT_SMD:SOT-23_Handsoldering, F.Cu at (78.7, 67.3)
- added R1: 400, Resistor_SMD:R_0805_2012Metric, B.Cu at (191.1, 64.8)
- added R1: 400, Resistor_SMD:R_0805_2012Metric, F.Cu at (103.5, 64.8)
- added R10: 680, Resistor_SMD:R_0805_2012Metric_Pad1.15x1.40mm_HandSolder, B.Cu at (232.4, 67.7)
- added R10: 680, Resistor_SMD:R_0805_2012Metric_Pad1.15x1.40mm_HandSolder, F.Cu at (62.2, 67.7)
- added R11: 10k, Resistor_SMD:R_0805_2012Metric, B.Cu at (219.3, 73.0)
- added R11: 10k, Resistor_SMD:R_0805_2012Metric, F.Cu at (75.3, 73.0)
- added R2: 100, Resistor_SMD:R_0805_2012Metric, B.Cu at (215.6, 73.0)
- added R2: 100, Resistor_SMD:R_0805_2012Metric, F.Cu at (79.0, 73.0)
- added R3: 100, Resistor_SMD:R_0805_2012Metric, B.Cu at (215.6, 88.3)
- added R3: 100, Resistor_SMD:R_0805_2012Metric, F.Cu at (79.1, 88.3)
- added R4: 100, Resistor_SMD:R_0805_2012Metric, B.Cu at (215.6, 103.5)
- added R4: 100, Resistor_SMD:R_0805_2012Metric, F.Cu at (79.1, 103.5)
- added R5: 100, Resistor_SMD:R_0805_2012Metric, B.Cu at (215.6, 118.7)
- added R5: 100, Resistor_SMD:R_0805_2012Metric, F.Cu at (79.1, 118.7)
- added R6: 47k, Resistor_SMD:R_0805_2012Metric, B.Cu at (217.5, 75.6)
- added R6: 47k, Resistor_SMD:R_0805_2012Metric, F.Cu at (77.2, 75.6)
- added R7: 47k, Resistor_SMD:R_0805_2012Metric, B.Cu at (217.5, 90.8)
- added R7: 47k, Resistor_SMD:R_0805_2012Metric, F.Cu at (77.2, 90.8)
- added R8: 47k, Resistor_SMD:R_0805_2012Metric, B.Cu at (217.5, 106.0)
- added R8: 47k, Resistor_SMD:R_0805_2012Metric, F.Cu at (77.2, 106.0)
- added R9: 47k, Resistor_SMD:R_0805_2012Metric, B.Cu at (217.5, 121.3)
- added R9: 47k, Resistor_SMD:R_0805_2012Metric, F.Cu at (77.2, 121.3)
- added U1: LM1117-5.0, Package_TO_SOT_SMD:SOT-223-3_TabPin2, B.Cu at (198.1, 66.0)
- added U1: LM1117-5.0, Package_TO_SOT_SMD:SOT-223-3_TabPin2, F.Cu at (96.5, 66.0)
- added U2: LTV-817S, Package_DIP:SMDIP-4_W9.53mm, B.Cu at (224.2, 67.9)
- added U2: LTV-817S, Package_DIP:SMDIP-4_W9.53mm, F.Cu at (70.5, 67.9)
Routing:
- net (no net): track 396.2 -> 1196.3 mm
- net Vin: track 92.8 -> 185.6 mm, vias 4 -> 8
- net gnd: track 87.1 -> 174.2 mm, vias 8 -> 16
- net Net-(D10-Pad2): track 86.3 -> 170.0 mm, vias 2 -> 4
- net Net-(C5-Pad2): track 41.7 -> 83.3 mm, vias 1 -> 2
- net Net-(C4-Pad2): track 41.7 -> 83.3 mm, vias 1 -> 2
- net Net-(C10-Pad1): track 41.6 -> 83.2 mm, vias 1 -> 2
- net Net-(C3-Pad2): track 40.7 -> 81.3 mm, vias 1 -> 2
- net Net-(C9-Pad2): track 28.4 -> 56.8 mm, vias 1 -> 2
- net Net-(C8-Pad2): track 28.1 -> 56.1 mm, vias 1 -> 2
- net Net-(C10-Pad2): track 27.6 -> 55.1 mm, vias 1 -> 2
- net Net-(C7-Pad2): track 25.3 -> 50.6 mm, vias 1 -> 2
- net Net-(D1-Pad2): track 17.1 -> 34.1 mm, vias 1 -> 2
- net Net-(C1-Pad1): track 13.3 -> 26.7 mm
- net Net-(J8-Pad1): track 12.6 -> 25.2 mm
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- added copper zone on B.Cu, net Vin
Other:
- board size 170.2 x 63.5 mm -> 311.1 x 191.8 mm

Commit message: visual fix
Parts:
- C1, C2: value C_Small -> 100n
- D10: value bat48 -> BAT48
- D2, D3, D4, D5, D6, D7, D8, D9: value D_TVS -> P6SMB18CA
- Q1: value batt1_sw -> IRL2203N
- Q2: value batt2_sw -> IRL2203N
- Q3: value batt3_sw -> IRL2203N
- Q4: value batt4_sw -> IRL2203N
- R2: value 100 -> 680
Connections:
- C6 pad 1: gnd -> Net-(C6-Pad1)
- D9 pad 1: gnd -> Net-(C6-Pad1)
- Q4 pad 2: gnd -> Net-(C6-Pad1)
Changed lines of the file:
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@@
     (zones 0)
     (modules 106)
-    (nets 22)
+    (nets 23)
   )
   (page A4)
@@
   (net 20 "Net-(D13-Pad1)")
   (net 21 "Net-(Q5-Pad1)")
+  (net 22 "Net-(C6-Pad1)")
   (net_class Default "To jest domyślna klasa połączeń."
     (clearance 0.2)
@@
     (add_net "Net-(C4-Pad2)")
     (add_net "Net-(C5-Pad2)")
+    (add_net "Net-(C6-Pad1)")
     (add_net "Net-(C7-Pad2)")
     (add_net "Net-(C8-Pad2)")
@@
       (effects (font (size 1 1) (thickness 0.15)))
     )
-    (fp_text value D_TVS (at 0 3.1 270) (layer F.Fab)
+    (fp_text value P6SMB18CA (at 0 3.1 270) (layer F.Fab)
       (effects (font (size 1 1) (thickness 0.15)))
     )
@@
       (effects (font (size 1 1) (thickness 0.15)))
     )
-    (fp_text value bat48 (at 5.08 2.12 90) (layer F.Fab)
+    (fp_text value BAT48 (at 5.08 2.12 90) (layer F.Fab)
       (effects (font (size 1 1) (thickness 0.15)))
     )
@@
       (effects (font (size 1 1) (thickness 0.15)))
     )
-    (fp_text value D_TVS (at 0 3.1 270) (layer F.Fab)
+    (fp_text value P6SMB18CA (at 0 3.1 270) (layer F.Fab)
       (effects (font (size 1 1) (thickness 0.15)))
     )
@@
       (effects (font (size 1 1) (thickness 0.15)) (justify mirror))
     )
-    (fp_text value batt1_sw (at 0 -6.65 180) (layer B.Fab)
+    (fp_text value IRL2203N (at 0 -6.65 180) (layer B.Fab)
       (effects (font (size 1 1) (thickness 0.15)) (justify mirror))
     )
@@
       (effects (font (size 1 1) (thickness 0.15)) (justify mirror))
     )
-    (fp_text value batt2_sw (at 0 -6.65 180) (layer B.Fab)
+    (fp_text value IRL2203N (at 0 -6.65 180) (layer B.Fab)
       (effects (font (size 1 1) (thickness 0.15)) (justify mirror))
     )
@@
       (effects (font (size 1 1) (thickness 0.15)))
     )
-    (fp_text value D_TVS (at 0 3.1 270) (layer F.Fab)
+    (fp_text value P6SMB18CA (at 0 3.1 270) (layer F.Fab)
       (effects (font (size 1 1) (thickness 0.15)))
     )
@@
       (effects (font (size 1 1) (thickness 0.15)))
     )
-    (fp_text value D_TVS (at 0 3.1 270) (layer F.Fab)
+    (fp_text value P6SMB18CA (at 0 3.1 270) (layer F.Fab)
       (effects (font (size 1 1) (thickness 0.15)))
     )
@@
     (fp_line (start -3.55 -2.15) (end 2.15 -2.15) (layer F.SilkS) (width 0.12))
     (pad 1 smd rect (at -2.15 0 270) (size 2.5 2.3) (layers F.Cu F.Paste F.Mask)
-      (net 3 gnd))
+      (net 22 "Net-(C6-Pad1)"))
     (pad 2 smd rect (at 2.15 0 270) (size 2.5 2.3) (layers F.Cu F.Paste F.Mask)
       (net 14 "Net-(C10-Pad1)"))
@@
       (effects (font (size 1 1) (thickness 0.15)) (justify mirror))
     )
-    (fp_text value batt4_sw (at 0 -6.65 180) (layer B.Fab)
+    (fp_text value IRL2203N (at 0 -6.65 180) (layer B.Fab)
       (effects (font (size 1 1) (thickness 0.15)) (justify mirror))
     )
@@
     (pad "" smd rect (at 5.8 -2.775 180) (size 4.55 5.25) (layers B.Paste))
     (pad 2 smd rect (at 3.375 0 180) (size 9.4 10.8) (layers B.Cu B.Mask)
-      (net 3 gnd))
+      (net 22 "Net-(C6-Pad1)"))
     (pad 3 smd rect (at -5.775 -2.54 180) (size 4.6 1.1) (layers B.Cu B.Paste B.Mask)
       (net 14 "Net-(C10-Pad1)"))
@@
       (effects (font (size 1 1) (thickness 0.15)) (justify mirror))
     )
-    (fp_text value C_Small (at -4.2 0 180) (layer B.Fab)
+    (fp_text value 100n (at -4.2 0 180) (layer B.Fab)
       (effects (font (size 1 1) (thickness 0.15)) (justify mirror))
     )
@@
       (net 14 "Net-(C10-Pad1)"))
     (pad 1 smd roundrect (at -1.4875 0 270) (size 1.425 1.75) (layers F.Cu F.Paste F.Mask) (roundrect_rratio 0.175439)
-      (net 3 gnd))
+      (net 22 "Net-(C6-Pad1)"))
     (model ${KISYS3DMOD}/Capacitor_SMD.3dshapes/C_1206_3216Metric.wrl
       (at (xyz 0 0 0))
@@
       (effects (font (size 1 1) (thickness 0.15)) (justify mirror))
     )
-    (fp_text value C_Small (at -0.39 1.27 180) (layer B.Fab)
+    (fp_text value 100n (at -0.39 1.27 180) (layer B.Fab)
       (effects (font (size 1 1) (thickness 0.15)) (justify mirror))
     )
@@
       (effects (font (size 1 1) (thickness 0.15)) (justify mirror))
     )
-    (fp_text value 100 (at 0.3325 -1.905 180) (layer B.Fab)
+    (fp_text value 680 (at 0.3325 -1.905 180) (layer B.Fab)
       (effects (font (size 1 1) (thickness 0.15)) (justify mirror))
     )
@@
       (effects (font (size 1 1) (thickness 0.15)))
     )
-    (fp_text value D_TVS (at 0 3.1 270) (layer F.Fab)
+    (fp_text value P6SMB18CA (at 0 3.1 270) (layer F.Fab)
       (effects (font (size 1 1) (thickness 0.15)))
     )
@@
       (effects (font (size 1 1) (thickness 0.15)))
     )
-    (fp_text value D_TVS (at 0 3.1 270) (layer F.Fab)
+    (fp_text value P6SMB18CA (at 0 3.1 270) (layer F.Fab)
       (effects (font (size 1 1) (thickness 0.15)))
     )
@@
       (effects (font (size 1 1) (thickness 0.15)) (justify mirror))
     )
-    (fp_text value batt3_sw (at 0 -6.65 180) (layer B.Fab)
+    (fp_text value IRL2203N (at 0 -6.65 180) (layer B.Fab)
       (effects (font (size 1 1) (thickness 0.15)) (justify mirror))
     )
@@
       (effects (font (size 1 1) (thickness 0.15)))
     )
-    (fp_text value D_TVS (at 0 3.1 270) (layer F.Fab)
+    (fp_text value P6SMB18CA (at 0 3.1 270) (layer F.Fab)
       (effects (font (size 1 1) (thickness 0.15)))
     )
@@
       (effects (font (size 1 1) (thickness 0.15)))
     )
-    (fp_text value D_TVS (at 0 3.1 270) (layer F.Fab)
-      (effects (font (size 1 1) (thickness 0.15)))
-    )
+    (fp_text value P6SMB18CA (at 0 3.1 270) (layer F.Fab)
+      (effects (font (size 1 1) (thickness 0.15)))
+    )
